Commit message: Modify/add UR3 Cranfield Cell - CAD.

File: ur3/ros2srrc_ur3_gazebo/urdf/ur3.urdf.xacro (robot description, xacro)
@@ -137,11 +137,11 @@
         <origin xyz="0.0 0.0 0.0" rpy="0 0 0" />
         <geometry>
-          <mesh filename="file://$(find ros2srrc_ur3_gazebo)/meshes/ur3_CranfieldCell/r3m_UR3cupboard.dae" scale="1 1 1" />
-        </geometry>
-      </visual>
-      <collision>
-        <origin xyz="0.0 0.0 0.0" rpy="0 0 0" />
-        <geometry>
-          <mesh filename="file://$(find ros2srrc_ur3_gazebo)/meshes/ur3_CranfieldCell/r3m_UR3cupboard.dae" scale="1 1 1" />
+          <mesh filename="file://$(find ros2srrc_ur3_gazebo)/meshes/ur3_CranfieldCell/UR3cupboard.dae" scale="1 1 1" />
+        </geometry>
+      </visual>
+      <collision>
+        <origin xyz="0.0 0.0 0.0" rpy="0 0 0" />
+        <geometry>
+          <mesh filename="file://$(find ros2srrc_ur3_gazebo)/meshes/ur3_CranfieldCell/UR3cupboard.dae" scale="1 1 1" />
         </geometry>
       </collision>
@@ -155,11 +155,11 @@
         <origin xyz="0.0 0.0 0.0" rpy="0 0 0" />
         <geometry>
-          <mesh filename="file://$(find ros2srrc_ur3_gazebo)/meshes/ur3_CranfieldCell/r3m_UR3wall.dae" scale="1 1 1" />
-        </geometry>
-      </visual>
-      <collision>
-        <origin xyz="0.0 0.0 0.0" rpy="0 0 0" />
-        <geometry>
-          <mesh filename="file://$(find ros2srrc_ur3_gazebo)/meshes/ur3_CranfieldCell/r3m_UR3wall.dae" scale="1 1 1" />
+          <mesh filename="file://$(find ros2srrc_ur3_gazebo)/meshes/ur3_CranfieldCell/UR3wall.dae" scale="1 1 1" />
+        </geometry>
+      </visual>
+      <collision>
+        <origin xyz="0.0 0.0 0.0" rpy="0 0 0" />
+        <geometry>
+          <mesh filename="file://$(find ros2srrc_ur3_gazebo)/meshes/ur3_CranfieldCell/UR3wall.dae" scale="1 1 1" />
         </geometry>
       </collision>
@@ -173,11 +173,11 @@
         <origin xyz="0.0 0.0 0.0" rpy="0 0 0" />
         <geometry>
-          <mesh filename="file://$(find ros2srrc_ur3_gazebo)/meshes/ur3_CranfieldCell/r3m_UR3emergencybutton.dae" scale="1 1 1" />
-        </geometry>
-      </visual>
-      <collision>
-        <origin xyz="0.0 0.0 0.0" rpy="0 0 0" />
-        <geometry>
-          <mesh filename="file://$(find ros2srrc_ur3_gazebo)/meshes/ur3_CranfieldCell/r3m_UR3emergencybutton.dae" scale="1 1 1" />
+          <mesh filename="file://$(find ros2srrc_ur3_gazebo)/meshes/ur3_CranfieldCell/UR3emergencybutton.dae" scale="1 1 1" />
+        </geometry>
+      </visual>
+      <collision>
+        <origin xyz="0.0 0.0 0.0" rpy="0 0 0" />
+        <geometry>
+          <mesh filename="file://$(find ros2srrc_ur3_gazebo)/meshes/ur3_CranfieldCell/UR3emergencybutton.dae" scale="1 1 1" />
         </geometry>
       </collision>
@@ -191,11 +191,29 @@
         <origin xyz="0.0 0.0 0.0" rpy="0 0 0" />
         <geometry>
-          <mesh filename="file://$(find ros2srrc_ur3_gazebo)/meshes/ur3_CranfieldCell/r3m_UR3button.dae" scale="1 1 1" />
-        </geometry>
-      </visual>
-      <collision>
-        <origin xyz="0.0 0.0 0.0" rpy="0 0 0" />
-        <geometry>
-          <mesh filename="file://$(find ros2srrc_ur3_gazebo)/meshes/ur3_CranfieldCell/r3m_UR3button.dae" scale="1 1 1" />
+          <mesh filename="file://$(find ros2srrc_ur3_gazebo)/meshes/ur3_CranfieldCell/UR3button.dae" scale="1 1 1" />
+        </geometry>
+      </visual>
+      <collision>
+        <origin xyz="0.0 0.0 0.0" rpy="0 0 0" />
+        <geometry>
+          <mesh filename="file://$(find ros2srrc_ur3_gazebo)/meshes/ur3_CranfieldCell/UR3button.dae" scale="1 1 1" />
+        </geometry>
+      </collision>
+      <inertial>
+        <mass value="1.0"/>
+        <inertia ixx="500.0" ixy="500.0" ixz="500.0" iyy="500.0" iyz="500.0" izz="500.0" />
+      </inertial>
+    </link>
+    <link name='ur3_L'>
+      <visual>
+        <origin xyz="0.0 0.0 0.0" rpy="0 0 0" />
+        <geometry>
+          <mesh filename="file://$(find ros2srrc_ur3_gazebo)/meshes/ur3_CranfieldCell/XVC4B4.dae" scale="1 1 1" />
+        </geometry>
+      </visual>
+      <collision>
+        <origin xyz="0.0 0.0 0.0" rpy="0 0 0" />
+        <geometry>
+          <mesh filename="file://$(find ros2srrc_ur3_gazebo)/meshes/ur3_CranfieldCell/XVC4B4.dae" scale="1 1 1" />
         </geometry>
       </collision>
@@ -222,11 +240,16 @@
     <joint name="eb_joint" type="fixed">
       <parent link="ur3_cell" />
+      <child link = "ur3_B" />
+      <origin xyz="-0.10 0.01 0.762" rpy="0.0 0.0 0.0" />
+    </joint>
+    <joint name="b_joint" type="fixed">
+      <parent link="ur3_cell" />
       <child link = "ur3_EB" />
-      <origin xyz="-0.10 0.01 0.762" rpy="0.0 0.0 0.0" />
-    </joint>
-    <joint name="b_joint" type="fixed">
-      <parent link="ur3_cell" />
-      <child link = "ur3_B" />
       <origin xyz="-0.18 0.01 0.762" rpy="0.0 0.0 0.0" />
+    </joint>
+    <joint name="l_joint" type="fixed">
+      <parent link="ur3_cell" />
+      <child link = "ur3_L" />
+      <origin xyz="0.0 0.0 0.0" rpy="0.0 0.0 0.0" />
     </joint>
   </xacro:if>
