Commit message: Add grasping plugin to RobotiQ 2f-85 gripper.

File: ur3/ros2srrc_ur3_gazebo/urdf/ur3_macro.urdf.xacro (robot description, xacro)
@@ -594,4 +594,24 @@
         <dynamics damping="1.0" friction="1.0"/>
       </joint>
+      <!-- SMALL CUBE FOR GRIPPER PLUGIN -->
+      <link name="EE_robotiq_2f85">
+        <inertial>
+          <origin xyz="0 0 0" rpy="0 0 0" />
+          <mass value="0.00001" />
+          <inertia ixx="0.001" ixy="0.0" ixz="0.0" iyy="0.001" iyz="0.0" izz="0.001"/>
+        </inertial>
+        <visual>
+          <geometry>
+            <box size= "0.001 0.001 0.001" />
+          </geometry>
+        </visual>
+      </link>
+      <joint name="EE_robotiq_2f85_joint" type="prismatic" >
+        <parent link="${prefix}robotiq_85_base_link" />
+        <child link="EE_robotiq_2f85" />
+        <limit effort="10000" lower="0.0" upper="0.0" velocity="0.0"/>
+        <axis xyz="1 0 0" />
+        <origin xyz="0.128 0.0 0.0" rpy="0 0 0"/>
+      </joint>
     </xacro:if>
     <!-- === ROBOTIQ 2f-85 GRIPPER === -->
