Commit message: Minor changes in .urdf files.

File: ur3/ros2srrc_ur3_gazebo/urdf/box.urdf (robot description, URDF)
Before this commit: robot box, 1 links, 0 joints
Links:
- link box: mass 0.1 -> 0.8

File: ur3/ros2srrc_ur3_gazebo/urdf/ur3.urdf.xacro (robot description, xacro)
@@ -154,4 +154,5 @@
       </inertial>
     </link>
+    <!--
     <link name='ur3_wall'>
       <visual>
@@ -172,4 +173,5 @@
       </inertial>
     </link>
+    -->
     <link name='ur3_EB'>
       <visual>
@@ -231,4 +233,5 @@
       <origin xyz="0.0 0.0 0.00" rpy="0.0 0.0 0.0" />
     </joint>
+    <!--
     <joint name="wall_joint" type="fixed">
       <parent link="world" />
@@ -236,4 +239,5 @@
       <origin xyz="0.0 0.0 0.00" rpy="0.0 0.0 0.0" />
     </joint>
+    -->
     <joint name="ur_joint" type="fixed">
       <parent link="ur3_cell" />

Commit message: Modify box.urdf for better p&p simulation.

File: ur3/ros2srrc_ur3_gazebo/urdf/box.urdf (robot description, URDF)
Before this commit: robot box, 1 links, 0 joints
Links:
- link box: mass 0.8 -> 0.01
