Commit message: Update repo: Remove dependence on ros2_RobotSimulation.

File: irb120/ros2srrc_irb120_gazebo/urdf/box.urdf (robot description, URDF)
Before this commit: robot box, 1 links, 0 joints
Links:
- link box: geometry collision box size=0.03 0.03 0.03; visual box size=0.03 0.03 0.03

Commit message: Modify inertial value for "box" and cubePP program.

File: irb120/ros2srrc_irb120_gazebo/urdf/box.urdf (robot description, URDF)
Before this commit: robot box, 1 links, 0 joints
Links:
- link box: mass 0.01 -> 0.1
