Commit message: Fix: IRB120 cell (I/O-s + egp64).

File: irb120/ros2srrc_irb120_gazebo/urdf/irb120.urdf.xacro (robot description, xacro)
@@ -104,5 +104,5 @@
       <parent link="cell"/>
       <child link="base_link"/>
-      <origin xyz="-0.7006 0.6489 0.8605" rpy="0.0 0.0 0.0" />
+      <origin xyz="-0.6506 0.6489 0.8605" rpy="0.0 0.0 0.0" />
     </joint>
   </xacro:if>

File: irb120/ros2srrc_irb120_gazebo/urdf/irb120_macro.urdf.xacro (robot description, xacro)
@@ -318,5 +318,5 @@
         </collision>
         <inertial>
-          <origin xyz="0 0 0" rpy="0 0 ${pi/4}" />
+          <origin xyz="0 0 0" rpy="0 0 ${pi/2}" />
           <mass value="0.001" />
           <inertia ixx="0.001" ixy="0.0" ixz="0.0" iyy="0.001" iyz="0.0" izz="0.001"/>
@@ -325,5 +325,5 @@
       <!-- Schunk coupler (JOINT): -->
       <joint name="schunk_coupler_joint" type="fixed">
-        <origin xyz="0 0 0.001" rpy="0 0 ${pi/4}" />
+        <origin xyz="0 0 0.001" rpy="0 0 ${pi/2}" />
         <parent link="tool0"/>
         <child link="schunk_coupler"/>

File: irb120/ros2srrc_irb120_gazebo/urdf/irb120_ros2control.xacro (robot description, xacro)
@@ -169,5 +169,5 @@
         </command_interface>
         <state_interface name="position">
-          <param name="initial_value">0.0</param>
+          <param name="initial_value">0.523599</param>
         </state_interface>
         <state_interface name="velocity"/>

Commit message: Add the pick&place layout variant to irb120.

File: irb120/ros2srrc_irb120_gazebo/urdf/irb120.urdf.xacro (robot description, xacro)
@@ -53,4 +53,6 @@
   <xacro:arg name="cell_layout_2" default="false"/>
   <xacro:property name="cell_layout_2" value="$(arg cell_layout_2)"/>
+  <xacro:arg name="cell_layout_3" default="false"/>
+  <xacro:property name="cell_layout_3" value="$(arg cell_layout_3)"/>
   <xacro:property name="EE_no" value="$(arg EE_no)"/>
   <xacro:arg name="EE_schunk" default="false"/>
@@ -108,3 +110,66 @@
   </xacro:if>
   <!-- === IA Lab - IRB120 Enclosure === -->
+  <!-- === Pick and Place use-case === -->
+  <xacro:if value="${cell_layout_3}">
+    <link name='irb120_block'>
+      <inertial>
+        <origin xyz="0 0 0" rpy="0 0 0"/>
+        <mass value="100"/>
+        <inertia ixx="0.01"  ixy="0"  ixz="0" iyy="0.01" iyz="0" izz="0.01" />
+      </inertial>
+      <collision name='collision'>
+        <origin xyz="0 0 0" rpy=" 0 0 0"/>
+        <geometry>
+          <box size = "0.2 0.2 0.5"/>
+        </geometry>
+      </collision>
+      <visual name='chassis_visual'>
+        <origin xyz="0 0 0" rpy=" 0 0 0"/>
+        <geometry>
+          <box size = "0.2 0.2 0.5"/>
+        </geometry>
+        <material name="red">
+          <color rgba="1 0 0 1"/>
+        </material>
+      </visual>
+    </link>
+    <joint name="world_joint" type="fixed">
+      <parent link="world" />
+      <child link = "irb120_block" />
+      <origin xyz="0.0 0.0 0.25" rpy="0.0 0.0 0.0" />
+    </joint>
+    <joint name="block-base" type="fixed">
+      <parent link="irb120_block" />
+      <child link = "base_link" />
+      <origin xyz="0.0 0.0 0.255" rpy="0.0 0.0 0.0" />
+    </joint>
+    <link name='table'>
+      <inertial>
+        <origin xyz="0 0 0" rpy="0 0 0"/>
+        <mass value="100"/>
+        <inertia ixx="0.01"  ixy="0"  ixz="0" iyy="0.01" iyz="0" izz="0.01" />
+      </inertial>
+      <collision name='collision'>
+        <origin xyz="0 0 0" rpy=" 0 0 0"/>
+        <geometry>
+          <box size = "0.5 1.0 0.7"/>
+        </geometry>
+      </collision>
+      <visual name='chassis_visual'>
+        <origin xyz="0 0 0" rpy=" 0 0 0"/>
+        <geometry>
+          <box size = "0.5 1.0 0.7"/>
+        </geometry>
+        <material name="black">
+          <color rgba="1 0 0 1"/>
+        </material>
+      </visual>
+    </link>
+    <joint name="table_world" type="fixed">
+      <parent link="world" />
+      <child link = "table" />
+      <origin xyz="0.7 0.0 0.35" rpy="0.0 0.0 0.0" />
+    </joint>
+  </xacro:if>
+  <!-- === Pick and Place use-case === -->
 </robot>

Commit message: Upload ergobox to IA-Lab (IRB120) layout.

File: irb120/ros2srrc_irb120_gazebo/urdf/irb120.urdf.xacro (robot description, xacro)
@@ -108,4 +108,27 @@
       <origin xyz="-0.6506 0.6489 0.8605" rpy="0.0 0.0 0.0" />
     </joint>
+    <link name="ergobox">
+      <visual>
+        <origin xyz="0.0 0.0 0.0" rpy="0 0 0" />
+        <geometry>
+          <mesh filename="file://$(find ros2srrc_irb120_gazebo)/meshes/IALab/ergobox.dae" scale="1 1 1" />
+        </geometry>
+      </visual>
+      <collision>
+        <origin xyz="0.0 0.0 0.0" rpy="0 0 0" />
+        <geometry>
+          <mesh filename="file://$(find ros2srrc_irb120_gazebo)/meshes/IALab/ergobox.dae" scale="1 1 1" />
+        </geometry>
+      </collision>
+      <inertial>
+        <mass value="10.0"/>
+        <inertia ixx="0.0002" ixy="0.0002" ixz="0.0002" iyy="0.0" iyz="0.0" izz="0.0" />
+      </inertial>
+    </link>
+    <joint name="cell-ergobox-fixed" type="fixed">
+      <parent link="cell"/>
+      <child link="ergobox"/>
+      <origin xyz="-0.3 0.32 0.8605" rpy="0.0 0.0 0.0" />
+    </joint>
   </xacro:if>
   <!-- === IA Lab - IRB120 Enclosure === -->

Commit message: Fix IRB120 packages: Coordinates (origin) + urdf.

File: irb120/ros2srrc_irb120_gazebo/urdf/irb120.urdf.xacro (robot description, xacro)
@@ -102,4 +102,5 @@
       <parent link="world"/>
       <child link="cell"/>
+      <origin xyz="0.926 -0.124 0.0" rpy="0.0 0.0 0.0" />
     </joint>
     <joint name="cell-base_link-fixed" type="fixed">

File: irb120/ros2srrc_irb120_gazebo/urdf/irb120_macro.urdf.xacro (robot description, xacro)
@@ -301,44 +301,4 @@
       <child link="${prefix}tool0" />
     </joint>
-    <!-- EXTRA LINK + JOINT for the base_link to appear in Gazebo and to be able to calculate TRANSFORMS: -->
-    <link name="BASE_TF">
-      <inertial>
-        <origin xyz="0 0 0" rpy="0 0 0" />
-        <mass value="0.00001" />
-        <inertia ixx="0.001" ixy="0.0" ixz="0.0" iyy="0.001" iyz="0.0" izz="0.001"/>
-      </inertial>
-      <visual>
-        <geometry>
-          <box size= "0.00001 0.00001 0.00001" />
-        </geometry>
-      </visual>
-    </link>
-    <joint name="BASE_TF_joint" type="prismatic" >
-      <parent link="base_link" />
-      <child link="BASE_TF" />
-      <limit effort="10000" lower="0.0" upper="0.0" velocity="0.0"/>
-      <axis xyz="1 0 0" />
-      <origin xyz="0.0 0.0 0.0" rpy="0 0 0"/>
-    </joint>
-    <!-- EXTRA LINK + JOINT for the TCP to appear in Gazebo and to be able to calculate TRANSFORMS: -->
-    <link name="TCP">
-      <inertial>
-        <origin xyz="0 0 0" rpy="0 0 0" />
-        <mass value="0.00001" />
-        <inertia ixx="0.001" ixy="0.0" ixz="0.0" iyy="0.001" iyz="0.0" izz="0.001"/>
-      </inertial>
-      <visual>
-        <geometry>
-          <box size= "0.00001 0.00001 0.00001" />
-        </geometry>
-      </visual>
-    </link>
-    <joint name="TCP_joint" type="prismatic" >
-      <parent link="${prefix}link_6" />
-      <child link="TCP" />
-      <limit effort="10000" lower="0.0" upper="0.0" velocity="0.0"/>
-      <axis xyz="1 0 0" />
-      <origin xyz="0.0 0.0 0.0" rpy="0 ${radians(90)} 0"/>
-    </joint>
     <!-- =================================== -->
     <!-- ========== END-EFFECTORS ========== -->
@@ -523,11 +483,20 @@
         </visual>
       </link>
-      <joint name="EE_egp64_joint" type="prismatic" >
-        <parent link="egp64_gripper_base_link" />
-        <child link="EE_egp64" />
-        <limit effort="10000" lower="0.0" upper="0.0" velocity="0.0"/>
-        <axis xyz="1 0 0" />
-        <origin xyz="0.033 -0.018 0.15" rpy="0 0 0"/>
-      </joint>
+      <xacro:unless value="${bringup}">
+        <joint name="EE_egp64_joint" type="prismatic" >
+          <parent link="tool0" />
+          <child link="EE_egp64" />
+          <limit effort="10000" lower="0.0" upper="0.0" velocity="0.0"/>
+          <axis xyz="1 0 0" />
+          <origin xyz="0.0 0.0 0.19" rpy="0 0 0"/>
+        </joint>
+      </xacro:unless>
+      <xacro:if value="${bringup}">
+        <joint name="EE_egp64_joint" type="fixed" >
+          <parent link="tool0" />
+          <child link="EE_egp64" />
+          <origin xyz="0.0 0.0 0.19" rpy="0 0 0"/>
+        </joint>
+      </xacro:if>
     </xacro:if>
     <!-- === SCHUNK EGP-64 GRIPPER === -->

File: irb120/ros2srrc_irb120_gazebo/urdf/irb120_ros2control.xacro (robot description, xacro)
@@ -161,6 +161,6 @@
       <joint name="${prefix}joint_5">
         <command_interface name="position">
-          <param name="min">-2.094395</param>
-          <param name="max">2.094395</param>
+          <param name="min">-2.00</param>       <!-- Joint5 limits lowered to +-2rad -->
+          <param name="max">2.00</param>
         </command_interface>
         <command_interface name="velocity">
@@ -169,5 +169,5 @@
         </command_interface>
         <state_interface name="position">
-          <param name="initial_value">0.523599</param>
+          <param name="initial_value">1.570796</param>
         </state_interface>
         <state_interface name="velocity"/>
@@ -221,4 +221,10 @@
             <state_interface name="velocity"/>
           </joint>
+          <joint name="EE_egp64_joint">
+            <command_interface name="position"/>
+            <command_interface name="velocity"/>
+            <state_interface name="position"/>
+            <state_interface name="velocity"/>
+          </joint>
         </xacro:if>
       </xacro:unless>

Commit message: Adapt the IRB120 packages to the new HMI input (layout/endeffector/robot_ip in terminal launch command).

File: irb120/ros2srrc_irb120_gazebo/urdf/irb120.urdf.xacro (robot description, xacro)
@@ -197,3 +197,78 @@
   </xacro:if>
   <!-- === Pick and Place use-case === -->
+  <xacro:unless value="${bringup}">
+  <!-- CAMERA for R3M-HMI -->
+    <link name="HMI_camera_link">
+      <collision>
+        <origin xyz="0 0 0" rpy="0 0 0"/>
+        <geometry>
+          <box size="0.05 0.05 0.05"/>
+        </geometry>
+      </collision>
+      <visual>
+        <origin xyz="0 0 0" rpy="0 0 0"/>
+        <geometry>
+          <box size="0.05 0.05 0.05"/>
+        </geometry>
+      </visual>
+      <inertial>
+        <mass value="1.0" />
+        <origin xyz="0 0 0" rpy="0 0 0"/>
+        <inertia ixx="0.0" ixy="0.0" ixz="0.0" iyy="0.0" iyz="0.0" izz="0.0" />
+      </inertial>
+    </link>
+    <xacro:if value="${cell_layout_1}">
+      <joint name="HMI_camera_joint" type="fixed">
+        <origin xyz="2.0 1.0 1.0" rpy="0 0.35 -2.6"/>
+        <parent link="world"/>
+        <child link="HMI_camera_link"/>
+      </joint>
+    </xacro:if>
+    <xacro:if value="${cell_layout_2}">
+      <joint name="HMI_camera_joint" type="fixed">
+        <origin xyz="2.0 1.5 2.0" rpy="0 0.35 -2.6"/>
+        <parent link="world"/>
+        <child link="HMI_camera_link"/>
+      </joint>
+    </xacro:if>
+    <xacro:if value="${cell_layout_3}">
+      <joint name="HMI_camera_joint" type="fixed">
+        <origin xyz="2.0 1.0 1.5" rpy="0 0.35 -2.6"/>
+        <parent link="world"/>
+        <child link="HMI_camera_link"/>
+      </joint>
+    </xacro:if>
+    <gazebo reference="HMI_camera_link">
+      <sensor name="HMI_camera" type="camera">
+        <update_rate>30</update_rate>
+        <camera name="head">
+          <horizontal_fov>1.22</horizontal_fov>
+          <image>
+            <width>1920</width>
+            <height>1080</height>
+            <format>R8G8B8</format>
+          </image>
+          <clip>
+            <near>0.02</near>
+            <far>300</far>
+          </clip>
+          <noise>
+            <type>gaussian</type>
+            <mean>0.0</mean>
+            <stddev>0.007</stddev>
+          </noise>
+        </camera>
+        <plugin filename="libgazebo_ros_camera.so" name="HMI_camera_controller">
+          <robotNamespace/>
+          <alwaysOn>true</alwaysOn>
+          <updateRate>0.0</updateRate>
+          <cameraName>HMI_camera</cameraName>
+          <imageTopicName>HMI_image_raw</imageTopicName>
+          <cameraInfoTopicName>HMI_camera_info</cameraInfoTopicName>
+          <frameName>HMI_camera</frameName>
+          <hackBaseline>0.07</hackBaseline>
+        </plugin>
+      </sensor>
+    </gazebo>
+  </xacro:unless>
 </robot>
