Commit message: Add the IALab/UR10e Collaborative Table (CAD).

File: ur10e/ros2srrc_ur10e_gazebo/urdf/ur10e.urdf.xacro (robot description, xacro)
@@ -131,5 +131,35 @@
   </xacro:if>
   <!-- === Cylindric BASE === -->
-  <!-- === Cranfield University - Lab Cell === -->
-  <!-- === Cranfield University - Lab Cell === -->
+  <!-- === Cranfield University - UR10e COOLLABORATIVE CELL === -->
+  <xacro:if value="${cell_layout_3}">
+    <link name="cell">
+      <visual>
+        <origin xyz="0.0 0.0 0.0" rpy="0 0 0" />
+        <geometry>
+          <mesh filename="file://$(find ros2srrc_ur10e_gazebo)/meshes/ur10e_CranfieldCell/IALab_CollabTableGz.dae" scale="1 1 1" />
+          <!-- If willing to use only the TOP of the table (lighter for simulation): /IALab_CollabTableTOP.dae -->
+        </geometry>
+      </visual>
+      <collision>
+        <origin xyz="0.0 0.0 0.0" rpy="0 0 0" />
+        <geometry>
+          <mesh filename="file://$(find ros2srrc_ur10e_gazebo)/meshes/ur10e_CranfieldCell/IALab_CollabTableGz.dae" scale="1 1 1" />
+        </geometry>
+      </collision>
+      <inertial>
+        <mass value="1000.0"/>
+        <inertia ixx="500.0" ixy="500.0" ixz="500.0" iyy="500.0" iyz="500.0" izz="500.0" />
+      </inertial>
+    </link>
+    <joint name="world-cell-fixed" type="fixed">
+      <parent link="world"/>
+      <child link="cell"/>
+    </joint>
+    <joint name="cell-base_link-fixed" type="fixed">
+      <parent link="cell"/>
+      <child link="base_link"/>
+      <origin xyz="-0.965 -1.0 0.866" rpy="0.0 0.0 -0.785398" />
+    </joint>
+  </xacro:if>
+  <!-- === Cranfield University - UR10e COOLLABORATIVE CELL === -->
 </robot>

File: ur10e/ros2srrc_ur10e_gazebo/urdf/ur10e_ros2control.xacro (robot description, xacro)
@@ -164,5 +164,5 @@
         </command_interface>
         <state_interface name="position">
-          <param name="initial_value">0.0</param>
+          <param name="initial_value">${pi/4}</param>
         </state_interface>
         <state_interface name="velocity"/>
@@ -194,5 +194,5 @@
         </command_interface>
         <state_interface name="position">
-          <param name="initial_value">0.0</param>
+          <param name="initial_value">${pi/2}</param>
         </state_interface>
         <state_interface name="velocity"/>

Commit message: Upload IALab "Table" and "Table+Wall" variants to UR10e packages.

File: ur10e/ros2srrc_ur10e_gazebo/urdf/ur10e.urdf.xacro (robot description, xacro)
@@ -62,4 +62,10 @@
   <xacro:arg name="cell_layout_3" default="false"/>
   <xacro:property name="cell_layout_3" value="$(arg cell_layout_3)"/>
+  <xacro:arg name="cell_layout_4" default="false"/>
+  <xacro:property name="cell_layout_4" value="$(arg cell_layout_4)"/>
+  <xacro:arg name="cell_layout_5" default="false"/>
+  <xacro:property name="cell_layout_5" value="$(arg cell_layout_5)"/>
+  <xacro:arg name="rotate_InitialPose" default="false"/>
+  <xacro:property name="rotate_InitialPose" value="$(arg rotate_InitialPose)"/>
   <xacro:arg name="EE_no" default="false"/>
   <xacro:property name="EE_no" value="$(arg EE_no)"/>
@@ -78,4 +84,5 @@
   <xacro:ur10e
     prefix=""
+    rotate_InitialPose="${rotate_InitialPose}"
     EE_no="${EE_no}"
     bringup="${bringup}"
@@ -163,3 +170,65 @@
   </xacro:if>
   <!-- === Cranfield University - UR10e COOLLABORATIVE CELL === -->
+  <!-- === Cranfield University - IA Lab Table === -->
+  <xacro:if value="${cell_layout_4}">
+    <link name="cell">
+      <visual>
+        <origin xyz="0.0 0.0 0.0" rpy="0 0 0" />
+        <geometry>
+          <mesh filename="file://$(find ros2srrc_ur10e_gazebo)/meshes/ur10e_CranfieldCell/IALab_Table.dae" scale="1 1 1" />
+        </geometry>
+      </visual>
+      <collision>
+        <origin xyz="0.0 0.0 0.0" rpy="0 0 0" />
+        <geometry>
+          <mesh filename="file://$(find ros2srrc_ur10e_gazebo)/meshes/ur10e_CranfieldCell/IALab_Table.dae" scale="1 1 1" />
+        </geometry>
+      </collision>
+      <inertial>
+        <mass value="1000.0"/>
+        <inertia ixx="500.0" ixy="500.0" ixz="500.0" iyy="500.0" iyz="500.0" izz="500.0" />
+      </inertial>
+    </link>
+    <joint name="world-cell-fixed" type="fixed">
+      <parent link="world"/>
+      <child link="cell"/>
+    </joint>
+    <joint name="cell-base_link-fixed" type="fixed">
+      <parent link="cell"/>
+      <child link="base_link"/>
+      <origin xyz="0.36 0.55 0.805" rpy="0.0 0.0 -1.5708" />
+    </joint>
+  </xacro:if>
+  <!-- === Cranfield University - IA Lab Table === -->
+  <!-- === Cranfield University - IA Lab Table + Wall === -->
+  <xacro:if value="${cell_layout_5}">
+    <link name="cell">
+      <visual>
+        <origin xyz="0.0 0.0 0.0" rpy="0 0 0" />
+        <geometry>
+          <mesh filename="file://$(find ros2srrc_ur10e_gazebo)/meshes/ur10e_CranfieldCell/IALab_TableWall.dae" scale="1 1 1" />
+        </geometry>
+      </visual>
+      <collision>
+        <origin xyz="0.0 0.0 0.0" rpy="0 0 0" />
+        <geometry>
+          <mesh filename="file://$(find ros2srrc_ur10e_gazebo)/meshes/ur10e_CranfieldCell/IALab_TableWall.dae" scale="1 1 1" />
+        </geometry>
+      </collision>
+      <inertial>
+        <mass value="1000.0"/>
+        <inertia ixx="500.0" ixy="500.0" ixz="500.0" iyy="500.0" iyz="500.0" izz="500.0" />
+      </inertial>
+    </link>
+    <joint name="world-cell-fixed" type="fixed">
+      <parent link="world"/>
+      <child link="cell"/>
+    </joint>
+    <joint name="cell-base_link-fixed" type="fixed">
+      <parent link="cell"/>
+      <child link="base_link"/>
+      <origin xyz="-1.45 -0.65 0.805" rpy="0.0 0.0 -1.5708" />
+    </joint>
+  </xacro:if>
+  <!-- === Cranfield University - IA Lab Table + Wall === -->
 </robot>

File: ur10e/ros2srrc_ur10e_gazebo/urdf/ur10e_macro.urdf.xacro (robot description, xacro)
@@ -58,5 +58,5 @@
   <xacro:include filename="$(find ros2srrc_ur10e_gazebo)/urdf/ur10e_common.xacro" />
   <!-- XACRO-MACRO of UR10e: -->
-  <xacro:macro name="ur10e" params="prefix EE_no bringup robot_ip script_filename input_recipe_filename output_recipe_filename">
+  <xacro:macro name="ur10e" params="prefix rotate_InitialPose EE_no bringup robot_ip script_filename input_recipe_filename output_recipe_filename">
     <!-- LOAD UR10e-Common: -->
     <xacro:ur10e_common/>
@@ -72,4 +72,5 @@
     <xacro:ur10e_ros2control
       prefix=""
+      rotate_InitialPose="${rotate_InitialPose}"
       EE_no="${EE_no}"
       bringup="${bringup}"

File: ur10e/ros2srrc_ur10e_gazebo/urdf/ur10e_ros2control.xacro (robot description, xacro)
@@ -95,5 +95,5 @@
   <xacro:property name="tool_tcp_port" value="$(arg tool_tcp_port)"/>
   <!-- UR10e_CONTROL: -->
-  <xacro:macro name="ur10e_ros2control" params="prefix EE_no bringup robot_ip script_filename input_recipe_filename output_recipe_filename" >
+  <xacro:macro name="ur10e_ros2control" params="prefix rotate_InitialPose EE_no bringup robot_ip script_filename input_recipe_filename output_recipe_filename" >
     <!-- 1. ROS2_CONTROL tag name: -->
     <!-- A. GAZEBO SIMULATION: -->
@@ -164,5 +164,10 @@
         </command_interface>
         <state_interface name="position">
-          <param name="initial_value">${pi/4}</param>
+          <xacro:unless value="${rotate_InitialPose}">
+            <param name="initial_value">${pi/4}</param>
+          </xacro:unless>
+          <xacro:if value="${rotate_InitialPose}">
+            <param name="initial_value">${pi/2}</param>
+          </xacro:if>
         </state_interface>
         <state_interface name="velocity"/>
