Commit message: Lower EE_gpp5010nc 1cm for better grasping.

File: ros2srrc_endeffectors/gpp5010nc/urdf/gpp5010ncv2_macro.urdf.xacro (robot description, xacro)
@@ -134,5 +134,5 @@
       <parent link="${parent_link}" />
       <child link="EE_gpp5010nc" />
-      <origin xyz="-0.16 0.0 0.0" rpy="0 0 0"/>
+      <origin xyz="-0.17 0.0 0.0" rpy="0 0 0"/>
     </joint>
     <gazebo reference="EE_gpp5010nc_joint">
