Commit message: Fix EE_gpp5010nc_joint position for BD gripper.

File: ros2srrc_endeffectors/gpp5010nc/urdf/gpp5010nc_macro.urdf.xacro (robot description, xacro)
@@ -134,5 +134,5 @@
       <parent link="${parent_link}" />
       <child link="EE_gpp5010nc" />
-      <origin xyz="-0.10 0.0 0.0" rpy="0 0 0"/>
+      <origin xyz="-0.118 0.0 0.0" rpy="0 0 0"/>
     </joint>
     <gazebo reference="EE_gpp5010nc_joint">

Commit message: natasha_ur5e

File: ros2srrc_endeffectors/gpp5010nc/urdf/gpp5010nc_macro.urdf.xacro (robot description, xacro)
@@ -134,5 +134,5 @@
       <parent link="${parent_link}" />
       <child link="EE_gpp5010nc" />
-      <origin xyz="-0.118 0.0 0.0" rpy="0 0 0"/>
+      <origin xyz="-0.10 0.0 0.0" rpy="0 0 0"/>
     </joint>
     <gazebo reference="EE_gpp5010nc_joint">

File: ros2srrc_endeffectors/gpp5010nc/urdf/gpp5010ncv2_macro.urdf.xacro (robot description, xacro)
@@ -134,5 +134,5 @@
       <parent link="${parent_link}" />
       <child link="EE_gpp5010nc" />
-      <origin xyz="-0.17 0.0 0.0" rpy="0 0 0"/>
+      <origin xyz="-0.16 0.0 0.0" rpy="0 0 0"/>
     </joint>
     <gazebo reference="EE_gpp5010nc_joint">

File: ros2srrc_robots/irb6640/urdf/irb6640_macro.urdf.xacro (robot description, xacro)
@@ -280,5 +280,5 @@
     </joint>
     <joint type="revolute" name="joint_5">
-      <origin xyz="1.142 0 0 " rpy="0 0 0"/>
+      <origin xyz="1.28 0 0 " rpy="0 0 0"/>
       <axis xyz="0 1 0"/>
       <parent link="link_4"/>

File: ros2srrc_robots/irb6640/urdf/irb6640_ros2control.xacro (robot description, xacro)
@@ -166,18 +166,16 @@
       </joint>
       <!-- CYLINDER&PISTON -->
-      <xacro:unless value="${bringup}">
-        <joint name="joint_cylinder">
-          <param name="mimic">joint_2</param>
-          <param name="multiplier">-0.35</param>
-          <state_interface name="position"/>
-          <state_interface name="velocity"/>
-        </joint>
-        <joint name="joint_piston">
-          <param name="mimic">joint_2</param>
-          <param name="multiplier">-1.35</param>
-          <state_interface name="position"/>
-          <state_interface name="velocity"/>
-        </joint>
-      </xacro:unless>
+      <joint name="joint_cylinder">
+        <param name="mimic">joint_2</param>
+        <param name="multiplier">-0.35</param>
+        <state_interface name="position"/>
+        <state_interface name="velocity"/>
+      </joint>
+      <joint name="joint_piston">
+        <param name="mimic">joint_2</param>
+        <param name="multiplier">-1.35</param>
+        <state_interface name="position"/>
+        <state_interface name="velocity"/>
+      </joint>
       <!-- END EFFECTOR -->
       <xacro:unless value="${bringup}">
