Commit message: Fix: IRB6640 urdf and (piston+cylinder).

File: ros2srrc_robots/irb6640/urdf/irb6640_macro.urdf.xacro (robot description, xacro)
@@ -252,5 +252,5 @@
     <!-- joint list -->
     <joint type="revolute" name="joint_1">
-      <origin xyz="0 0 0" rpy="0 0 0"/>
+      <origin xyz="0 0 0.78" rpy="0 0 0"/>
       <axis xyz="0 0 1"/>
       <parent link="base_link"/>
@@ -259,5 +259,5 @@
     </joint>
     <joint type="revolute" name="joint_2">
-      <origin xyz="0 0 0" rpy="0 0 0"/>
+      <origin xyz="0.32 0 0" rpy="0 0 0"/>
       <axis xyz="0 1 0"/>
       <parent link="link_1"/>
@@ -266,5 +266,5 @@
     </joint>
     <joint type="revolute" name="joint_3">
-      <origin xyz="0 0 0" rpy="0 0 0"/>
+      <origin xyz="0 0 1.28" rpy="0 0 0"/>
       <axis xyz="0 1 0"/>
       <parent link="link_2"/>
@@ -273,5 +273,5 @@
     </joint>
     <joint type="revolute" name="joint_4">
-      <origin xyz="0 0 0" rpy="0 0 0"/>
+      <origin xyz="0 0 0.2" rpy="0 0 0"/>
       <axis xyz="1 0 0"/>
       <parent link="link_3"/>
@@ -280,5 +280,5 @@
     </joint>
     <joint type="revolute" name="joint_5">
-      <origin xyz="0 0 0 " rpy="0 0 0"/>
+      <origin xyz="1.28 0 0 " rpy="0 0 0"/>
       <axis xyz="0 1 0"/>
       <parent link="link_4"/>
@@ -287,5 +287,5 @@
     </joint>
     <joint type="revolute" name="joint_6">
-      <origin xyz="0 0 0 " rpy="0 0 0"/>
+      <origin xyz="0.2 0 0 " rpy="0 0 0"/>
       <axis xyz="1 0 0"/>
       <parent link="link_5"/>
@@ -294,16 +294,16 @@
     </joint>
     <joint type="continuous" name="joint_cylinder">
-      <origin xyz="0 0 0" rpy="0 0 0"/>
+      <origin xyz="-0.365 0 -0.145" rpy="0 0 0"/>
       <axis xyz="0 1 0"/>
       <parent link="link_1"/>
       <child link="link_cylinder"/>
-      <mimic joint="joint_2" multiplier="-0.25"/>
+      <mimic joint="joint_2" multiplier="-0.35" offset="0.0"/>
     </joint>
     <joint type="continuous" name="joint_piston">
-      <origin xyz="0 0 0" rpy="0 0 0"/>
+      <origin xyz="-0.22 0 -0.0673" rpy="0 0 0"/>
       <axis xyz="0 1 0"/>
       <parent link="link_2"/>
       <child link="link_piston"/>
-      <mimic joint="joint_2" multiplier="-1.25"/>
+      <mimic joint="joint_2" multiplier="-1.35" offset="0.0"/>
     </joint>
     <!-- end of joint list -->

File: ros2srrc_robots/irb6640/urdf/irb6640_ros2control.xacro (robot description, xacro)
@@ -165,4 +165,17 @@
         <state_interface name="velocity"/>
       </joint>
+      <!-- CYLINDER&PISTON -->
+      <joint name="joint_cylinder">
+        <param name="mimic">joint_2</param>
+        <param name="multiplier">-0.35</param>
+        <state_interface name="position"/>
+        <state_interface name="velocity"/>
+      </joint>
+      <joint name="joint_piston">
+        <param name="mimic">joint_2</param>
+        <param name="multiplier">-1.35</param>
+        <state_interface name="position"/>
+        <state_interface name="velocity"/>
+      </joint>
       <!-- END EFFECTOR -->
       <xacro:unless value="${bringup}">
@@ -180,7 +193,4 @@
         <selfCollide>false</selfCollide>
       </gazebo>
-      <gazebo reference="link_2_low">
-        <selfCollide>false</selfCollide>
-      </gazebo>
       <gazebo reference="link_2">
         <selfCollide>false</selfCollide>
@@ -198,8 +208,8 @@
         <selfCollide>false</selfCollide>
       </gazebo>
-      <gazebo reference="cylinder">
-        <selfCollide>false</selfCollide>
-      </gazebo>
-      <gazebo reference="piston">
+      <gazebo reference="link_cylinder">
+        <selfCollide>false</selfCollide>
+      </gazebo>
+      <gazebo reference="link_piston">
         <selfCollide>false</selfCollide>
       </gazebo>

File: ros2srrc_robots/irb6640/urdf/irb6640_transmission.xacro (robot description, xacro)
@@ -103,4 +103,22 @@
       </actuator>
     </transmission>
+    <transmission name="joint_cylinder_trans">
+      <type>transmission_interface/SimpleTransmission</type>
+      <joint name="joint_cylinder">
+        <hardwareInterface>hardware_interface/PositionJointInterface</hardwareInterface>
+      </joint>
+      <actuator name="joint_cylinder_motor">
+        <mechanicalReduction>1</mechanicalReduction>
+      </actuator>
+    </transmission>
+    <transmission name="joint_piston_trans">
+      <type>transmission_interface/SimpleTransmission</type>
+      <joint name="joint_piston">
+        <hardwareInterface>hardware_interface/PositionJointInterface</hardwareInterface>
+      </joint>
+      <actuator name="joint_piston_motor">
+        <mechanicalReduction>1</mechanicalReduction>
+      </actuator>
+    </transmission>
   </xacro:macro>
 </robot>

Commit message: Fix: joint_1 limits for IRB6640.

File: ros2srrc_robots/irb6640/urdf/irb6640_macro.urdf.xacro (robot description, xacro)
@@ -256,5 +256,5 @@
       <parent link="base_link"/>
       <child link="link_1"/>
-      <limit effort="0" lower="-1.2217" upper="1.2217" velocity="1.7453"/>
+      <limit effort="0" lower="-2.96706" upper="2.96706" velocity="1.7453"/>
     </joint>
     <joint type="revolute" name="joint_2">

File: ros2srrc_robots/irb6640/urdf/irb6640_ros2control.xacro (robot description, xacro)
@@ -78,6 +78,6 @@
       <joint name="joint_1">
         <command_interface name="position">
-          <param name="min">-1.2217</param>
-          <param name="max">1.2217</param>
+          <param name="min">-2.96706</param>
+          <param name="max">2.96706</param>
         </command_interface>
         <command_interface name="velocity">

Commit message: Fix: Zimmer gripper client + IRB6640 urdf for bringup control.

File: ros2srrc_robots/irb6640/urdf/irb6640_macro.urdf.xacro (robot description, xacro)
@@ -280,5 +280,5 @@
     </joint>
     <joint type="revolute" name="joint_5">
-      <origin xyz="1.28 0 0 " rpy="0 0 0"/>
+      <origin xyz="1.142 0 0 " rpy="0 0 0"/>
       <axis xyz="0 1 0"/>
       <parent link="link_4"/>

File: ros2srrc_robots/irb6640/urdf/irb6640_ros2control.xacro (robot description, xacro)
@@ -166,16 +166,18 @@
       </joint>
       <!-- CYLINDER&PISTON -->
-      <joint name="joint_cylinder">
-        <param name="mimic">joint_2</param>
-        <param name="multiplier">-0.35</param>
-        <state_interface name="position"/>
-        <state_interface name="velocity"/>
-      </joint>
-      <joint name="joint_piston">
-        <param name="mimic">joint_2</param>
-        <param name="multiplier">-1.35</param>
-        <state_interface name="position"/>
-        <state_interface name="velocity"/>
-      </joint>
+      <xacro:unless value="${bringup}">
+        <joint name="joint_cylinder">
+          <param name="mimic">joint_2</param>
+          <param name="multiplier">-0.35</param>
+          <state_interface name="position"/>
+          <state_interface name="velocity"/>
+        </joint>
+        <joint name="joint_piston">
+          <param name="mimic">joint_2</param>
+          <param name="multiplier">-1.35</param>
+          <state_interface name="position"/>
+          <state_interface name="velocity"/>
+        </joint>
+      </xacro:unless>
       <!-- END EFFECTOR -->
       <xacro:unless value="${bringup}">
