Commit message: Fix joint names in <transmission> for consistency.

File: ros2srrc_robots/iiwa/urdf/iiwa_transmission.xacro (robot description, xacro)
@@ -51,5 +51,5 @@
     <transmission name="iiwa_joint1_trans">
       <type>transmission_interface/SimpleTransmission</type>
-      <joint name="iiwa_joint1">
+      <joint name="joint_1">
         <hardwareInterface>hardware_interface/PositionJointInterface</hardwareInterface>
       </joint>
@@ -60,5 +60,5 @@
     <transmission name="iiwa_joint2_trans">
       <type>transmission_interface/SimpleTransmission</type>
-      <joint name="iiwa_joint2">
+      <joint name="joint_2">
         <hardwareInterface>hardware_interface/PositionJointInterface</hardwareInterface>
       </joint>
@@ -69,5 +69,5 @@
     <transmission name="iiwa_joint3_trans">
       <type>transmission_interface/SimpleTransmission</type>
-      <joint name="iiwa_joint3">
+      <joint name="joint_3">
         <hardwareInterface>hardware_interface/PositionJointInterface</hardwareInterface>
       </joint>
@@ -78,5 +78,5 @@
     <transmission name="iiwa_joint4_trans">
       <type>transmission_interface/SimpleTransmission</type>
-      <joint name="iiwa_joint4">
+      <joint name="joint_4">
         <hardwareInterface>hardware_interface/PositionJointInterface</hardwareInterface>
       </joint>
@@ -87,5 +87,5 @@
     <transmission name="iiwa_joint5_trans">
       <type>transmission_interface/SimpleTransmission</type>
-      <joint name="iiwa_joint5">
+      <joint name="joint_5">
         <hardwareInterface>hardware_interface/PositionJointInterface</hardwareInterface>
       </joint>
@@ -96,5 +96,5 @@
     <transmission name="iiwa_joint6_trans">
       <type>transmission_interface/SimpleTransmission</type>
-      <joint name="iiwa_joint6">
+      <joint name="joint_6">
         <hardwareInterface>hardware_interface/PositionJointInterface</hardwareInterface>
       </joint>
@@ -105,5 +105,5 @@
     <transmission name="iiwa_joint7_trans">
       <type>transmission_interface/SimpleTransmission</type>
-      <joint name="iiwa_joint7">
+      <joint name="joint_7">
         <hardwareInterface>hardware_interface/PositionJointInterface</hardwareInterface>
       </joint>

File: ros2srrc_robots/irb120/urdf/irb120_transmission.xacro (robot description, xacro)
@@ -51,5 +51,5 @@
     <transmission name="irb120_joint1_trans">
       <type>transmission_interface/SimpleTransmission</type>
-      <joint name="irb120_joint1">
+      <joint name="joint_1">
         <hardwareInterface>hardware_interface/PositionJointInterface</hardwareInterface>
       </joint>
@@ -60,5 +60,5 @@
     <transmission name="irb120_joint2_trans">
       <type>transmission_interface/SimpleTransmission</type>
-      <joint name="irb120_joint2">
+      <joint name="joint_2">
         <hardwareInterface>hardware_interface/PositionJointInterface</hardwareInterface>
       </joint>
@@ -69,5 +69,5 @@
     <transmission name="irb120_joint3_trans">
       <type>transmission_interface/SimpleTransmission</type>
-      <joint name="irb120_joint3">
+      <joint name="joint_3">
         <hardwareInterface>hardware_interface/PositionJointInterface</hardwareInterface>
       </joint>
@@ -78,5 +78,5 @@
     <transmission name="irb120_joint4_trans">
       <type>transmission_interface/SimpleTransmission</type>
-      <joint name="irb120_joint4">
+      <joint name="joint_4">
         <hardwareInterface>hardware_interface/PositionJointInterface</hardwareInterface>
       </joint>
@@ -87,5 +87,5 @@
     <transmission name="irb120_joint5_trans">
       <type>transmission_interface/SimpleTransmission</type>
-      <joint name="irb120_joint5">
+      <joint name="joint_5">
         <hardwareInterface>hardware_interface/PositionJointInterface</hardwareInterface>
       </joint>
@@ -96,5 +96,5 @@
     <transmission name="irb120_joint6_trans">
       <type>transmission_interface/SimpleTransmission</type>
-      <joint name="irb120_joint6">
+      <joint name="joint_6">
         <hardwareInterface>hardware_interface/PositionJointInterface</hardwareInterface>
       </joint>

File: ros2srrc_robots/irb1200/urdf/irb1200_transmission.xacro (robot description, xacro)
@@ -51,5 +51,5 @@
     <transmission name="irb1200_joint1_trans">
       <type>transmission_interface/SimpleTransmission</type>
-      <joint name="irb1200_joint1">
+      <joint name="joint_1">
         <hardwareInterface>hardware_interface/PositionJointInterface</hardwareInterface>
       </joint>
@@ -60,5 +60,5 @@
     <transmission name="irb1200_joint2_trans">
       <type>transmission_interface/SimpleTransmission</type>
-      <joint name="irb1200_joint2">
+      <joint name="joint_2">
         <hardwareInterface>hardware_interface/PositionJointInterface</hardwareInterface>
       </joint>
@@ -69,5 +69,5 @@
     <transmission name="irb1200_joint3_trans">
       <type>transmission_interface/SimpleTransmission</type>
-      <joint name="irb1200_joint3">
+      <joint name="joint_3">
         <hardwareInterface>hardware_interface/PositionJointInterface</hardwareInterface>
       </joint>
@@ -78,5 +78,5 @@
     <transmission name="irb1200_joint4_trans">
       <type>transmission_interface/SimpleTransmission</type>
-      <joint name="irb1200_joint4">
+      <joint name="joint_4">
         <hardwareInterface>hardware_interface/PositionJointInterface</hardwareInterface>
       </joint>
@@ -87,5 +87,5 @@
     <transmission name="irb1200_joint5_trans">
       <type>transmission_interface/SimpleTransmission</type>
-      <joint name="irb1200_joint5">
+      <joint name="joint_5">
         <hardwareInterface>hardware_interface/PositionJointInterface</hardwareInterface>
       </joint>
@@ -96,5 +96,5 @@
     <transmission name="irb1200_joint6_trans">
       <type>transmission_interface/SimpleTransmission</type>
-      <joint name="irb1200_joint6">
+      <joint name="joint_6">
         <hardwareInterface>hardware_interface/PositionJointInterface</hardwareInterface>
       </joint>
