Commit message: Migrate to GzFortress: KUKA LBR-IIWA robot.

File: ros2srrc_robots/iiwa/urdf/iiwa_ros2control.xacro (robot description, xacro)
@@ -52,5 +52,5 @@
     <!-- A. GAZEBO SIMULATION: -->
     <xacro:unless value="${bringup}">
-      <xacro:property name="name" value="GazeboSystem"/>
+      <xacro:property name="name" value="GazeboSimSystem"/>
     </xacro:unless>
     <!-- B. ROBOT BRINGUP: -->
@@ -63,5 +63,5 @@
       <xacro:unless value="${bringup}">
         <hardware>
-          <plugin>gazebo_ros2_control/GazeboSystem</plugin>
+          <plugin>gz_ros2_control/GazeboSimSystem</plugin>
         </hardware>
       </xacro:unless>
@@ -129,5 +129,5 @@
         </command_interface>
         <state_interface name="position">
-          <param name="initial_value">0.0</param>
+          <param name="initial_value">-1.5708</param>
         </state_interface>
         <state_interface name="velocity"/>
@@ -159,5 +159,5 @@
         </command_interface>
         <state_interface name="position">
-          <param name="initial_value">0.0</param>
+          <param name="initial_value">1.5708</param>
         </state_interface>
         <state_interface name="velocity"/>
@@ -174,5 +174,5 @@
         </command_interface>
         <state_interface name="position">
-          <param name="initial_value">0.0</param>
+          <param name="initial_value">1.5708</param>
         </state_interface>
         <state_interface name="velocity"/>
