Commit message: Update: iiwa robot (ready).

File: ros2srrc_robots/iiwa/urdf/iiwa_transmission.xacro (robot description, xacro)
@@ -48,56 +48,65 @@
 -->
 <robot xmlns:xacro="http://wiki.ros.org/xacro">
-  <xacro:macro name="irb120_transmission" params="">
-    <transmission name="irb120_joint1_trans">
+  <xacro:macro name="iiwa_transmission" params="">
+    <transmission name="iiwa_joint1_trans">
       <type>transmission_interface/SimpleTransmission</type>
-      <joint name="irb120_joint1">
+      <joint name="iiwa_joint1">
         <hardwareInterface>hardware_interface/PositionJointInterface</hardwareInterface>
       </joint>
-      <actuator name="irb120_joint1_motor">
+      <actuator name="iiwa_joint1_motor">
         <mechanicalReduction>1</mechanicalReduction>
       </actuator>
     </transmission>
-    <transmission name="irb120_joint2_trans">
+    <transmission name="iiwa_joint2_trans">
       <type>transmission_interface/SimpleTransmission</type>
-      <joint name="irb120_joint2">
+      <joint name="iiwa_joint2">
         <hardwareInterface>hardware_interface/PositionJointInterface</hardwareInterface>
       </joint>
-      <actuator name="irb120_joint2_motor">
+      <actuator name="iiwa_joint2_motor">
         <mechanicalReduction>1</mechanicalReduction>
       </actuator>
     </transmission>
-    <transmission name="irb120_joint3_trans">
+    <transmission name="iiwa_joint3_trans">
       <type>transmission_interface/SimpleTransmission</type>
-      <joint name="irb120_joint3">
+      <joint name="iiwa_joint3">
         <hardwareInterface>hardware_interface/PositionJointInterface</hardwareInterface>
       </joint>
-      <actuator name="irb120_joint3_motor">
+      <actuator name="iiwa_joint3_motor">
         <mechanicalReduction>1</mechanicalReduction>
       </actuator>
     </transmission>
-    <transmission name="irb120_joint4_trans">
+    <transmission name="iiwa_joint4_trans">
       <type>transmission_interface/SimpleTransmission</type>
-      <joint name="irb120_joint4">
+      <joint name="iiwa_joint4">
         <hardwareInterface>hardware_interface/PositionJointInterface</hardwareInterface>
       </joint>
-      <actuator name="irb120_joint4_motor">
+      <actuator name="iiwa_joint4_motor">
         <mechanicalReduction>1</mechanicalReduction>
       </actuator>
     </transmission>
-    <transmission name="irb120_joint5_trans">
+    <transmission name="iiwa_joint5_trans">
       <type>transmission_interface/SimpleTransmission</type>
-      <joint name="irb120_joint5">
+      <joint name="iiwa_joint5">
         <hardwareInterface>hardware_interface/PositionJointInterface</hardwareInterface>
       </joint>
-      <actuator name="irb120_joint5_motor">
+      <actuator name="iiwa_joint5_motor">
         <mechanicalReduction>1</mechanicalReduction>
       </actuator>
     </transmission>
-    <transmission name="irb120_joint6_trans">
+    <transmission name="iiwa_joint6_trans">
       <type>transmission_interface/SimpleTransmission</type>
-      <joint name="irb120_joint6">
+      <joint name="iiwa_joint6">
         <hardwareInterface>hardware_interface/PositionJointInterface</hardwareInterface>
       </joint>
-      <actuator name="irb120_joint6_motor">
+      <actuator name="iiwa_joint6_motor">
+        <mechanicalReduction>1</mechanicalReduction>
+      </actuator>
+    </transmission>
+    <transmission name="iiwa_joint7_trans">
+      <type>transmission_interface/SimpleTransmission</type>
+      <joint name="iiwa_joint7">
+        <hardwareInterface>hardware_interface/PositionJointInterface</hardwareInterface>
+      </joint>
+      <actuator name="iiwa_joint7_motor">
         <mechanicalReduction>1</mechanicalReduction>
       </actuator>

Commit message: Fix: Damping values in robot's urdf files.

File: ros2srrc_robots/iiwa/urdf/iiwa_macro.urdf.xacro (robot description, xacro)
@@ -251,4 +251,5 @@
       <axis xyz="0 0 1"/>
       <limit effort="320" lower="-2.9668" upper="2.9668" velocity="1.4834"/>
+      <dynamics damping="1.0" friction="0.0"/>
     </joint>
     <joint name="joint_2" type="revolute">
@@ -258,4 +259,5 @@
       <axis xyz="0 1 0"/>
       <limit effort="320" lower="-2.0942" upper="2.0942" velocity="1.4834"/>
+      <dynamics damping="1.0" friction="0.0"/>
     </joint>
     <joint name="joint_3" type="revolute">
@@ -265,4 +267,5 @@
       <axis xyz="0 0 1"/>
       <limit effort="176" lower="-2.9668" upper="2.9668" velocity="1.7452"/>
+      <dynamics damping="1.0" friction="0.0"/>
     </joint>
     <joint name="joint_4" type="revolute">
@@ -272,4 +275,5 @@
       <axis xyz="0 -1 0"/>
       <limit effort="176" lower="-2.0942" upper="2.0942" velocity="1.3089"/>
+      <dynamics damping="10.0" friction="1.0"/> <!-- High values of damping + friction were added, to avoid bac joint behaviour in GzFortress. -->
     </joint>
     <joint name="joint_5" type="revolute">
@@ -279,4 +283,5 @@
       <axis xyz="0 0 1"/>
       <limit effort="110" lower="-2.9668" upper="2.9668" velocity="2.2688"/>
+      <dynamics damping="1.0" friction="0.0"/>
     </joint>
     <joint name="joint_6" type="revolute">
@@ -286,4 +291,5 @@
       <axis xyz="0 1 0"/>
       <limit effort="40" lower="-2.0942" upper="2.0942" velocity="2.356"/>
+      <dynamics damping="1.0" friction="0.0"/>
     </joint>
     <joint name="joint_7" type="revolute">
@@ -293,4 +299,5 @@
       <axis xyz="0 0 1"/>
       <limit effort="40" lower="-3.0541" upper="3.0541" velocity="2.356"/>
+      <dynamics damping="1.0" friction="0.0"/>
     </joint>
     <!-- end of joint list -->

File: ros2srrc_robots/irb120/urdf/irb120_macro.urdf.xacro (robot description, xacro)
@@ -223,5 +223,5 @@
       <limit effort="1000" lower="-2.87979" upper="2.87979" velocity="4.36332"/>
       <axis xyz="0 0 1"/>
-      <dynamics damping="0.0" friction="0.0"/>
+      <dynamics damping="1.0" friction="0.0"/>
     </joint>
     <!-- joint_2 -->
@@ -232,5 +232,5 @@
       <limit effort="1000" lower="-1.91986" upper="1.91986" velocity="4.36332"/>
       <axis xyz="0 1 0"/>
-      <dynamics damping="0.0" friction="0.0"/>
+      <dynamics damping="0.5" friction="0.0"/>
     </joint>
     <!-- joint_3 -->
@@ -241,5 +241,5 @@
       <limit effort="1000" lower="-1.91986" upper="1.22173" velocity="4.36332"/>
       <axis xyz="0 1 0"/>
-      <dynamics damping="0.0" friction="0.0"/>
+      <dynamics damping="0.3" friction="0.0"/>
     </joint>
     <!-- joint_4 -->
@@ -250,5 +250,5 @@
       <limit effort="1000" lower="-2.79253" upper="2.79253" velocity="5.58505"/>
       <axis xyz="1 0 0"/>
-      <dynamics damping="0.0" friction="0.0"/>
+      <dynamics damping="0.1" friction="0.0"/>
     </joint>
     <!-- joint_5 -->
@@ -259,5 +259,5 @@
       <limit effort="1000" lower="-2.094395" upper="2.094395" velocity="5.58505"/>
       <axis xyz="0 1 0"/>
-      <dynamics damping="0.0" friction="0.0"/>
+      <dynamics damping="0.05" friction="0.0"/>
     </joint>
     <!-- joint_6 -->
@@ -268,5 +268,5 @@
       <limit effort="1000" lower="-6.98132" upper="6.98132" velocity="7.33038"/>
       <axis xyz="1 0 0"/>
-      <dynamics damping="0.0" friction="0.0"/>
+      <dynamics damping="0.01" friction="0.0"/>
     </joint>
     <!-- end of joint list -->

File: ros2srrc_robots/irb1200/urdf/irb1200_macro.urdf.xacro (robot description, xacro)
@@ -216,4 +216,5 @@
       <child link="link_1"/>
       <limit effort="1000" lower="-2.967" upper="2.967" velocity="5.027"/>
+      <dynamics damping="1.0" friction="0.0"/>
     </joint>
     <!-- joint_2 -->
@@ -224,4 +225,5 @@
       <child link="link_2"/>
       <limit effort="1000" lower="-1.745" upper="2.269" velocity="4.189"/>
+      <dynamics damping="0.5" friction="0.0"/>
     </joint>
     <!-- joint_3 -->
@@ -232,4 +234,5 @@
       <child link="link_3"/>
       <limit effort="1000" lower="-3.491" upper="1.222" velocity="5.236"/>
+      <dynamics damping="0.3" friction="0.0"/>
     </joint>
     <!-- joint_4 -->
@@ -240,4 +243,5 @@
       <child link="link_4"/>
       <limit effort="1000" lower="-4.712" upper="4.712" velocity="6.981"/>
+      <dynamics damping="0.1" friction="0.0"/>
     </joint>
     <!-- joint_5 -->
@@ -248,4 +252,5 @@
       <child link="link_5"/>
       <limit effort="1000" lower="-2.269" upper="2.269" velocity="7.069"/>
+      <dynamics damping="0.05" friction="0.0"/>
     </joint>
     <!-- joint_6 -->
@@ -256,4 +261,5 @@
       <child link="link_6"/>
       <limit effort="1000" lower="-6.98132" upper="6.98132" velocity="10.472"/>
+      <dynamics damping="0.05" friction="0.0"/>
     </joint>
     <!-- end of joint list -->
