Commit message: Migrate from Gazebo Classic to Gz Fortress: ABB IRB-120 robot.

File: packages/ros2srrc_irb120/urdf/irb120.urdf.xacro (robot description, xacro)
@@ -49,6 +49,5 @@
   <xacro:unless value="${bringup}">
     <gazebo>
-      <plugin filename="libgazebo_ros2_control.so" name="gazebo_ros2_control">
-        <robot_sim_type>gazebo_ros2_control/GazeboSystem</robot_sim_type>
+      <plugin filename="gz_ros2_control-system" name="gz_ros2_control::GazeboSimROS2ControlPlugin">
         <!-- IRB120 Controller -->
         <parameters>$(find ros2srrc_robots)/irb120/config/controller.yaml</parameters>

File: ros2srrc_robots/irb120/urdf/irb120_macro.urdf.xacro (robot description, xacro)
@@ -79,5 +79,4 @@
           <mesh filename="file://$(find ros2srrc_robots)/irb120/meshes/visual/base_link.dae"/>
         </geometry>
-        <xacro:material_abb_orange />
       </visual>
       <collision>
@@ -101,5 +100,4 @@
           <mesh filename="file://$(find ros2srrc_robots)/irb120/meshes/visual/link_1.dae"/>
         </geometry>
-        <xacro:material_abb_orange />
       </visual>
       <collision>
@@ -123,5 +121,4 @@
           <mesh filename="file://$(find ros2srrc_robots)/irb120/meshes/visual/link_2.dae"/>
         </geometry>
-        <xacro:material_abb_orange />
       </visual>
       <collision>
@@ -145,5 +142,4 @@
           <mesh filename="file://$(find ros2srrc_robots)/irb120/meshes/visual/link_3.dae"/>
         </geometry>
-        <xacro:material_abb_orange />
       </visual>
       <collision>
@@ -167,5 +163,4 @@
           <mesh filename="file://$(find ros2srrc_robots)/irb120/meshes/visual/link_4.dae"/>
         </geometry>
-        <xacro:material_abb_orange />
       </visual>
       <collision>
@@ -189,5 +184,4 @@
           <mesh filename="file://$(find ros2srrc_robots)/irb120/meshes/visual/link_5.dae"/>
         </geometry>
-        <xacro:material_abb_orange />
       </visual>
       <collision>
@@ -211,5 +205,4 @@
           <mesh filename="file://$(find ros2srrc_robots)/irb120/meshes/visual/link_6.dae"/>
         </geometry>
-        <xacro:material_abb_black />
       </visual>
       <collision>

File: ros2srrc_robots/irb120/urdf/irb120_ros2control.xacro (robot description, xacro)
@@ -52,5 +52,5 @@
     <!-- A. GAZEBO SIMULATION: -->
     <xacro:unless value="${bringup}">
-      <xacro:property name="name" value="GazeboSystem"/>
+      <xacro:property name="name" value="GazeboSimSystem"/>
     </xacro:unless>
     <!-- B. ROBOT BRINGUP: -->
@@ -63,5 +63,5 @@
       <xacro:unless value="${bringup}">
         <hardware>
-          <plugin>gazebo_ros2_control/GazeboSystem</plugin>
+          <plugin>gz_ros2_control/GazeboSimSystem</plugin>
         </hardware>
       </xacro:unless>
