Commit message: Migrate to GzFortress: Schunk EGP 64 gripper.

File: packages/ros2srrc_irb120/urdf/irb120_egp64.urdf.xacro (robot description, xacro)
@@ -55,6 +55,5 @@
   <xacro:unless value="${bringup}">
     <gazebo>
-      <plugin filename="libgazebo_ros2_control.so" name="gazebo_ros2_control">
-        <robot_sim_type>gazebo_ros2_control/GazeboSystem</robot_sim_type>
+      <plugin filename="gz_ros2_control-system" name="gz_ros2_control::GazeboSimROS2ControlPlugin">
         <!-- IRB120 Controller -->
         <parameters>$(find ros2srrc_robots)/irb120/config/controller.yaml</parameters>

File: packages/ros2srrc_irb120/urdf/irb120_egp64v2.urdf.xacro (robot description, xacro)
@@ -55,6 +55,5 @@
   <xacro:unless value="${bringup}">
     <gazebo>
-      <plugin filename="libgazebo_ros2_control.so" name="gazebo_ros2_control">
-        <robot_sim_type>gazebo_ros2_control/GazeboSystem</robot_sim_type>
+      <plugin filename="gz_ros2_control-system" name="gz_ros2_control::GazeboSimROS2ControlPlugin">
         <!-- IRB120 Controller -->
         <parameters>$(find ros2srrc_robots)/irb120/config/controller.yaml</parameters>

File: packages/ros2srrc_irb120/urdf/irb120_ls_vgr.urdf.xacro (robot description, xacro)
@@ -55,6 +55,5 @@
   <xacro:unless value="${bringup}">
     <gazebo>
-      <plugin filename="libgazebo_ros2_control.so" name="gazebo_ros2_control">
-        <robot_sim_type>gazebo_ros2_control/GazeboSystem</robot_sim_type>
+      <plugin filename="gz_ros2_control-system" name="gz_ros2_control::GazeboSimROS2ControlPlugin">
         <!-- IRB120 Controller -->
         <parameters>$(find ros2srrc_robots)/irb120/config/controller.yaml</parameters>

File: ros2srrc_endeffectors/egp64/urdf/egp64_macro.urdf.xacro (robot description, xacro)
@@ -76,6 +76,6 @@
           <mesh filename="file://$(find ros2srrc_endeffectors)/egp64/meshes/egp64_BaseNoAdapter.dae" />
         </geometry>
-        <material name="blue">
-          <color rgba="0 0 1 1"/>
+        <material name="silver">
+          <color rgba="0.8 0.8 0.8 1"/>
         </material>
       </visual>
@@ -84,5 +84,4 @@
           <mesh filename="file://$(find ros2srrc_endeffectors)/egp64/meshes/egp64_BaseNoAdapter.dae" />
         </geometry>
-        <material name="blue"/>
       </collision>
     </link>

File: ros2srrc_endeffectors/egp64/urdf/egp64v2_macro.urdf.xacro (robot description, xacro)
@@ -76,6 +76,6 @@
           <mesh filename="file://$(find ros2srrc_endeffectors)/egp64/meshes/egp64_BaseNoAdapter.dae" />
         </geometry>
-        <material name="blue">
-          <color rgba="0 0 1 1"/>
+        <material name="silver">
+          <color rgba="0.8 0.8 0.8 1"/>
         </material>
       </visual>
@@ -84,5 +84,4 @@
           <mesh filename="file://$(find ros2srrc_endeffectors)/egp64/meshes/egp64_BaseNoAdapter.dae" />
         </geometry>
-        <material name="blue"/>
       </collision>
     </link>

File: ros2srrc_endeffectors/egp64/urdf/egp64v3_macro.urdf.xacro (robot description, xacro)
@@ -76,6 +76,6 @@
           <mesh filename="file://$(find ros2srrc_endeffectors)/egp64/meshes/egp64_BaseNoAdapter.dae" />
         </geometry>
-        <material name="blue">
-          <color rgba="0 0 1 1"/>
+        <material name="silver">
+          <color rgba="0.8 0.8 0.8 1"/>
         </material>
       </visual>
@@ -84,5 +84,4 @@
           <mesh filename="file://$(find ros2srrc_endeffectors)/egp64/meshes/egp64_BaseNoAdapter.dae" />
         </geometry>
-        <material name="blue"/>
       </collision>
     </link>
