Commit message: Add colour to LS for Gz Fortress.

File: ros2srrc_endeffectors/ls_vgr/urdf/ls_vgr_macro.urdf.xacro (robot description, xacro)
@@ -48,4 +48,7 @@
           <mesh filename="file://$(find ros2srrc_endeffectors)/ls_vgr/meshes/ls_vgr.dae"/>
         </geometry>
+        <material name="silver">
+          <color rgba="0.8 0.8 0.8 1"/>
+        </material>
       </visual>
     </link>
