Commit message: Migrate to GzFortress: Robotiq 2f85 gripper.

File: ros2srrc_endeffectors/robotiq_2f85/urdf/robotiq_2f85_macro.urdf.xacro (robot description, xacro)
@@ -116,6 +116,6 @@
       <axis xyz="0 0 1"/>
       <origin rpy="${pi} 0.0 0.0" xyz="0.05490451627 0.03060114443 0.0"/>
-      <limit lower="-0.05" upper="0.80285" velocity="0.5" effort="1000"/>
-      <dynamics damping="0.0" friction="0.0"/>
+      <limit lower="-0.0001" upper="0.8001" velocity="1.0" effort="1000"/>
+      <dynamics damping="0.2" friction="0.05"/>
     </joint>
     <!-- Robotiq: right_knuckle -->
@@ -139,11 +139,11 @@
       </inertial>
     </link>
-    <joint name="robotiq_85_right_knuckle_joint" type="continuous">
+    <joint name="robotiq_85_right_knuckle_joint" type="revolute">
       <parent link="robotiq_85_base_link"/>
       <child link="robotiq_85_right_knuckle_link"/>
       <axis xyz="0 0 1"/>
       <origin rpy="0.0 0.0 0.0" xyz="0.05490451627 -0.03060114443 0.0"/>
-      <limit lower="-0.05" upper="0.80285" velocity="0.5" effort="1000"/>
-      <dynamics damping="0.0" friction="0.0"/>
+      <limit lower="-0.0001" upper="0.8001" velocity="1.0" effort="1000"/>
+      <dynamics damping="0.2" friction="0.05"/>
     </joint>
     <!-- Robotiq: left_finger -->
@@ -171,5 +171,4 @@
       <child link="robotiq_85_left_finger_link"/>
       <origin xyz="-0.00408552455 -0.03148604435 0.0" rpy="0 0 0" />
-      <dynamics damping="0.0" friction="0.0"/>
     </joint>
     <!-- Robotiq: right_finger -->
@@ -197,5 +196,4 @@
       <child link="robotiq_85_right_finger_link"/>
       <origin xyz="-0.00408552455 -0.03148604435 0.0" rpy="0 0 0" />
-      <dynamics damping="0.0" friction="0.0"/>
     </joint>
     <!-- Robotiq: left_inner_knuckle -->
@@ -219,11 +217,11 @@
       </inertial>
     </link>
-    <joint name="robotiq_85_left_inner_knuckle_joint" type="continuous">
+    <joint name="robotiq_85_left_inner_knuckle_joint" type="revolute">
       <parent link="robotiq_85_base_link"/>
       <child link="robotiq_85_left_inner_knuckle_link"/>
       <axis xyz="0 0 1"/>
       <origin xyz="0.06142 0.0127 0" rpy="${pi} 0.0 0.0" />
-      <limit lower="-0.05" upper="0.80285" velocity="0.5" effort="1000"/>
-      <dynamics damping="0.0" friction="0.0"/>
+      <limit lower="-0.0001" upper="0.8001" velocity="1.0" effort="1000"/>
+      <dynamics damping="0.2" friction="0.05"/>
     </joint>
     <!-- Robotiq: right_inner_knuckle -->
@@ -247,11 +245,11 @@
       </inertial>
     </link>
-    <joint name="robotiq_85_right_inner_knuckle_joint" type="continuous">
+    <joint name="robotiq_85_right_inner_knuckle_joint" type="revolute">
       <parent link="robotiq_85_base_link"/>
       <child link="robotiq_85_right_inner_knuckle_link"/>
       <axis xyz="0 0 1"/>
       <origin xyz="0.06142 -0.0127 0" rpy="0 0 0"/>
-      <limit lower="-0.05" upper="0.80285" velocity="0.5" effort="1000"/>
-      <dynamics damping="0.0" friction="0.0"/>
+      <limit lower="-0.0001" upper="0.8001" velocity="1.0" effort="1000"/>
+      <dynamics damping="0.2" friction="0.05"/>
     </joint>
     <!-- Robotiq: left_finger_tip -->
@@ -275,11 +273,11 @@
       </inertial>
     </link>
-    <joint name="robotiq_85_left_finger_tip_joint" type="continuous">
+    <joint name="robotiq_85_left_finger_tip_joint" type="revolute">
       <parent link="robotiq_85_left_inner_knuckle_link"/>
       <child link="robotiq_85_left_finger_tip_link"/>
       <axis xyz="0 0 1"/>
       <origin xyz="0.04303959807 -0.03759940821 0.0" rpy="0.0 0.0 0.0"/>
-      <limit lower="-0.80285" upper="0.05" velocity="0.5" effort="1000"/>
-      <dynamics damping="0.0" friction="0.0"/>
+      <limit lower="-0.8001" upper="0.0001" velocity="1.0" effort="1000"/>
+      <dynamics damping="0.2" friction="0.05"/>
     </joint>
     <!-- Robotiq: right_finger_tip -->
@@ -303,11 +301,11 @@
       </inertial>
     </link>
-    <joint name="robotiq_85_right_finger_tip_joint" type="continuous">
+    <joint name="robotiq_85_right_finger_tip_joint" type="revolute">
       <parent link="robotiq_85_right_inner_knuckle_link"/>
       <child link="robotiq_85_right_finger_tip_link"/>
       <axis xyz="0 0 1"/>
       <origin rpy="0.0 0.0 0.0" xyz="0.04303959807 -0.03759940821  0.0"/>
-      <limit lower="-0.80285" upper="0.05" velocity="0.5" effort="1000"/>
-      <dynamics damping="0.0" friction="0.0"/>
+      <limit lower="-0.8001" upper="0.0001" velocity="1.0" effort="1000"/>
+      <dynamics damping="0.2" friction="0.05"/>
     </joint>
     <!-- SMALL CUBE FOR GRIPPER PLUGIN -->

File: ros2srrc_endeffectors/robotiq_2f85/urdf/robotiq_2f85_ros2control.xacro (robot description, xacro)
@@ -32,10 +32,6 @@
     <joint name="robotiq_85_left_knuckle_joint">
       <command_interface name="position">
-        <param name="min">-0.05</param>
-        <param name="max">0.80285</param>
-      </command_interface>
-      <command_interface name="velocity">
-        <param name="min">0.5</param>
-        <param name="max">0.5</param>
+        <param name="min">-0.0001</param>
+        <param name="max">0.8001</param>
       </command_interface>
       <state_interface name="position">
@@ -47,10 +43,6 @@
     <joint name="robotiq_85_right_knuckle_joint">
       <command_interface name="position">
-        <param name="min">-0.05</param>
-        <param name="max">0.80285</param>
-      </command_interface>
-      <command_interface name="velocity">
-        <param name="min">0.5</param>
-        <param name="max">0.5</param>
+        <param name="min">-0.0001</param>
+        <param name="max">0.8001</param>
       </command_interface>
       <state_interface name="position">
@@ -62,10 +54,6 @@
     <joint name="robotiq_85_left_inner_knuckle_joint">
       <command_interface name="position">
-        <param name="min">-0.05</param>
-        <param name="max">0.80285</param>
-      </command_interface>
-      <command_interface name="velocity">
-        <param name="min">0.5</param>
-        <param name="max">0.5</param>
+        <param name="min">-0.0001</param>
+        <param name="max">0.8001</param>
       </command_interface>
       <state_interface name="position">
@@ -77,10 +65,6 @@
     <joint name="robotiq_85_right_inner_knuckle_joint">
       <command_interface name="position">
-        <param name="min">-0.05</param>
-        <param name="max">0.80285</param>
-      </command_interface>
-      <command_interface name="velocity">
-        <param name="min">0.5</param>
-        <param name="max">0.5</param>
+        <param name="min">-0.0001</param>
+        <param name="max">0.8001</param>
       </command_interface>
       <state_interface name="position">
@@ -92,10 +76,6 @@
     <joint name="robotiq_85_left_finger_tip_joint">
       <command_interface name="position">
-        <param name="min">-0.80285</param>
-        <param name="max">0.05</param>
-      </command_interface>
-      <command_interface name="velocity">
-        <param name="min">0.5</param>
-        <param name="max">0.5</param>
+        <param name="min">-0.8001</param>
+        <param name="max">0.0001</param>
       </command_interface>
       <state_interface name="position">
@@ -107,10 +87,6 @@
     <joint name="robotiq_85_right_finger_tip_joint">
       <command_interface name="position">
-        <param name="min">-0.80285</param>
-        <param name="max">0.05</param>
-      </command_interface>
-      <command_interface name="velocity">
-        <param name="min">0.5</param>
-        <param name="max">0.5</param>
+        <param name="min">-0.8001</param>
+        <param name="max">0.0001</param>
       </command_interface>
       <state_interface name="position">
