Commit message: Remove Cranfield Uni's cable management bracket (no longer needed).

File: ros2srrc_endeffectors/robotiq_hande/urdf/robotiq_hande_macro.urdf.xacro (robot description, xacro)
@@ -37,5 +37,5 @@
     </xacro:unless>
     <!-- ***** Robotiq HandE GRIPPER .urdf SERIAL CHAIN ***** -->
-    <!-- Robotiq: bracket -->
+    <!-- Robotiq: bracket
     <link name="robotiq_bracket">
       <visual>
@@ -60,5 +60,5 @@
       <parent link="${parent_link}"/>
       <child link="robotiq_bracket"/>
-    </joint>
+    </joint> -->
     <!-- Robotiq: coupler -->
     <link name="robotiq_coupler">
@@ -81,6 +81,6 @@
     </link>
     <joint name="robotiq_coupler_joint" type="fixed">
-      <origin xyz="0 0 0" rpy="0 0 0" />
-      <parent link="robotiq_bracket"/>
+      <origin xyz="0 0 -0.008" rpy="0 0 0" />
+      <parent link="${parent_link}"/>
       <child link="robotiq_coupler"/>
     </joint>

File: ros2srrc_endeffectors/robotiq_hande/urdf/robotiq_handev2_macro.urdf.xacro (robot description, xacro)
@@ -37,5 +37,5 @@
     </xacro:unless>
     <!-- ***** Robotiq HandE GRIPPER .urdf SERIAL CHAIN ***** -->
-    <!-- Robotiq: bracket -->
+    <!-- Robotiq: bracket
     <link name="robotiq_bracket">
       <visual>
@@ -60,5 +60,5 @@
       <parent link="${parent_link}"/>
       <child link="robotiq_bracket"/>
-    </joint>
+    </joint> -->
     <!-- Robotiq: coupler -->
     <link name="robotiq_coupler">
@@ -81,6 +81,6 @@
     </link>
     <joint name="robotiq_coupler_joint" type="fixed">
-      <origin xyz="0 0 0" rpy="0 0 0" />
-      <parent link="robotiq_bracket"/>
+      <origin xyz="0 0 -0.008" rpy="0 0 0" />
+      <parent link="${parent_link}"/>
       <child link="robotiq_coupler"/>
     </joint>

Commit message: Fix: Robotiq HandE gripper movement limits.

File: ros2srrc_endeffectors/robotiq_hande/urdf/robotiq_hande_macro.urdf.xacro (robot description, xacro)
@@ -147,5 +147,5 @@
       <child link="robotiq_hande_left_finger"/>
       <axis xyz="-1 0 0"/>
-      <limit effort="130" lower="-0.05" upper="0.025" velocity="0.15"/>
+      <limit effort="130" lower="-0.0001" upper="0.025" velocity="0.15"/>
     </joint>
     <!-- Robotiq: right finger -->
@@ -177,5 +177,5 @@
       <child link="robotiq_hande_right_finger"/>
       <axis xyz="1 0 0"/>
-      <limit effort="130" lower="-0.05" upper="0.025" velocity="0.15"/>
+      <limit effort="130" lower="-0.0001" upper="0.025" velocity="0.15"/>
     </joint>
     <!-- SMALL CUBE FOR GRIPPER PLUGIN -->

Commit message: Fix HandE gripper's limits (urdf).

File: ros2srrc_endeffectors/robotiq_hande/urdf/robotiq_hande_macro.urdf.xacro (robot description, xacro)
@@ -147,5 +147,6 @@
       <child link="robotiq_hande_left_finger"/>
       <axis xyz="-1 0 0"/>
-      <limit effort="130" lower="-0.0001" upper="0.025" velocity="0.15"/>
+      <limit effort="130" lower="-0.0001" upper="0.0251" velocity="0.15"/>
+      <dynamics damping="0.2" friction="0.05"/>
     </joint>
     <!-- Robotiq: right finger -->
@@ -177,5 +178,6 @@
       <child link="robotiq_hande_right_finger"/>
       <axis xyz="1 0 0"/>
-      <limit effort="130" lower="-0.0001" upper="0.025" velocity="0.15"/>
+      <limit effort="130" lower="-0.0001" upper="0.0251" velocity="0.15"/>
+      <dynamics damping="0.2" friction="0.05"/>
     </joint>
     <!-- SMALL CUBE FOR GRIPPER PLUGIN -->

File: ros2srrc_endeffectors/robotiq_hande/urdf/robotiq_hande_ros2control.xacro (robot description, xacro)
@@ -32,6 +32,6 @@
     <joint name="robotiq_hande_left_finger_joint">
       <command_interface name="position">
-        <param name="min">-0.05</param>
-        <param name="max">0.025</param>
+        <param name="min">-0.0001</param>
+        <param name="max">0.0251</param>
       </command_interface>
       <command_interface name="velocity">
@@ -47,6 +47,6 @@
     <joint name="robotiq_hande_right_finger_joint">
       <command_interface name="position">
-        <param name="min">-0.05</param>
-        <param name="max">0.025</param>
+        <param name="min">-0.0001</param>
+        <param name="max">0.0251</param>
       </command_interface>
       <command_interface name="velocity">

File: ros2srrc_endeffectors/robotiq_hande/urdf/robotiq_handev2_macro.urdf.xacro (robot description, xacro)
@@ -142,5 +142,6 @@
       <child link="robotiq_hande_left_finger"/>
       <axis xyz="-1 0 0"/>
-      <limit effort="130" lower="-0.05" upper="0.025" velocity="0.15"/>
+      <limit effort="130" lower="-0.0001" upper="0.0251" velocity="0.15"/>
+      <dynamics damping="0.2" friction="0.05"/>
     </joint>
     <!-- Robotiq: right finger -->
@@ -172,5 +173,6 @@
       <child link="robotiq_hande_right_finger"/>
       <axis xyz="1 0 0"/>
-      <limit effort="130" lower="-0.05" upper="0.025" velocity="0.15"/>
+      <limit effort="130" lower="-0.0001" upper="0.0251" velocity="0.15"/>
+      <dynamics damping="0.2" friction="0.05"/>
     </joint>
     <!-- SMALL CUBE FOR GRIPPER PLUGIN -->
