Commit message: Migrate to GzFortress: ABB IRB1200 robot.

File: ros2srrc_robots/irb1200/urdf/irb1200_macro.urdf.xacro (robot description, xacro)
@@ -85,5 +85,4 @@
           <mesh filename="file://$(find ros2srrc_robots)/irb1200/meshes/visual/base_link.dae"/>
         </geometry>
-        <xacro:material_abb_yellow />
       </visual>
     </link>
@@ -106,5 +105,4 @@
           <mesh filename="file://$(find ros2srrc_robots)/irb1200/meshes/visual/link_1.dae"/>
         </geometry>
-        <xacro:material_abb_yellow />
       </visual>
     </link>
@@ -127,5 +125,4 @@
           <mesh filename="file://$(find ros2srrc_robots)/irb1200/meshes/visual/link_2.dae"/>
         </geometry>
-        <xacro:material_abb_yellow />
       </visual>
     </link>
@@ -148,5 +145,4 @@
           <mesh filename="file://$(find ros2srrc_robots)/irb1200/meshes/visual/link_3.dae"/>
         </geometry>
-        <xacro:material_abb_yellow />
       </visual>
     </link>
@@ -169,5 +165,4 @@
           <mesh filename="file://$(find ros2srrc_robots)/irb1200/meshes/visual/link_4.dae"/>
         </geometry>
-        <xacro:material_abb_yellow />
       </visual>
     </link>
@@ -190,5 +185,4 @@
           <mesh filename="file://$(find ros2srrc_robots)/irb1200/meshes/visual/link_5.dae"/>
         </geometry>
-        <xacro:material_abb_yellow />
       </visual>
     </link>
@@ -211,5 +205,4 @@
           <mesh filename="file://$(find ros2srrc_robots)/irb1200/meshes/visual/link_6.dae"/>
         </geometry>
-        <xacro:material_abb_yellow />
       </visual>
     </link>
@@ -223,5 +216,4 @@
       <child link="link_1"/>
       <limit effort="1000" lower="-2.967" upper="2.967" velocity="5.027"/>
-      <dynamics damping="50.0" friction="1.0"/>
     </joint>
     <!-- joint_2 -->
@@ -232,5 +224,4 @@
       <child link="link_2"/>
       <limit effort="1000" lower="-1.745" upper="2.269" velocity="4.189"/>
-      <dynamics damping="50.0" friction="1.0"/>
     </joint>
     <!-- joint_3 -->
@@ -241,5 +232,4 @@
       <child link="link_3"/>
       <limit effort="1000" lower="-3.491" upper="1.222" velocity="5.236"/>
-      <dynamics damping="10.0" friction="1.0"/>
     </joint>
     <!-- joint_4 -->
@@ -250,5 +240,4 @@
       <child link="link_4"/>
       <limit effort="1000" lower="-4.712" upper="4.712" velocity="6.981"/>
-      <dynamics damping="5.0" friction="1.0"/>
     </joint>
     <!-- joint_5 -->
@@ -259,5 +248,4 @@
       <child link="link_5"/>
       <limit effort="1000" lower="-2.269" upper="2.269" velocity="7.069"/>
-      <dynamics damping="2.0" friction="1.0"/>
     </joint>
     <!-- joint_6 -->
@@ -268,5 +256,4 @@
       <child link="link_6"/>
       <limit effort="1000" lower="-6.98132" upper="6.98132" velocity="10.472"/>
-      <dynamics damping="1.0" friction="1.0"/>
     </joint>
     <!-- end of joint list -->

File: ros2srrc_robots/irb1200/urdf/irb1200_ros2control.xacro (robot description, xacro)
@@ -52,5 +52,5 @@
     <!-- A. GAZEBO SIMULATION: -->
     <xacro:unless value="${bringup}">
-      <xacro:property name="name" value="GazeboSystem"/>
+      <xacro:property name="name" value="GazeboSimSystem"/>
     </xacro:unless>
     <!-- B. ROBOT BRINGUP: -->
@@ -63,5 +63,5 @@
       <xacro:unless value="${bringup}">
         <hardware>
-          <plugin>gazebo_ros2_control/GazeboSystem</plugin>
+          <plugin>gz_ros2_control/GazeboSimSystem</plugin>
         </hardware>
       </xacro:unless>
