Commit message: Migrate to GzFortress: UR3 Robot.

File: ros2srrc_robots/ur3/urdf/ur3_macro.urdf.xacro (robot description, xacro)
@@ -86,7 +86,4 @@
           <mesh filename="file://$(find ros2srrc_robots)/ur3/meshes/visual/base.dae"/>
         </geometry>
-        <material name="LightGrey">
-          <color rgba="0.7 0.7 0.7 1.0"/>
-        </material>
       </visual>
       <collision>
@@ -106,7 +103,4 @@
           <mesh filename="file://$(find ros2srrc_robots)/ur3/meshes/visual/shoulder.dae"/>
         </geometry>
-        <material name="LightGrey">
-          <color rgba="0.7 0.7 0.7 1.0"/>
-        </material>
       </visual>
       <collision>
@@ -126,7 +120,4 @@
           <mesh filename="file://$(find ros2srrc_robots)/ur3/meshes/visual/upperarm.dae"/>
         </geometry>
-        <material name="LightGrey">
-          <color rgba="0.7 0.7 0.7 1.0"/>
-        </material>
       </visual>
       <collision>
@@ -146,7 +137,4 @@
           <mesh filename="file://$(find ros2srrc_robots)/ur3/meshes/visual/forearm.dae"/>
         </geometry>
-        <material name="LightGrey">
-          <color rgba="0.7 0.7 0.7 1.0"/>
-        </material>
       </visual>
       <collision>
@@ -166,7 +154,4 @@
           <mesh filename="file://$(find ros2srrc_robots)/ur3/meshes/visual/wrist1.dae"/>
         </geometry>
-        <material name="LightGrey">
-          <color rgba="0.7 0.7 0.7 1.0"/>
-        </material>
       </visual>
       <collision>
@@ -186,7 +171,4 @@
           <mesh filename="file://$(find ros2srrc_robots)/ur3/meshes/visual/wrist2.dae"/>
         </geometry>
-        <material name="LightGrey">
-          <color rgba="0.7 0.7 0.7 1.0"/>
-        </material>
       </visual>
       <collision>
@@ -206,7 +188,4 @@
           <mesh filename="file://$(find ros2srrc_robots)/ur3/meshes/visual/wrist3.dae"/>
         </geometry>
-        <material name="LightGrey">
-          <color rgba="0.7 0.7 0.7 1.0"/>
-        </material>
       </visual>
       <collision>
@@ -238,5 +217,5 @@
       <limit lower="${shoulder_pan_lower_limit}" upper="${shoulder_pan_upper_limit}"
         effort="${shoulder_pan_effort_limit}" velocity="${shoulder_pan_velocity_limit}"/>
-      <dynamics damping="1.0" friction="100.0"/>
+      <dynamics damping="0.0" friction="0.0"/>
     </joint>
     <joint name="shoulder_lift_joint" type="revolute">
@@ -247,5 +226,5 @@
       <limit lower="${shoulder_lift_lower_limit}" upper="${shoulder_lift_upper_limit}"
         effort="${shoulder_lift_effort_limit}" velocity="${shoulder_lift_velocity_limit}"/>
-      <dynamics damping="1.0" friction="100.0"/>
+      <dynamics damping="0.0" friction="0.0"/>
     </joint>
     <joint name="elbow_joint" type="revolute">
@@ -256,5 +235,5 @@
       <limit lower="${elbow_joint_lower_limit}" upper="${elbow_joint_upper_limit}"
         effort="${elbow_joint_effort_limit}" velocity="${elbow_joint_velocity_limit}"/>
-      <dynamics damping="1.0" friction="100.0"/>
+      <dynamics damping="0.0" friction="0.0"/>
     </joint>
     <joint name="wrist_1_joint" type="revolute">
@@ -265,5 +244,5 @@
       <limit lower="${wrist_1_lower_limit}" upper="${wrist_1_upper_limit}"
         effort="${wrist_1_effort_limit}" velocity="${wrist_1_velocity_limit}"/>
-      <dynamics damping="1.0" friction="10.0"/>
+      <dynamics damping="0.0" friction="0.0"/>
     </joint>
     <joint name="wrist_2_joint" type="revolute">
@@ -274,5 +253,5 @@
       <limit lower="${wrist_2_lower_limit}" upper="${wrist_2_upper_limit}"
              effort="${wrist_2_effort_limit}" velocity="${wrist_2_velocity_limit}"/>
-      <dynamics damping="1.0" friction="10.0"/>
+      <dynamics damping="0.0" friction="0.0"/>
     </joint>
     <joint name="wrist_3_joint" type="revolute">
@@ -283,5 +262,5 @@
       <limit lower="${wrist_3_lower_limit}" upper="${wrist_3_upper_limit}"
              effort="${wrist_3_effort_limit}" velocity="${wrist_3_velocity_limit}"/>
-      <dynamics damping="1.0" friction="1.0"/>
+      <dynamics damping="0.0" friction="0.0"/>
     </joint>
     <!-- ROS-Industrial 'base' frame - base_link to UR 'Base' Coordinates transform -->

File: ros2srrc_robots/ur3/urdf/ur3_ros2control.xacro (robot description, xacro)
@@ -102,5 +102,5 @@
     <!-- A. GAZEBO SIMULATION: -->
     <xacro:unless value="${bringup}">
-      <xacro:property name="name" value="GazeboSystem"/>
+      <xacro:property name="name" value="GazeboSimSystem"/>
     </xacro:unless>
     <!-- B. ROBOT BRINGUP: -->
@@ -113,5 +113,5 @@
       <xacro:unless value="${bringup}">
         <hardware>
-          <plugin>gazebo_ros2_control/GazeboSystem</plugin>
+          <plugin>gz_ros2_control/GazeboSimSystem</plugin>
         </hardware>
       </xacro:unless>

Commit message: Remove empty dynamics tags (UR3).

File: ros2srrc_robots/ur3/urdf/ur3_macro.urdf.xacro (robot description, xacro)
@@ -217,5 +217,4 @@
       <limit lower="${shoulder_pan_lower_limit}" upper="${shoulder_pan_upper_limit}"
         effort="${shoulder_pan_effort_limit}" velocity="${shoulder_pan_velocity_limit}"/>
-      <dynamics damping="0.0" friction="0.0"/>
     </joint>
     <joint name="shoulder_lift_joint" type="revolute">
@@ -226,5 +225,4 @@
       <limit lower="${shoulder_lift_lower_limit}" upper="${shoulder_lift_upper_limit}"
         effort="${shoulder_lift_effort_limit}" velocity="${shoulder_lift_velocity_limit}"/>
-      <dynamics damping="0.0" friction="0.0"/>
     </joint>
     <joint name="elbow_joint" type="revolute">
@@ -235,5 +233,4 @@
       <limit lower="${elbow_joint_lower_limit}" upper="${elbow_joint_upper_limit}"
         effort="${elbow_joint_effort_limit}" velocity="${elbow_joint_velocity_limit}"/>
-      <dynamics damping="0.0" friction="0.0"/>
     </joint>
     <joint name="wrist_1_joint" type="revolute">
@@ -244,5 +241,4 @@
       <limit lower="${wrist_1_lower_limit}" upper="${wrist_1_upper_limit}"
         effort="${wrist_1_effort_limit}" velocity="${wrist_1_velocity_limit}"/>
-      <dynamics damping="0.0" friction="0.0"/>
     </joint>
     <joint name="wrist_2_joint" type="revolute">
@@ -253,5 +249,4 @@
       <limit lower="${wrist_2_lower_limit}" upper="${wrist_2_upper_limit}"
              effort="${wrist_2_effort_limit}" velocity="${wrist_2_velocity_limit}"/>
-      <dynamics damping="0.0" friction="0.0"/>
     </joint>
     <joint name="wrist_3_joint" type="revolute">
@@ -262,5 +257,4 @@
       <limit lower="${wrist_3_lower_limit}" upper="${wrist_3_upper_limit}"
              effort="${wrist_3_effort_limit}" velocity="${wrist_3_velocity_limit}"/>
-      <dynamics damping="0.0" friction="0.0"/>
     </joint>
     <!-- ROS-Industrial 'base' frame - base_link to UR 'Base' Coordinates transform -->
