Commit message: Migrate to GzFortress: IRB1600 + IRB6640 robots and Zimmer gripper.

File: packages/ros2srrc_irb1600/urdf/irb1600.urdf.xacro (robot description, xacro)
@@ -1,3 +1,3 @@
-<?xml version="1.0"?>
+<?xml version="1.0" ?>
 <!--
 # ===================================== COPYRIGHT ===================================== #
@@ -28,36 +28,64 @@
 # IFRA-Cranfield (2023) ROS 2 Sim-to-Real Robot Control. URL: https://github.com/IFRA-Cranfield/ros2_SimRealRobotControl.
 -->
-<robot xmlns:xacro="http://www.ros.org/wiki/xacro">
-  <xacro:macro name="EE_ros2control" params="" >
-    <!-- gpp5010nc_finger_left_joint -->
-    <joint name="gpp5010nc_finger_left_joint">
-      <command_interface name="position">
-        <param name="min">-0.0001</param>
-        <param name="max">0.0101</param>
-      </command_interface>
-      <command_interface name="velocity">
-        <param name="min">-1.0</param>
-        <param name="max">1.0</param>
-      </command_interface>
-      <state_interface name="position">
-        <param name="initial_value">0.0</param>
-      </state_interface>
-      <state_interface name="velocity"/>
-    </joint>
-    <!-- gpp5010nc_finger_right_joint -->
-    <joint name="gpp5010nc_finger_right_joint">
-      <command_interface name="position">
-        <param name="min">-0.0001</param>
-        <param name="max">0.0101</param>
-      </command_interface>
-      <command_interface name="velocity">
-        <param name="min">-1.0</param>
-        <param name="max">1.0</param>
-      </command_interface>
-      <state_interface name="position">
-        <param name="initial_value">0.0</param>
-      </state_interface>
-      <state_interface name="velocity"/>
-    </joint>
-  </xacro:macro>
+<robot name="irb1600" xmlns:xacro="http://ros.org/wiki/xacro">
+  <!-- PASS ARGUMENTS: -->
+  <xacro:arg name="bringup" default="false"/>
+  <xacro:property name="bringup" value="$(arg bringup)"/>
+  <xacro:arg name="robot_ip" default="0.0.0.0"/>
+  <xacro:property name="robot_ip" value="$(arg robot_ip)"/>
+  <xacro:arg name="EE" default="false"/>
+  <xacro:property name="EE" value="$(arg EE)"/>
+  <xacro:arg name="EE_name" default="none"/>
+  <xacro:property name="EE_name" value="$(arg EE_name)"/>
+  <!-- Include XACRO-MACRO file of the IRB1600: -->
+  <xacro:include filename="$(find ros2srrc_robots)/irb1600/urdf/irb1600_macro.urdf.xacro"/>
+  <xacro:irb1600
+    bringup="${bringup}"
+    robot_ip="${robot_ip}"
+    EE="${EE}"
+    EE_name="${EE_name}"
+  />
+  <!-- Load ROS 2 Gazebo Plugin -->
+  <xacro:unless value="${bringup}">
+    <gazebo>
+      <plugin filename="gz_ros2_control-system" name="gz_ros2_control::GazeboSimROS2ControlPlugin">
+        <!-- IRB1600 Controller -->
+        <parameters>$(find ros2srrc_robots)/irb1600/config/controller.yaml</parameters>
+      </plugin>
+    </gazebo>
+  </xacro:unless>
+  <!-- World: LINK -->
+  <link name="world"/>
+  <!-- Robot Stand: LINK -->
+  <link name='robot_stand'>
+    <inertial>
+      <origin xyz="0 0 0" rpy="0 0 0"/>
+      <mass value="10000"/>
+      <inertia ixx="0.01"  ixy="0"  ixz="0" iyy="0.01" iyz="0" izz="0.01" />
+    </inertial>
+    <collision name='collision'>
+      <origin xyz="0 0 0" rpy=" 0 0 0"/>
+      <geometry>
+        <box size = "1.5 1.5 0.5"/>
+      </geometry>
+    </collision>
+    <visual name='chassis_visual'>
+      <origin xyz="0 0 0" rpy=" 0 0 0"/>
+      <geometry>
+        <box size = "1.5 1.5 0.5"/>
+      </geometry>
+    </visual>
+  </link>
+  <!-- Robot Stand: FIXED JOINT -->
+  <joint name="world_joint" type="fixed">
+    <parent link="world" />
+    <child link = "robot_stand" />
+    <origin xyz="0.0 0.0 0.25" rpy="0.0 0.0 0.0" />
+  </joint>
+  <!-- Robot Stand: Robot+Stand JOINT -->
+  <joint name="stand_joint" type="fixed">
+    <parent link="robot_stand" />
+    <child link = "base_link" />
+    <origin xyz="0.0 0.0 0.255" rpy="0.0 0.0 0.0" />
+  </joint>
 </robot>

File: packages/ros2srrc_irb6640/urdf/irb6640.urdf.xacro (robot description, xacro)
@@ -1,3 +1,3 @@
-<?xml version="1.0"?>
+<?xml version="1.0" ?>
 <!--
 # ===================================== COPYRIGHT ===================================== #
@@ -28,36 +28,64 @@
 # IFRA-Cranfield (2023) ROS 2 Sim-to-Real Robot Control. URL: https://github.com/IFRA-Cranfield/ros2_SimRealRobotControl.
 -->
-<robot xmlns:xacro="http://www.ros.org/wiki/xacro">
-  <xacro:macro name="EE_ros2control" params="" >
-    <!-- gpp5010nc_finger_left_joint -->
-    <joint name="gpp5010nc_finger_left_joint">
-      <command_interface name="position">
-        <param name="min">-0.0001</param>
-        <param name="max">0.0101</param>
-      </command_interface>
-      <command_interface name="velocity">
-        <param name="min">-1.0</param>
-        <param name="max">1.0</param>
-      </command_interface>
-      <state_interface name="position">
-        <param name="initial_value">0.0</param>
-      </state_interface>
-      <state_interface name="velocity"/>
-    </joint>
-    <!-- gpp5010nc_finger_right_joint -->
-    <joint name="gpp5010nc_finger_right_joint">
-      <command_interface name="position">
-        <param name="min">-0.0001</param>
-        <param name="max">0.0101</param>
-      </command_interface>
-      <command_interface name="velocity">
-        <param name="min">-1.0</param>
-        <param name="max">1.0</param>
-      </command_interface>
-      <state_interface name="position">
-        <param name="initial_value">0.0</param>
-      </state_interface>
-      <state_interface name="velocity"/>
-    </joint>
-  </xacro:macro>
+<robot name="irb6640" xmlns:xacro="http://ros.org/wiki/xacro">
+  <!-- PASS ARGUMENTS: -->
+  <xacro:arg name="bringup" default="false"/>
+  <xacro:property name="bringup" value="$(arg bringup)"/>
+  <xacro:arg name="robot_ip" default="0.0.0.0"/>
+  <xacro:property name="robot_ip" value="$(arg robot_ip)"/>
+  <xacro:arg name="EE" default="false"/>
+  <xacro:property name="EE" value="$(arg EE)"/>
+  <xacro:arg name="EE_name" default="none"/>
+  <xacro:property name="EE_name" value="$(arg EE_name)"/>
+  <!-- Include XACRO-MACRO file of the IRB6640: -->
+  <xacro:include filename="$(find ros2srrc_robots)/irb6640/urdf/irb6640_macro.urdf.xacro"/>
+  <xacro:irb6640
+    bringup="${bringup}"
+    robot_ip="${robot_ip}"
+    EE="${EE}"
+    EE_name="${EE_name}"
+  />
+  <!-- Load ROS 2 Gazebo Plugin -->
+  <xacro:unless value="${bringup}">
+    <gazebo>
+      <plugin filename="gz_ros2_control-system" name="gz_ros2_control::GazeboSimROS2ControlPlugin">
+        <!-- IRB6640 Controller -->
+        <parameters>$(find ros2srrc_robots)/irb6640/config/controller.yaml</parameters>
+      </plugin>
+    </gazebo>
+  </xacro:unless>
+  <!-- World: LINK -->
+  <link name="world"/>
+  <!-- Robot Stand: LINK -->
+  <link name='robot_stand'>
+    <inertial>
+      <origin xyz="0 0 0" rpy="0 0 0"/>
+      <mass value="10000"/>
+      <inertia ixx="0.01"  ixy="0"  ixz="0" iyy="0.01" iyz="0" izz="0.01" />
+    </inertial>
+    <collision name='collision'>
+      <origin xyz="0 0 0" rpy=" 0 0 0"/>
+      <geometry>
+        <box size = "1.5 1.5 0.5"/>
+      </geometry>
+    </collision>
+    <visual name='chassis_visual'>
+      <origin xyz="0 0 0" rpy=" 0 0 0"/>
+      <geometry>
+        <box size = "1.5 1.5 0.5"/>
+      </geometry>
+    </visual>
+  </link>
+  <!-- Robot Stand: FIXED JOINT -->
+  <joint name="world_joint" type="fixed">
+    <parent link="world" />
+    <child link = "robot_stand" />
+    <origin xyz="0.0 0.0 0.25" rpy="0.0 0.0 0.0" />
+  </joint>
+  <!-- Robot Stand: Robot+Stand JOINT -->
+  <joint name="stand_joint" type="fixed">
+    <parent link="robot_stand" />
+    <child link = "base_link" />
+    <origin xyz="0.0 0.0 0.255" rpy="0.0 0.0 0.0" />
+  </joint>
 </robot>

File: ros2srrc_endeffectors/gpp5010nc/urdf/gpp5010nc_macro.urdf.xacro (robot description, xacro)
@@ -48,4 +48,7 @@
           <mesh filename="file://$(find ros2srrc_endeffectors)/gpp5010nc/meshes/gpp5010nc_MainBody.dae" />
         </geometry>
+        <material name="silver">
+          <color rgba="0.8 0.8 0.8 1"/>
+        </material>
       </visual>
       <collision>
@@ -81,8 +84,8 @@
       <parent link="gpp5010nc_gripper_base_link" />
       <child link="gpp5010nc_finger_left_link" />
-      <limit effort="1000" lower="-0.001" upper="0.011" velocity="1.0"/>
+      <limit effort="1000" lower="-0.0001" upper="0.0101" velocity="1.0"/>
       <origin xyz="0.0 0.0 0.0" rpy="0 0 0" />
       <axis xyz="0 -1 0" />
-      <dynamics damping="1.0" friction="1.0"/>
+      <dynamics damping="0.2" friction="0.05"/>
     </joint>
     <!-- RIGHT FINGER -->
@@ -107,8 +110,8 @@
       <parent link="gpp5010nc_gripper_base_link" />
       <child link="gpp5010nc_finger_right_link" />
-      <limit effort="1000" lower="-0.001" upper="0.011" velocity="1.0"/>
+      <limit effort="1000" lower="-0.0001" upper="0.0101" velocity="1.0"/>
       <origin xyz="0.0 0.0 0.0" rpy="0 0 0" />
       <axis xyz="0 1 0" />
-      <dynamics damping="1.0" friction="1.0"/>
+      <dynamics damping="0.2" friction="0.05"/>
     </joint>
     <gazebo reference="gpp5010nc_finger_right_link">

File: ros2srrc_robots/irb1600/urdf/irb1600_macro.urdf.xacro (robot description, xacro)
@@ -177,5 +177,5 @@
         <mass value="0.38"/>
         <origin xyz="0.0 0.0 0.0"/>
-        <inertia ixx="0.0" ixy="0.0" ixz="0.0" iyy="0.0" iyz="0.0" izz="0.0"/>
+          <inertia ixx="2.1e-04" ixy="0.0" ixz="0.0" iyy="2.1e-04" iyz="0.0" izz="3.0e-04"/>
       </inertial>
       <collision name="collision">
@@ -198,5 +198,5 @@
         <mass value="0.08"/>
         <origin xyz="0.0 0.0 0.0"/>
-        <inertia ixx="0.0" ixy="0.0" ixz="0.0" iyy="0.0" iyz="0.0" izz="0.0"/>
+          <inertia ixx="2.2e-05" ixy="0.0" ixz="0.0" iyy="2.2e-05" iyz="0.0" izz="2.5e-05"/>
       </inertial>
       <collision name="collision">
@@ -223,5 +223,5 @@
       <child link="link_1"/>
       <limit lower="-3.142" upper="3.142" effort="1000" velocity="3.142"/>
-      <dynamics damping="50.0" friction="1.0"/>
+      <dynamics damping="0.3" friction="0.0"/>
     </joint>
     <!-- joint_2 -->
@@ -232,5 +232,5 @@
       <child link="link_2"/>
       <limit lower="-1.571" upper="2.094" effort="1000" velocity="3.142"/>
-      <dynamics damping="50.0" friction="1.0"/>
+      <dynamics damping="0.3" friction="0.0"/>
     </joint>
     <!-- joint_3 -->
@@ -241,5 +241,5 @@
       <child link="link_3"/>
       <limit lower="-4.276" upper="1.134" effort="1000" velocity="3.228"/>
-      <dynamics damping="10.0" friction="1.0"/>
+      <dynamics damping="0.2" friction="0.0"/>
     </joint>
     <!-- joint_4 -->
@@ -250,5 +250,5 @@
       <child link="link_4"/>
       <limit lower="-3.490" upper="3.490" effort="1000" velocity="6.719"/>
-      <dynamics damping="5.0" friction="1.0"/>
+      <dynamics damping="0.05" friction="0.0"/>
     </joint>
     <!-- joint_5 -->
@@ -259,5 +259,5 @@
       <child link="link_5"/>
       <limit lower="-2.007" upper="2.007" effort="1000" velocity="6.981"/>
-      <dynamics damping="2.0" friction="1.0"/>
+      <dynamics damping="0.03" friction="0.0"/>
     </joint>
     <!-- joint_6 -->
@@ -268,5 +268,5 @@
       <child link="link_6"/>
       <limit lower="-6.981" upper="6.981" effort="1000" velocity="8.028"/>
-      <dynamics damping="1.0" friction="1.0"/>
+      <dynamics damping="0.02" friction="0.0"/>
     </joint>
     <!-- end of joint list -->

File: ros2srrc_robots/irb1600/urdf/irb1600_ros2control.xacro (robot description, xacro)
@@ -52,5 +52,5 @@
     <!-- A. GAZEBO SIMULATION: -->
     <xacro:unless value="${bringup}">
-      <xacro:property name="name" value="GazeboSystem"/>
+      <xacro:property name="name" value="GazeboSimSystem"/>
     </xacro:unless>
     <!-- B. ROBOT BRINGUP: -->
@@ -63,5 +63,5 @@
       <xacro:unless value="${bringup}">
         <hardware>
-          <plugin>gazebo_ros2_control/GazeboSystem</plugin>
+          <plugin>gz_ros2_control/GazeboSimSystem</plugin>
         </hardware>
       </xacro:unless>
@@ -146,5 +146,5 @@
         </command_interface>
         <state_interface name="position">
-          <param name="initial_value">0.0</param>
+          <param name="initial_value">1.5708</param>
         </state_interface>
         <state_interface name="velocity"/>

File: ros2srrc_robots/irb6640/urdf/irb6640_macro.urdf.xacro (robot description, xacro)
@@ -92,5 +92,5 @@
         <origin xyz="0 0 0" rpy="0 0 0"/>
         <geometry>
-          <mesh filename="file://$(find ros2srrc_robots)/irb6640/meshes/base_link.dae"/>
+          <mesh filename="file://$(find ros2srrc_robots)/irb6640/meshes/base_link.stl"/>
         </geometry>
       </collision>
@@ -111,5 +111,5 @@
         <origin xyz="0 0 0" rpy="0 0 0"/>
         <geometry>
-          <mesh filename="file://$(find ros2srrc_robots)/irb6640/meshes/link_1.dae"/>
+          <mesh filename="file://$(find ros2srrc_robots)/irb6640/meshes/link_1.stl"/>
         </geometry>
       </collision>
@@ -130,5 +130,5 @@
         <origin xyz="0 0 0" rpy="0 0 0"/>
         <geometry>
-          <mesh filename="file://$(find ros2srrc_robots)/irb6640/meshes/link_2.dae"/>
+          <mesh filename="file://$(find ros2srrc_robots)/irb6640/meshes/link_2.stl"/>
         </geometry>
       </collision>
@@ -149,5 +149,5 @@
         <origin xyz="0 0 0" rpy="0 0 0"/>
         <geometry>
-          <mesh filename="file://$(find ros2srrc_robots)/irb6640/meshes/link_3.dae"/>
+          <mesh filename="file://$(find ros2srrc_robots)/irb6640/meshes/link_3.stl"/>
         </geometry>
       </collision>
@@ -168,5 +168,5 @@
         <origin xyz="0 0 0" rpy="0 0 0"/>
         <geometry>
-          <mesh filename="file://$(find ros2srrc_robots)/irb6640/meshes/link_4.dae"/>
+          <mesh filename="file://$(find ros2srrc_robots)/irb6640/meshes/link_4.stl"/>
         </geometry>
       </collision>
@@ -187,5 +187,5 @@
         <origin xyz="0 0 0" rpy="0 0 0"/>
         <geometry>
-          <mesh filename="file://$(find ros2srrc_robots)/irb6640/meshes/link_5.dae"/>
+          <mesh filename="file://$(find ros2srrc_robots)/irb6640/meshes/link_5.stl"/>
         </geometry>
       </collision>
@@ -206,5 +206,5 @@
         <origin xyz="0 0 0" rpy="0 0 0"/>
         <geometry>
-          <mesh filename="file://$(find ros2srrc_robots)/irb6640/meshes/link_6.dae"/>
+          <mesh filename="file://$(find ros2srrc_robots)/irb6640/meshes/link_6.stl"/>
         </geometry>
       </collision>
@@ -215,5 +215,5 @@
         <mass value="1.34" />
         <origin xyz="0.0 0.0 0.0" rpy="0 0 0"/>
-        <inertia ixx="0.0" ixy="0.0" ixz="0.01" iyy="0.05" iyz="0.0" izz="0.04"/>
+          <inertia ixx="0.02" ixy="0.0" ixz="0.01" iyy="0.05" iyz="0.0" izz="0.04"/>
       </inertial>
       <visual>
@@ -226,5 +226,5 @@
         <origin xyz="0 0 0" rpy="0 0 0"/>
         <geometry>
-          <mesh filename="file://$(find ros2srrc_robots)/irb6640/meshes/link_piston.dae"/>
+          <mesh filename="file://$(find ros2srrc_robots)/irb6640/meshes/link_piston.stl"/>
         </geometry>
       </collision>
@@ -245,5 +245,5 @@
         <origin xyz="0 0 0" rpy="0 0 0"/>
         <geometry>
-          <mesh filename="file://$(find ros2srrc_robots)/irb6640/meshes/link_cylinder.dae"/>
+          <mesh filename="file://$(find ros2srrc_robots)/irb6640/meshes/link_cylinder.stl"/>
         </geometry>
       </collision>
@@ -256,5 +256,6 @@
       <parent link="base_link"/>
       <child link="link_1"/>
-      <limit effort="0" lower="-2.96706" upper="2.96706" velocity="1.7453"/>
+      <limit effort="3000" lower="-2.96706" upper="2.96706" velocity="1.7453"/>
+      <dynamics damping="0.5" friction="0.0"/>
     </joint>
     <joint type="revolute" name="joint_2">
@@ -263,5 +264,6 @@
       <parent link="link_1"/>
       <child link="link_2"/>
-      <limit effort="0" lower="-1.134" upper="1.4835" velocity="1.5708"/>
+      <limit effort="3000" lower="-1.134" upper="1.4835" velocity="1.5708"/>
+      <dynamics damping="0.3" friction="0.0"/>
     </joint>
     <joint type="revolute" name="joint_3">
@@ -270,5 +272,6 @@
       <parent link="link_2"/>
       <child link="link_3"/>
-      <limit effort="0" lower="-3.1416" upper="1.2217" velocity="1.5708"/>
+      <limit effort="2500" lower="-3.1416" upper="1.2217" velocity="1.5708"/>
+      <dynamics damping="0.2" friction="0.0"/>
     </joint>
     <joint type="revolute" name="joint_4">
@@ -277,5 +280,6 @@
       <parent link="link_3"/>
       <child link="link_4"/>
-      <limit effort="0" lower="-5.236" upper="5.236" velocity="2.9671"/>
+      <limit effort="800" lower="-5.236" upper="5.236" velocity="2.9671"/>
+      <dynamics damping="0.1" friction="0.0"/>
     </joint>
     <joint type="revolute" name="joint_5">
@@ -284,5 +288,6 @@
       <parent link="link_4"/>
       <child link="link_5"/>
-      <limit effort="0" lower="-2.0944" upper="2.0944" velocity="2.0944"/>
+      <limit effort="600" lower="-2.0944" upper="2.0944" velocity="2.0944"/>
+      <dynamics damping="0.05" friction="0.0"/>
     </joint>
     <joint type="revolute" name="joint_6">
@@ -291,5 +296,6 @@
       <parent link="link_5"/>
       <child link="link_6"/>
-      <limit effort="0" lower="-6.283" upper="6.283" velocity="3.3161"/>
+      <limit effort="400" lower="-6.283" upper="6.283" velocity="3.3161"/>
+      <dynamics damping="0.01" friction="0.0"/>
     </joint>
     <joint type="continuous" name="joint_cylinder">
@@ -299,4 +305,5 @@
       <child link="link_cylinder"/>
       <mimic joint="joint_2" multiplier="-0.35" offset="0.0"/>
+      <dynamics damping="0.1" friction="0.0"/>
     </joint>
     <joint type="continuous" name="joint_piston">
@@ -306,4 +313,5 @@
       <child link="link_piston"/>
       <mimic joint="joint_2" multiplier="-1.35" offset="0.0"/>
+      <dynamics damping="0.1" friction="0.0"/>
     </joint>
     <!-- end of joint list -->

File: ros2srrc_robots/irb6640/urdf/irb6640_ros2control.xacro (robot description, xacro)
@@ -52,5 +52,5 @@
     <!-- A. GAZEBO SIMULATION: -->
     <xacro:unless value="${bringup}">
-      <xacro:property name="name" value="GazeboSystem"/>
+      <xacro:property name="name" value="GazeboSimSystem"/>
     </xacro:unless>
     <!-- B. ROBOT BRINGUP: -->
@@ -63,5 +63,5 @@
       <xacro:unless value="${bringup}">
         <hardware>
-          <plugin>gazebo_ros2_control/GazeboSystem</plugin>
+          <plugin>gz_ros2_control/GazeboSimSystem</plugin>
         </hardware>
       </xacro:unless>
