Commit message: Fix colour in urdf file.

File: ros2srrc_robots/irb1600/urdf/irb1600_macro.urdf.xacro (robot description, xacro)
@@ -85,5 +85,7 @@
           <mesh filename="file://$(find ros2srrc_robots)/irb1600/meshes/visual/base_link.stl"/>
         </geometry>
-        <xacro:material_abb_yellow />
+        <material name="silver">
+          <color rgba="0.75 0.75 0.75 1"/>
+        </material>
       </visual>
     </link>
@@ -106,5 +108,7 @@
           <mesh filename="file://$(find ros2srrc_robots)/irb1600/meshes/visual/link_1.stl"/>
         </geometry>
-        <xacro:material_abb_yellow />
+        <material name="silver">
+          <color rgba="0.75 0.75 0.75 1"/>
+        </material>
       </visual>
     </link>
@@ -127,5 +131,7 @@
           <mesh filename="file://$(find ros2srrc_robots)/irb1600/meshes/visual/link_2.stl"/>
         </geometry>
-        <xacro:material_abb_yellow />
+        <material name="silver">
+          <color rgba="0.75 0.75 0.75 1"/>
+        </material>
       </visual>
     </link>
@@ -148,5 +154,7 @@
           <mesh filename="file://$(find ros2srrc_robots)/irb1600/meshes/visual/link_3.stl"/>
         </geometry>
-        <xacro:material_abb_yellow />
+        <material name="silver">
+          <color rgba="0.75 0.75 0.75 1"/>
+        </material>
       </visual>
     </link>
@@ -169,5 +177,7 @@
           <mesh filename="file://$(find ros2srrc_robots)/irb1600/meshes/visual/link_4.stl"/>
         </geometry>
-        <xacro:material_abb_yellow />
+        <material name="silver">
+          <color rgba="0.75 0.75 0.75 1"/>
+        </material>
       </visual>
     </link>
@@ -190,5 +200,7 @@
           <mesh filename="file://$(find ros2srrc_robots)/irb1600/meshes/visual/link_5.stl"/>
         </geometry>
-        <xacro:material_abb_yellow />
+        <material name="silver">
+          <color rgba="0.75 0.75 0.75 1"/>
+        </material>
       </visual>
     </link>
@@ -211,5 +223,7 @@
           <mesh filename="file://$(find ros2srrc_robots)/irb1600/meshes/visual/link_6.stl"/>
         </geometry>
-        <xacro:material_abb_yellow />
+        <material name="black">
+          <color rgba="0.0 0.0 0.0 1"/>
+        </material>
       </visual>
     </link>
