Commit message: Fix: If->EE, /RobPose to refer EE_link, /RobMove to refer EE_link (before it was tool0).

File: ros2srrc_endeffectors/egp64/urdf/egp64_macro.urdf.xacro (robot description, xacro)
@@ -215,26 +215,9 @@
       </visual>
     </link>
-    <xacro:unless value="${bringup}">
-      <joint name="EE_egp64_joint" type="prismatic" >
-        <parent link="${parent_link}" />
-        <child link="EE_egp64" />
-        <limit effort="10000" lower="0.0" upper="0.0" velocity="0.0"/>
-        <axis xyz="1 0 0" />
-        <origin xyz="0.0 0.0 0.19" rpy="0 0 0"/>
-      </joint>
-      <!-- LOAD LinkPose Gazebo (ROS2) PLUGIN: -->
-      <gazebo>
-        <plugin name="ros2_linkpose_plugin" filename="libros2_linkpose_plugin.so" >
-          <link>EE_egp64</link>
-        </plugin>
-      </gazebo>
-    </xacro:unless>
-    <xacro:if value="${bringup}">
-      <joint name="EE_egp64_joint" type="fixed" >
-        <parent link="${parent_link}" />
-        <child link="EE_egp64" />
-        <origin xyz="0.0 0.0 0.19" rpy="0 0 0"/>
-      </joint>
-    </xacro:if>
+    <joint name="EE_egp64_joint" type="fixed" >
+      <parent link="${parent_link}" />
+      <child link="EE_egp64" />
+      <origin xyz="0.0 0.0 0.19" rpy="0 0 0"/>
+    </joint>
   </xacro:macro>
 </robot>

File: ros2srrc_endeffectors/egp64/urdf/egp64_ros2control.xacro (robot description, xacro)
@@ -60,10 +60,4 @@
       <state_interface name="velocity"/>
     </joint>
-    <joint name="EE_egp64_joint">
-      <command_interface name="position"/>
-      <command_interface name="velocity"/>
-      <state_interface name="position"/>
-      <state_interface name="velocity"/>
-    </joint>
   </xacro:macro>
 </robot>

File: ros2srrc_endeffectors/robotiq_2f85/urdf/robotiq_2f85_macro.urdf.xacro (robot description, xacro)
@@ -324,26 +324,9 @@
       </visual>
     </link>
-    <xacro:unless value="${bringup}">
-      <joint name="EE_robotiq_2f85_joint" type="prismatic" >
-        <parent link="robotiq_85_base_link" />
-        <child link="EE_robotiq_2f85" />
-        <limit effort="10000" lower="0.0" upper="0.0" velocity="0.0"/>
-        <axis xyz="1 0 0" />
-        <origin xyz="0.128 0.0 0.0" rpy="0 0 0"/>
-      </joint>
-      <!-- LOAD LinkPose Gazebo (ROS2) PLUGIN: -->
-      <gazebo>
-        <plugin name="ros2_linkpose_plugin" filename="libros2_linkpose_plugin.so" >
-          <link>EE_robotiq_2f85</link>
-        </plugin>
-      </gazebo>
-    </xacro:unless>
-    <xacro:if value="${bringup}">
-      <joint name="EE_robotiq_2f85_joint" type="fixed" >
-        <parent link="robotiq_85_base_link" />
-        <child link="EE_robotiq_2f85" />
-        <origin xyz="0.128 0.0 0.0" rpy="0 0 0"/>
-      </joint>
-    </xacro:if>
+    <joint name="EE_robotiq_2f85_joint" type="fixed" >
+      <parent link="robotiq_85_base_link" />
+      <child link="EE_robotiq_2f85" />
+      <origin xyz="0.128 0.0 0.0" rpy="0 0 0"/>
+    </joint>
   </xacro:macro>
 </robot>

File: ros2srrc_endeffectors/robotiq_2f85/urdf/robotiq_2f85_ros2control.xacro (robot description, xacro)
@@ -120,10 +120,4 @@
       <state_interface name="effort"/>
     </joint>
-    <joint name="EE_robotiq_2f85_joint">
-      <command_interface name="position"/>
-      <command_interface name="velocity"/>
-      <state_interface name="position"/>
-      <state_interface name="velocity"/>
-    </joint>
   </xacro:macro>
 </robot>

File: ros2srrc_endeffectors/robotiq_hande/urdf/robotiq_hande_macro.urdf.xacro (robot description, xacro)
@@ -189,26 +189,9 @@
       </visual>
     </link>
-    <xacro:unless value="${bringup}">
-      <joint name="EE_robotiq_hande_joint" type="prismatic" >
-        <parent link="robotiq_hande_base_link" />
-        <child link="EE_robotiq_hande" />
-        <limit effort="10000" lower="0.0" upper="0.0" velocity="0.0"/>
-        <axis xyz="1 0 0" />
-        <origin xyz="0.0 0.0 0.135" rpy="0 0 0"/>
-      </joint>
-      <!-- LOAD LinkPose Gazebo (ROS2) PLUGIN: -->
-      <gazebo>
-        <plugin name="ros2_linkpose_plugin" filename="libros2_linkpose_plugin.so" >
-          <link>EE_robotiq_hande</link>
-        </plugin>
-      </gazebo>
-    </xacro:unless>
-    <xacro:if value="${bringup}">
-      <joint name="EE_robotiq_hande_joint" type="fixed" >
-        <parent link="robotiq_hande_base_link" />
-        <child link="EE_robotiq_hande" />
-        <origin xyz="0.0 0.0 0.135" rpy="0 0 0"/>
-      </joint>
-    </xacro:if>
+    <joint name="EE_robotiq_hande_joint" type="fixed" >
+      <parent link="robotiq_hande_base_link" />
+      <child link="EE_robotiq_hande" />
+      <origin xyz="0.0 0.0 0.135" rpy="0 0 0"/>
+    </joint>
   </xacro:macro>
 </robot>

File: ros2srrc_endeffectors/robotiq_hande/urdf/robotiq_hande_ros2control.xacro (robot description, xacro)
@@ -60,10 +60,4 @@
       <state_interface name="effort"/>
     </joint>
-    <joint name="EE_robotiq_hande_joint">
-      <command_interface name="position"/>
-      <command_interface name="velocity"/>
-      <state_interface name="position"/>
-      <state_interface name="velocity"/>
-    </joint>
   </xacro:macro>
 </robot>

Commit message: Fix inertia, colour and dynamics tags in urdf files.

File: ros2srrc_endeffectors/egp64/urdf/egp64_macro.urdf.xacro (robot description, xacro)
@@ -119,5 +119,5 @@
       <origin xyz="0.01483 -0.00782 0" rpy="0 0 0" />
       <axis xyz="-1 0 0" />
-      <dynamics damping="1.0" friction="1.0"/>
+      <dynamics damping="0.0" friction="0.0"/>
     </joint>
     <!-- LEFT FINGERTIP -->
@@ -174,5 +174,5 @@
       <origin xyz="-0.0153 -0.00602 0" rpy="0 0 0" />
       <axis xyz="1 0 0" />
-      <dynamics damping="1.0" friction="1.0"/>
+      <dynamics damping="0.0" friction="0.0"/>
     </joint>
     <!-- RIGHT FINGERTIP -->

File: ros2srrc_endeffectors/robotiq_2f85/urdf/robotiq_2f85_macro.urdf.xacro (robot description, xacro)
@@ -117,5 +117,5 @@
       <origin rpy="${pi} 0.0 0.0" xyz="0.05490451627 0.03060114443 0.0"/>
       <limit lower="-0.05" upper="0.80285" velocity="0.5" effort="1000"/>
-      <dynamics damping="1.0" friction="1.0"/>
+      <dynamics damping="0.0" friction="0.0"/>
     </joint>
     <!-- Robotiq: right_knuckle -->
@@ -145,5 +145,5 @@
       <origin rpy="0.0 0.0 0.0" xyz="0.05490451627 -0.03060114443 0.0"/>
       <limit lower="-0.05" upper="0.80285" velocity="0.5" effort="1000"/>
-      <dynamics damping="1.0" friction="1.0"/>
+      <dynamics damping="0.0" friction="0.0"/>
     </joint>
     <!-- Robotiq: left_finger -->
@@ -171,5 +171,5 @@
       <child link="robotiq_85_left_finger_link"/>
       <origin xyz="-0.00408552455 -0.03148604435 0.0" rpy="0 0 0" />
-      <dynamics damping="1.0" friction="1.0"/>
+      <dynamics damping="0.0" friction="0.0"/>
     </joint>
     <!-- Robotiq: right_finger -->
@@ -197,5 +197,5 @@
       <child link="robotiq_85_right_finger_link"/>
       <origin xyz="-0.00408552455 -0.03148604435 0.0" rpy="0 0 0" />
-      <dynamics damping="1.0" friction="1.0"/>
+      <dynamics damping="0.0" friction="0.0"/>
     </joint>
     <!-- Robotiq: left_inner_knuckle -->
@@ -225,5 +225,5 @@
       <origin xyz="0.06142 0.0127 0" rpy="${pi} 0.0 0.0" />
       <limit lower="-0.05" upper="0.80285" velocity="0.5" effort="1000"/>
-      <dynamics damping="1.0" friction="1.0"/>
+      <dynamics damping="0.0" friction="0.0"/>
     </joint>
     <!-- Robotiq: right_inner_knuckle -->
@@ -253,5 +253,5 @@
       <origin xyz="0.06142 -0.0127 0" rpy="0 0 0"/>
       <limit lower="-0.05" upper="0.80285" velocity="0.5" effort="1000"/>
-      <dynamics damping="1.0" friction="1.0"/>
+      <dynamics damping="0.0" friction="0.0"/>
     </joint>
     <!-- Robotiq: left_finger_tip -->
@@ -281,5 +281,5 @@
       <origin xyz="0.04303959807 -0.03759940821 0.0" rpy="0.0 0.0 0.0"/>
       <limit lower="-0.80285" upper="0.05" velocity="0.5" effort="1000"/>
-      <dynamics damping="1.0" friction="1.0"/>
+      <dynamics damping="0.0" friction="0.0"/>
     </joint>
     <!-- Robotiq: right_finger_tip -->
@@ -309,5 +309,5 @@
       <origin rpy="0.0 0.0 0.0" xyz="0.04303959807 -0.03759940821  0.0"/>
       <limit lower="-0.80285" upper="0.05" velocity="0.5" effort="1000"/>
-      <dynamics damping="1.0" friction="1.0"/>
+      <dynamics damping="0.0" friction="0.0"/>
     </joint>
     <!-- SMALL CUBE FOR GRIPPER PLUGIN -->

File: ros2srrc_endeffectors/robotiq_hande/urdf/robotiq_hande_macro.urdf.xacro (robot description, xacro)
@@ -67,4 +67,7 @@
           <mesh filename="file://$(find ros2srrc_endeffectors)/robotiq_hande/meshes/robotiq_hande_coupler.stl" />
         </geometry>
+        <material name="dark_grey">
+          <color rgba="0.2 0.2 0.2 1"/>
+        </material>
       </visual>
       <collision>
@@ -121,5 +124,5 @@
         <origin rpy="0 0 0" xyz="0.02262 -0.00759 0.00738"/>
         <mass value="0.03804"/>
-        <inertia ixx="13567E-9" ixy="1849E-9" ixz="3622E-9" iyy="15784E-9" iyz="3616E-9" izz="7478E-9"/>
+        <inertia ixx="1.3567e-05" ixy="0" ixz="0" iyy="1.5784e-05" iyz="0" izz="7.478e-06"/>
       </inertial>
       <visual>
@@ -128,4 +131,7 @@
           <mesh filename="file://$(find ros2srrc_endeffectors)/robotiq_hande/meshes/finger_1.dae"/>
         </geometry>
+        <material name="dark_grey">
+          <color rgba="0.2 0.2 0.2 1"/>
+        </material>
       </visual>
       <collision>
@@ -136,7 +142,4 @@
       </collision>
     </link>
-    <gazebo reference="robotiq_hande_left_finger">
-      <material>Gazebo/Grey</material>
-    </gazebo>
     <joint name="robotiq_hande_left_finger_joint" type="prismatic">
       <origin rpy="0 0 0" xyz="0.0 0.0 0.099"/>
@@ -151,5 +154,5 @@
         <origin rpy="0 0 0" xyz="-0.02262 0.00759 0.00738"/>
         <mass value="0.03804"/>
-        <inertia ixx="13567E-9" ixy="1849E-9" ixz="3622E-9" iyy="15784E-9" iyz="3616E-9" izz="7478E-9"/>
+        <inertia ixx="1.3567e-05" ixy="0" ixz="0" iyy="1.5784e-05" iyz="0" izz="7.478e-06"/>
       </inertial>
       <visual>
@@ -158,4 +161,7 @@
           <mesh filename="file://$(find ros2srrc_endeffectors)/robotiq_hande/meshes/finger_2.dae"/>
         </geometry>
+        <material name="dark_grey">
+          <color rgba="0.2 0.2 0.2 1"/>
+        </material>
       </visual>
       <collision>
@@ -166,7 +172,4 @@
       </collision>
     </link>
-    <gazebo reference="robotiq_hande_right_finger">
-      <material>Gazebo/Grey</material>
-    </gazebo>
     <joint name="robotiq_hande_right_finger_joint" type="prismatic">
       <origin rpy="0 0 0" xyz="0 0 0.099"/>

File: ros2srrc_endeffectors/robotiq_hande/urdf/robotiq_handev2_macro.urdf.xacro (robot description, xacro)
@@ -67,4 +67,7 @@
           <mesh filename="file://$(find ros2srrc_endeffectors)/robotiq_hande/meshes/robotiq_hande_coupler.stl" />
         </geometry>
+        <material name="dark_grey">
+          <color rgba="0.2 0.2 0.2 1"/>
+        </material>
       </visual>
       <collision>
@@ -85,9 +88,4 @@
       <child link="robotiq_coupler"/>
     </joint>
-    <gazebo reference="robotiq_coupler">
-      <mu1>0.9</mu1>
-      <mu2>0.9</mu2>
-      <material>Gazebo/FlatBlack</material>
-    </gazebo>
     <!-- Robotiq: base_link -->
     <link name="robotiq_hande_base_link">
@@ -121,5 +119,5 @@
         <origin rpy="0 0 0" xyz="0.02262 -0.00759 0.00738"/>
         <mass value="0.03804"/>
-        <inertia ixx="13567E-9" ixy="1849E-9" ixz="3622E-9" iyy="15784E-9" iyz="3616E-9" izz="7478E-9"/>
+        <inertia ixx="1.3567e-05" ixy="0" ixz="0" iyy="1.5784e-05" iyz="0" izz="7.478e-06"/>
       </inertial>
       <visual>
@@ -128,4 +126,7 @@
           <mesh filename="file://$(find ros2srrc_endeffectors)/robotiq_hande/meshes/finger_1v2.dae"/>
         </geometry>
+        <material name="dark_grey">
+          <color rgba="0.2 0.2 0.2 1"/>
+        </material>
       </visual>
       <collision>
@@ -136,7 +137,4 @@
       </collision>
     </link>
-    <gazebo reference="robotiq_hande_left_finger">
-      <material>Gazebo/Grey</material>
-    </gazebo>
     <joint name="robotiq_hande_left_finger_joint" type="prismatic">
       <origin rpy="0 0 0" xyz="0.0 0.0 0.099"/>
@@ -151,5 +149,5 @@
         <origin rpy="0 0 0" xyz="-0.02262 0.00759 0.00738"/>
         <mass value="0.03804"/>
-        <inertia ixx="13567E-9" ixy="1849E-9" ixz="3622E-9" iyy="15784E-9" iyz="3616E-9" izz="7478E-9"/>
+        <inertia ixx="1.3567e-05" ixy="0" ixz="0" iyy="1.5784e-05" iyz="0" izz="7.478e-06"/>
       </inertial>
       <visual>
@@ -158,4 +156,7 @@
           <mesh filename="file://$(find ros2srrc_endeffectors)/robotiq_hande/meshes/finger_2v2.dae"/>
         </geometry>
+        <material name="dark_grey">
+          <color rgba="0.2 0.2 0.2 1"/>
+        </material>
       </visual>
       <collision>
@@ -166,7 +167,4 @@
       </collision>
     </link>
-    <gazebo reference="robotiq_hande_right_finger">
-      <material>Gazebo/Grey</material>
-    </gazebo>
     <joint name="robotiq_hande_right_finger_joint" type="prismatic">
       <origin rpy="0 0 0" xyz="0 0 0.099"/>

File: ros2srrc_robots/irb120/urdf/irb120_macro.urdf.xacro (robot description, xacro)
@@ -223,5 +223,5 @@
       <limit effort="1000" lower="-2.87979" upper="2.87979" velocity="4.36332"/>
       <axis xyz="0 0 1"/>
-      <dynamics damping="50.0" friction="1.0"/>
+      <dynamics damping="0.0" friction="0.0"/>
     </joint>
     <!-- joint_2 -->
@@ -232,5 +232,5 @@
       <limit effort="1000" lower="-1.91986" upper="1.91986" velocity="4.36332"/>
       <axis xyz="0 1 0"/>
-      <dynamics damping="50.0" friction="1.0"/>
+      <dynamics damping="0.0" friction="0.0"/>
     </joint>
     <!-- joint_3 -->
@@ -241,5 +241,5 @@
       <limit effort="1000" lower="-1.91986" upper="1.22173" velocity="4.36332"/>
       <axis xyz="0 1 0"/>
-      <dynamics damping="10.0" friction="1.0"/>
+      <dynamics damping="0.0" friction="0.0"/>
     </joint>
     <!-- joint_4 -->
@@ -250,5 +250,5 @@
       <limit effort="1000" lower="-2.79253" upper="2.79253" velocity="5.58505"/>
       <axis xyz="1 0 0"/>
-      <dynamics damping="5.0" friction="1.0"/>
+      <dynamics damping="0.0" friction="0.0"/>
     </joint>
     <!-- joint_5 -->
@@ -259,5 +259,5 @@
       <limit effort="1000" lower="-2.094395" upper="2.094395" velocity="5.58505"/>
       <axis xyz="0 1 0"/>
-      <dynamics damping="2.0" friction="1.0"/>
+      <dynamics damping="0.0" friction="0.0"/>
     </joint>
     <!-- joint_6 -->
@@ -268,5 +268,5 @@
       <limit effort="1000" lower="-6.98132" upper="6.98132" velocity="7.33038"/>
       <axis xyz="1 0 0"/>
-      <dynamics damping="1.0" friction="1.0"/>
+      <dynamics damping="0.0" friction="0.0"/>
     </joint>
     <!-- end of joint list -->

Commit message: Fix: EGP64 gripper urdf (limits and physics).

File: ros2srrc_endeffectors/egp64/urdf/egp64_macro.urdf.xacro (robot description, xacro)
@@ -116,8 +116,8 @@
       <parent link="egp64_gripper_base_link" />
       <child link="egp64_finger_left_link" />
-      <limit effort="1000" lower="-0.001" upper="0.04" velocity="0.2"/>
+      <limit effort="1000" lower="-0.0001" upper="0.027" velocity="0.2"/>
       <origin xyz="0.01483 -0.00782 0" rpy="0 0 0" />
       <axis xyz="-1 0 0" />
-      <dynamics damping="0.0" friction="0.0"/>
+      <dynamics damping="0.2" friction="0.05"/>
     </joint>
     <!-- LEFT FINGERTIP -->
@@ -171,8 +171,8 @@
       <parent link="egp64_gripper_base_link" />
       <child link="egp64_finger_right_link" />
-      <limit effort="1000" lower="-0.001" upper="0.04" velocity="0.2"/>
+      <limit effort="1000" lower="-0.0001" upper="0.027" velocity="0.2"/>
       <origin xyz="-0.0153 -0.00602 0" rpy="0 0 0" />
       <axis xyz="1 0 0" />
-      <dynamics damping="0.0" friction="0.0"/>
+      <dynamics damping="0.2" friction="0.05"/>
     </joint>
     <!-- RIGHT FINGERTIP -->

File: ros2srrc_endeffectors/egp64/urdf/egp64_ros2control.xacro (robot description, xacro)
@@ -33,10 +33,6 @@
     <joint name="egp64_finger_left_joint">
       <command_interface name="position">
-        <param name="min">-0.001</param>
-        <param name="max">0.04</param>
-      </command_interface>
-      <command_interface name="velocity">
-        <param name="min">-0.2</param>
-        <param name="max">0.2</param>
+        <param name="min">-0.0001</param>
+        <param name="max">0.027</param>
       </command_interface>
       <state_interface name="position">
@@ -48,10 +44,6 @@
     <joint name="egp64_finger_right_joint">
       <command_interface name="position">
-        <param name="min">-0.001</param>
-        <param name="max">0.04</param>
-      </command_interface>
-      <command_interface name="velocity">
-        <param name="min">-0.2</param>
-        <param name="max">0.2</param>
+        <param name="min">-0.0001</param>
+        <param name="max">0.027</param>
       </command_interface>
       <state_interface name="position">

File: ros2srrc_endeffectors/egp64/urdf/egp64v2_macro.urdf.xacro (robot description, xacro)
@@ -116,8 +116,8 @@
       <parent link="egp64_gripper_base_link" />
       <child link="egp64_finger_left_link" />
-      <limit effort="1000" lower="-0.001" upper="0.04" velocity="0.2"/>
+      <limit effort="1000" lower="-0.0001" upper="0.027" velocity="0.2"/>
       <origin xyz="0.01483 -0.00782 0" rpy="0 0 0" />
       <axis xyz="-1 0 0" />
-      <dynamics damping="1.0" friction="1.0"/>
+      <dynamics damping="0.2" friction="0.05"/>
     </joint>
     <!-- LEFT FINGERTIP -->
@@ -171,8 +171,8 @@
       <parent link="egp64_gripper_base_link" />
       <child link="egp64_finger_right_link" />
-      <limit effort="1000" lower="-0.001" upper="0.04" velocity="0.2"/>
+      <limit effort="1000" lower="-0.0001" upper="0.027" velocity="0.2"/>
       <origin xyz="-0.0153 -0.00602 0" rpy="0 0 0" />
       <axis xyz="1 0 0" />
-      <dynamics damping="1.0" friction="1.0"/>
+      <dynamics damping="0.2" friction="0.05"/>
     </joint>
     <!-- RIGHT FINGERTIP -->

File: ros2srrc_endeffectors/egp64/urdf/egp64v3_macro.urdf.xacro (robot description, xacro)
@@ -116,8 +116,8 @@
       <parent link="egp64_gripper_base_link" />
       <child link="egp64_finger_left_link" />
-      <limit effort="1000" lower="-0.001" upper="0.04" velocity="0.2"/>
+      <limit effort="1000" lower="-0.0001" upper="0.027" velocity="0.2"/>
       <origin xyz="0.01483 -0.00782 0" rpy="0 0 0" />
       <axis xyz="-1 0 0" />
-      <dynamics damping="1.0" friction="1.0"/>
+      <dynamics damping="0.2" friction="0.05"/>
     </joint>
     <!-- LEFT FINGERTIP -->
@@ -171,8 +171,8 @@
       <parent link="egp64_gripper_base_link" />
       <child link="egp64_finger_right_link" />
-      <limit effort="1000" lower="-0.001" upper="0.04" velocity="0.2"/>
+      <limit effort="1000" lower="-0.0001" upper="0.027" velocity="0.2"/>
       <origin xyz="-0.0153 -0.00602 0" rpy="0 0 0" />
       <axis xyz="1 0 0" />
-      <dynamics damping="1.0" friction="1.0"/>
+      <dynamics damping="0.2" friction="0.05"/>
     </joint>
     <!-- RIGHT FINGERTIP -->

Commit message: Fix: EGP-64 inertia/mass values.

File: ros2srrc_endeffectors/egp64/urdf/egp64_macro.urdf.xacro (robot description, xacro)
@@ -51,6 +51,8 @@
       <inertial>
         <origin xyz="0 0 0" rpy="0 0 ${pi/2}" />
-        <mass value="0.001" />
-        <inertia ixx="0.001" ixy="0.0" ixz="0.0" iyy="0.001" iyz="0.0" izz="0.001"/>
+        <mass value="0.03"/>
+        <inertia ixx="4.09e-06" ixy="0.0" ixz="0.0"
+                iyy="4.09e-06" iyz="0.0"
+                izz="8.00e-06"/>
       </inertial>
     </link>
@@ -68,7 +70,9 @@
     <link name="egp64_gripper_base_link">
       <inertial>
-        <origin xyz="0 0 0" rpy="0 0 0" />
-        <mass value="0.005" />
-        <inertia ixx="0.001" ixy="0.0" ixz="0.0" iyy="0.001" iyz="0.0" izz="0.001"/>
+        <origin xyz="0 0 0" rpy="0 0 0"/>
+        <mass value="0.72"/>
+        <inertia ixx="9.375e-04" ixy="0.0" ixz="0.0"
+                iyy="1.10976e-03" iyz="0.0"
+                izz="3.1926e-04"/>
       </inertial>
       <visual>
@@ -95,6 +99,8 @@
       <inertial>
         <origin xyz="0.01483 -0.00782 0" rpy="0 0 0" />
-        <mass value="0.002" />
-        <inertia ixx="0.001" ixy="0.0" ixz="0.0" iyy="0.001" iyz="0.0" izz="0.001"/>
+        <mass value="0.02"/>
+        <inertia ixx="3.47e-07" ixy="0.0" ixz="0.0"
+                iyy="2.77e-06" iyz="0.0"
+                izz="2.91e-06"/>
       </inertial>
       <visual>
@@ -110,5 +116,4 @@
           <mesh filename="file://$(find ros2srrc_endeffectors)/egp64/meshes/egp64_LeftFingerBase.dae" />
         </geometry>
-        <material name="black" />
       </collision>
     </link>
@@ -125,6 +130,8 @@
       <inertial>
         <origin xyz="0.03869 -0.0005 0.00093" rpy="0 0 0" />
-        <mass value="0.001" />
-        <inertia ixx="0.001" ixy="0.0" ixz="0.0" iyy="0.001" iyz="0.0" izz="0.001"/>
+        <mass value="0.005"/>
+        <inertia ixx="3.71e-08" ixy="0.0" ixz="0.0"
+                iyy="1.77e-07" iyz="0.0"
+                izz="1.93e-07"/>
       </inertial>
       <visual>
@@ -140,5 +147,4 @@
           <mesh filename="file://$(find ros2srrc_endeffectors)/egp64/meshes/egp64_LeftFinger.dae" />
         </geometry>
-        <material name="black"/>
       </collision>
     </link>
@@ -152,6 +158,8 @@
       <inertial>
         <origin xyz="-0.0153 -0.00602 0" rpy="0 0 0" />
-        <mass value="0.002" />
-        <inertia ixx="0.001" ixy="0.0" ixz="0.0" iyy="0.001" iyz="0.0" izz="0.001"/>
+        <mass value="0.02"/>
+        <inertia ixx="3.47e-07" ixy="0.0" ixz="0.0"
+                iyy="2.77e-06" iyz="0.0"
+                izz="2.91e-06"/>
       </inertial>
       <visual>
@@ -165,5 +173,4 @@
           <mesh filename="file://$(find ros2srrc_endeffectors)/egp64/meshes/egp64_RightFingerBase.dae" />
         </geometry>
-        <material name="black"/>
       </collision>
     </link>
@@ -180,6 +187,8 @@
       <inertial>
         <origin xyz="-0.01211 -0.00197 0.00093" rpy="0 0 0" />
-        <mass value="0.001" />
-        <inertia ixx="0.001" ixy="0.0" ixz="0.0" iyy="0.001" iyz="0.0" izz="0.001"/>
+        <mass value="0.005"/>
+        <inertia ixx="3.71e-08" ixy="0.0" ixz="0.0"
+                iyy="1.77e-07" iyz="0.0"
+                izz="1.93e-07"/>
       </inertial>
       <visual>
@@ -193,5 +202,4 @@
           <mesh filename="file://$(find ros2srrc_endeffectors)/egp64/meshes/egp64_RightFinger.dae" />
         </geometry>
-        <material name="black"/>
       </collision>
     </link>
