Commit message: Fix end-effector joint limits + add open/half/full poses in srdf.

File: ros2srrc_endeffectors/egp64/urdf/egp64_macro.urdf.xacro (robot description, xacro)
@@ -117,5 +117,5 @@
       <parent link="egp64_gripper_base_link" />
       <child link="egp64_finger_left_link" />
-      <limit effort="1000" lower="-0.001" upper="0.04" velocity="0.2"/>
+      <limit effort="1000" lower="-0.0001" upper="0.0271" velocity="0.2"/>
       <origin xyz="0.01483 -0.00782 0" rpy="0 0 0" />
       <axis xyz="-1 0 0" />
@@ -172,5 +172,5 @@
       <parent link="egp64_gripper_base_link" />
       <child link="egp64_finger_right_link" />
-      <limit effort="1000" lower="-0.001" upper="0.04" velocity="0.2"/>
+      <limit effort="1000" lower="-0.0001" upper="0.0271" velocity="0.2"/>
       <origin xyz="-0.0153 -0.00602 0" rpy="0 0 0" />
       <axis xyz="1 0 0" />

File: ros2srrc_endeffectors/egp64/urdf/egp64_ros2control.xacro (robot description, xacro)
@@ -33,6 +33,6 @@
     <joint name="egp64_finger_left_joint">
       <command_interface name="position">
-        <param name="min">-0.001</param>
-        <param name="max">0.04</param>
+        <param name="min">-0.0001</param>
+        <param name="max">0.0271</param>
       </command_interface>
       <command_interface name="velocity">
@@ -48,6 +48,6 @@
     <joint name="egp64_finger_right_joint">
       <command_interface name="position">
-        <param name="min">-0.001</param>
-        <param name="max">0.04</param>
+        <param name="min">-0.0001</param>
+        <param name="max">0.0271</param>
       </command_interface>
       <command_interface name="velocity">

File: ros2srrc_endeffectors/egp64/urdf/egp64v2_macro.urdf.xacro (robot description, xacro)
@@ -117,5 +117,5 @@
       <parent link="egp64_gripper_base_link" />
       <child link="egp64_finger_left_link" />
-      <limit effort="1000" lower="-0.001" upper="0.04" velocity="0.2"/>
+      <limit effort="1000" lower="-0.0001" upper="0.0271" velocity="0.2"/>
       <origin xyz="0.01483 -0.00782 0" rpy="0 0 0" />
       <axis xyz="-1 0 0" />
@@ -172,5 +172,5 @@
       <parent link="egp64_gripper_base_link" />
       <child link="egp64_finger_right_link" />
-      <limit effort="1000" lower="-0.001" upper="0.04" velocity="0.2"/>
+      <limit effort="1000" lower="-0.0001" upper="0.0271" velocity="0.2"/>
       <origin xyz="-0.0153 -0.00602 0" rpy="0 0 0" />
       <axis xyz="1 0 0" />

File: ros2srrc_endeffectors/egp64/urdf/egp64v3_macro.urdf.xacro (robot description, xacro)
@@ -117,5 +117,5 @@
       <parent link="egp64_gripper_base_link" />
       <child link="egp64_finger_left_link" />
-      <limit effort="1000" lower="-0.001" upper="0.04" velocity="0.2"/>
+      <limit effort="1000" lower="-0.0001" upper="0.0271" velocity="0.2"/>
       <origin xyz="0.01483 -0.00782 0" rpy="0 0 0" />
       <axis xyz="-1 0 0" />
@@ -172,5 +172,5 @@
       <parent link="egp64_gripper_base_link" />
       <child link="egp64_finger_right_link" />
-      <limit effort="1000" lower="-0.001" upper="0.04" velocity="0.2"/>
+      <limit effort="1000" lower="-0.0001" upper="0.0271" velocity="0.2"/>
       <origin xyz="-0.0153 -0.00602 0" rpy="0 0 0" />
       <axis xyz="1 0 0" />

File: ros2srrc_endeffectors/robotiq_hande/urdf/robotiq_hande_macro.urdf.xacro (robot description, xacro)
@@ -144,5 +144,5 @@
       <child link="robotiq_hande_left_finger"/>
       <axis xyz="-1 0 0"/>
-      <limit effort="130" lower="-0.05" upper="0.025" velocity="0.15"/>
+      <limit effort="130" lower="-0.0001" upper="0.0251" velocity="0.15"/>
     </joint>
     <!-- Robotiq: right finger -->
@@ -174,5 +174,5 @@
       <child link="robotiq_hande_right_finger"/>
       <axis xyz="1 0 0"/>
-      <limit effort="130" lower="-0.05" upper="0.025" velocity="0.15"/>
+      <limit effort="130" lower="-0.0001" upper="0.0251" velocity="0.15"/>
     </joint>
     <!-- SMALL CUBE FOR GRIPPER PLUGIN -->

File: ros2srrc_endeffectors/robotiq_hande/urdf/robotiq_handev2_macro.urdf.xacro (robot description, xacro)
@@ -144,5 +144,5 @@
       <child link="robotiq_hande_left_finger"/>
       <axis xyz="-1 0 0"/>
-      <limit effort="130" lower="-0.05" upper="0.025" velocity="0.15"/>
+      <limit effort="130" lower="-0.0001" upper="0.0251" velocity="0.15"/>
     </joint>
     <!-- Robotiq: right finger -->
@@ -174,5 +174,5 @@
       <child link="robotiq_hande_right_finger"/>
       <axis xyz="1 0 0"/>
-      <limit effort="130" lower="-0.05" upper="0.025" velocity="0.15"/>
+      <limit effort="130" lower="-0.0001" upper="0.0251" velocity="0.15"/>
     </joint>
     <!-- SMALL CUBE FOR GRIPPER PLUGIN -->
