Commit message: Migrate to GzFortress: Staubli RX-160.

File: ros2srrc_robots/rx160/urdf/rx160_macro.urdf.xacro (robot description, xacro)
@@ -73,9 +73,9 @@
         <origin xyz="0 0 0" rpy="0 0 0"/>
         <geometry>
-          <mesh filename="file://$(find ros2srrc_robots)/rx160/meshes/visual/base_link.stl"/>
-        </geometry>
-        <material name="base_link_material">
-          <color rgba="1.0 0.607843137255 0.0 1.0"/>
-        </material>
+          <mesh filename="file://$(find ros2srrc_robots)/rx160/meshes/visual/base_link.dae"/>
+        </geometry>
+        <!--<material name="base_link_material">
+          <color rgba="1.0 0.607843137255 0.0 1.0"/>
+        </material>-->
       </visual>
       <collision>
@@ -96,9 +96,9 @@
         <origin xyz="0 0 0" rpy="0 0 0"/>
         <geometry>
-          <mesh filename="file://$(find ros2srrc_robots)/rx160/meshes/visual/link_1.stl"/>
-        </geometry>
-        <material name="link_1_material">
-          <color rgba="1.0 0.607843137255 0.0 1.0"/>
-        </material>
+          <mesh filename="file://$(find ros2srrc_robots)/rx160/meshes/visual/link_1.dae"/>
+        </geometry>
+        <!--<material name="link_1_material">
+          <color rgba="1.0 0.607843137255 0.0 1.0"/>
+        </material>-->
       </visual>
       <collision>
@@ -119,9 +119,9 @@
         <origin xyz="0 0 0" rpy="0 0 0"/>
         <geometry>
-          <mesh filename="file://$(find ros2srrc_robots)/rx160/meshes/visual/link_2.stl"/>
-        </geometry>
-        <material name="link_2_material">
-          <color rgba="1.0 0.607843137255 0.0 1.0"/>
-        </material>
+          <mesh filename="file://$(find ros2srrc_robots)/rx160/meshes/visual/link_2.dae"/>
+        </geometry>
+        <!--<material name="link_2_material">
+          <color rgba="1.0 0.607843137255 0.0 1.0"/>
+        </material>-->
       </visual>
       <collision>
@@ -142,9 +142,9 @@
         <origin xyz="0 0 0" rpy="0 0 0"/>
         <geometry>
-          <mesh filename="file://$(find ros2srrc_robots)/rx160/meshes/visual/link_3.stl"/>
-        </geometry>
-        <material name="link_3_material">
-          <color rgba="1.0 0.607843137255 0.0 1.0"/>
-        </material>
+          <mesh filename="file://$(find ros2srrc_robots)/rx160/meshes/visual/link_3.dae"/>
+        </geometry>
+        <!--<material name="link_3_material">
+          <color rgba="1.0 0.607843137255 0.0 1.0"/>
+        </material>-->
       </visual>
       <collision>
@@ -165,9 +165,9 @@
         <origin xyz="0 0 0" rpy="0 0 0"/>
         <geometry>
-          <mesh filename="file://$(find ros2srrc_robots)/rx160/meshes/visual/link_4.stl"/>
-        </geometry>
-        <material name="link_4_material">
-          <color rgba="1.0 0.607843137255 0.0 1.0"/>
-        </material>
+          <mesh filename="file://$(find ros2srrc_robots)/rx160/meshes/visual/link_4.dae"/>
+        </geometry>
+        <!--<material name="link_4_material">
+          <color rgba="1.0 0.607843137255 0.0 1.0"/>
+        </material>-->
       </visual>
       <collision>
@@ -188,9 +188,9 @@
         <origin xyz="0 0 0" rpy="0 0 0"/>
         <geometry>
-          <mesh filename="file://$(find ros2srrc_robots)/rx160/meshes/visual/link_5.stl"/>
-        </geometry>
-        <material name="link_5_material">
+          <mesh filename="file://$(find ros2srrc_robots)/rx160/meshes/visual/link_5.dae"/>
+        </geometry>
+        <!--<material name="link_5_material">
           <color rgba="0.529411764706 0.521568627451 0.505882352941 1.0"/>
-        </material>
+        </material>-->
       </visual>
       <collision>
@@ -211,9 +211,9 @@
         <origin xyz="0 0 0" rpy="0 0 0"/>
         <geometry>
-          <mesh filename="file://$(find ros2srrc_robots)/rx160/meshes/visual/link_6.stl"/>
-        </geometry>
-        <material name="link_6_material">
+          <mesh filename="file://$(find ros2srrc_robots)/rx160/meshes/visual/link_6.dae"/>
+        </geometry>
+        <!--<material name="link_6_material">
           <color rgba="0.529411764706 0.521568627451 0.505882352941 1.0"/>
-        </material>
+        </material>-->
       </visual>
       <collision>
@@ -232,5 +232,4 @@
       <axis xyz="0 0 1"/>
       <limit effort="692.0" lower="-2.967060" upper="2.967060" velocity="2.88"/>
-      <dynamics damping="0.0" friction="0.0"/>
     </joint>
     <joint name="joint_2" type="revolute">
@@ -240,5 +239,4 @@
       <axis xyz="0 1 0"/>
       <limit effort="574.0" lower="-2.4" upper="2.4" velocity="2.62"/>
-      <dynamics damping="0.0" friction="0.0"/>
     </joint>
     <joint name="joint_3" type="revolute">
@@ -248,5 +246,4 @@
       <axis xyz="0 1 0"/>
       <limit effort="242.0" lower="-2.62" upper="2.62" velocity="3.32"/>
-      <dynamics damping="0.0" friction="0.0"/>
     </joint>
     <joint name="joint_4" type="revolute">
@@ -256,5 +253,4 @@
       <axis xyz="0 0 1"/>
       <limit effort="58.0" lower="-4.71" upper="4.71" velocity="5.15"/>
-      <dynamics damping="0.0" friction="0.0"/>
     </joint>
     <joint name="joint_5" type="revolute">
@@ -264,5 +260,4 @@
       <axis xyz="0 1 0"/>
       <limit effort="29.0" lower="-1.83" upper="2.09" velocity="4.54"/>
-      <dynamics damping="0.0" friction="0.0"/>
     </joint>
     <joint name="joint_6" type="revolute">
@@ -272,5 +267,4 @@
       <axis xyz="0 0 1"/>
       <limit effort="29.0" lower="-4.71" upper="4.71" velocity="7.68"/>
-      <dynamics damping="0.0" friction="0.0"/>
     </joint>
     <!-- end of joint list -->

File: ros2srrc_robots/rx160/urdf/rx160_ros2control.xacro (robot description, xacro)
@@ -50,5 +50,5 @@
     <!-- A. GAZEBO SIMULATION: -->
     <xacro:unless value="${bringup}">
-      <xacro:property name="name" value="GazeboSystem"/>
+      <xacro:property name="name" value="GazeboSimSystem"/>
     </xacro:unless>
     <!-- B. ROBOT BRINGUP:
@@ -61,5 +61,5 @@
       <xacro:unless value="${bringup}">
         <hardware>
-          <plugin>gazebo_ros2_control/GazeboSystem</plugin>
+          <plugin>gz_ros2_control/GazeboSimSystem</plugin>
         </hardware>
       </xacro:unless>

Commit message: Add some damping for joint stability in GzFortress.

File: ros2srrc_robots/rx160/urdf/rx160_macro.urdf.xacro (robot description, xacro)
@@ -232,4 +232,5 @@
       <axis xyz="0 0 1"/>
       <limit effort="692.0" lower="-2.967060" upper="2.967060" velocity="2.88"/>
+      <dynamics damping="0.3" friction="0.0"/>
     </joint>
     <joint name="joint_2" type="revolute">
@@ -239,4 +240,5 @@
       <axis xyz="0 1 0"/>
       <limit effort="574.0" lower="-2.4" upper="2.4" velocity="2.62"/>
+      <dynamics damping="0.3" friction="0.0"/>
     </joint>
     <joint name="joint_3" type="revolute">
@@ -246,4 +248,5 @@
       <axis xyz="0 1 0"/>
       <limit effort="242.0" lower="-2.62" upper="2.62" velocity="3.32"/>
+      <dynamics damping="0.3" friction="0.0"/>
     </joint>
     <joint name="joint_4" type="revolute">
@@ -253,4 +256,5 @@
       <axis xyz="0 0 1"/>
       <limit effort="58.0" lower="-4.71" upper="4.71" velocity="5.15"/>
+      <dynamics damping="0.1" friction="0.0"/>
     </joint>
     <joint name="joint_5" type="revolute">
@@ -260,4 +264,5 @@
       <axis xyz="0 1 0"/>
       <limit effort="29.0" lower="-1.83" upper="2.09" velocity="4.54"/>
+      <dynamics damping="0.05" friction="0.0"/>
     </joint>
     <joint name="joint_6" type="revolute">
@@ -267,4 +272,5 @@
       <axis xyz="0 0 1"/>
       <limit effort="29.0" lower="-4.71" upper="4.71" velocity="7.68"/>
+      <dynamics damping="0.01" friction="0.0"/>
     </joint>
     <!-- end of joint list -->

Commit message: Fix: Staubli RX-160 visual .dae files.

File: ros2srrc_robots/rx160/urdf/rx160_macro.urdf.xacro (robot description, xacro)
@@ -73,5 +73,5 @@
         <origin xyz="0 0 0" rpy="0 0 0"/>
         <geometry>
-          <mesh filename="file://$(find ros2srrc_robots)/rx160/meshes/visual/base_link.stl"/>
+          <mesh filename="file://$(find ros2srrc_robots)/rx160/meshes/visual/base_link.dae"/>
         </geometry>
         <material name="base_link_material">
@@ -96,5 +96,5 @@
         <origin xyz="0 0 0" rpy="0 0 0"/>
         <geometry>
-          <mesh filename="file://$(find ros2srrc_robots)/rx160/meshes/visual/link_1.stl"/>
+          <mesh filename="file://$(find ros2srrc_robots)/rx160/meshes/visual/link_1.dae"/>
         </geometry>
         <material name="link_1_material">
@@ -119,5 +119,5 @@
         <origin xyz="0 0 0" rpy="0 0 0"/>
         <geometry>
-          <mesh filename="file://$(find ros2srrc_robots)/rx160/meshes/visual/link_2.stl"/>
+          <mesh filename="file://$(find ros2srrc_robots)/rx160/meshes/visual/link_2.dae"/>
         </geometry>
         <material name="link_2_material">
@@ -142,5 +142,5 @@
         <origin xyz="0 0 0" rpy="0 0 0"/>
         <geometry>
-          <mesh filename="file://$(find ros2srrc_robots)/rx160/meshes/visual/link_3.stl"/>
+          <mesh filename="file://$(find ros2srrc_robots)/rx160/meshes/visual/link_3.dae"/>
         </geometry>
         <material name="link_3_material">
@@ -165,5 +165,5 @@
         <origin xyz="0 0 0" rpy="0 0 0"/>
         <geometry>
-          <mesh filename="file://$(find ros2srrc_robots)/rx160/meshes/visual/link_4.stl"/>
+          <mesh filename="file://$(find ros2srrc_robots)/rx160/meshes/visual/link_4.dae"/>
         </geometry>
         <material name="link_4_material">
@@ -188,5 +188,5 @@
         <origin xyz="0 0 0" rpy="0 0 0"/>
         <geometry>
-          <mesh filename="file://$(find ros2srrc_robots)/rx160/meshes/visual/link_5.stl"/>
+          <mesh filename="file://$(find ros2srrc_robots)/rx160/meshes/visual/link_5.dae"/>
         </geometry>
         <material name="link_5_material">
@@ -211,5 +211,5 @@
         <origin xyz="0 0 0" rpy="0 0 0"/>
         <geometry>
-          <mesh filename="file://$(find ros2srrc_robots)/rx160/meshes/visual/link_6.stl"/>
+          <mesh filename="file://$(find ros2srrc_robots)/rx160/meshes/visual/link_6.dae"/>
         </geometry>
         <material name="link_6_material">
