Commit message: Fix ros2control name (add prefix) and add {prefix} to EE_ros2control file load.

File: ros2srrc_robots/ar4/urdf/ar4_ros2control.xacro (robot description, xacro)
@@ -49,5 +49,5 @@
     <!-- A. GAZEBO SIMULATION: -->
     <xacro:unless value="${bringup}">
-      <xacro:property name="name" value="GazeboSystem"/>
+      <xacro:property name="name" value="${prefix}GazeboSystem"/>
     </xacro:unless>
     <!-- B. ROBOT BRINGUP:
@@ -161,5 +161,5 @@
         <xacro:if value="${EE}">
           <xacro:include filename="$(find ros2srrc_endeffectors)/${EE_name}/urdf/${EE_name}_ros2control.xacro" />
-          <xacro:EE_ros2control prefix="" />
+          <xacro:EE_ros2control prefix="${prefix}" />
         </xacro:if>
       </xacro:unless>

File: ros2srrc_robots/iiwa/urdf/iiwa_ros2control.xacro (robot description, xacro)
@@ -52,9 +52,9 @@
     <!-- A. GAZEBO SIMULATION: -->
     <xacro:unless value="${bringup}">
-      <xacro:property name="name" value="GazeboSystem"/>
+      <xacro:property name="name" value="${prefix}GazeboSystem"/>
     </xacro:unless>
     <!-- B. ROBOT BRINGUP: -->
     <xacro:if value="${bringup}">
-      <xacro:property name="name" value="TBD"/>
+      <xacro:property name="name" value="${prefix}TBD"/>
     </xacro:if>
     <!-- 3. Load ROS2_CONTROL: -->
@@ -182,5 +182,5 @@
         <xacro:if value="${EE}">
           <xacro:include filename="$(find ros2srrc_endeffectors)/${EE_name}/urdf/${EE_name}_ros2control.xacro" />
-          <xacro:EE_ros2control prefix="" />
+          <xacro:EE_ros2control prefix="${prefix}" />
         </xacro:if>
       </xacro:unless>

File: ros2srrc_robots/irb120/urdf/irb120_ros2control.xacro (robot description, xacro)
@@ -52,9 +52,9 @@
     <!-- A. GAZEBO SIMULATION: -->
     <xacro:unless value="${bringup}">
-      <xacro:property name="name" value="GazeboSystem"/>
+      <xacro:property name="name" value="${prefix}GazeboSystem"/>
     </xacro:unless>
     <!-- B. ROBOT BRINGUP: -->
     <xacro:if value="${bringup}">
-      <xacro:property name="name" value="ABBMultiInterfaceHardware"/>
+      <xacro:property name="name" value="${prefix}ABBMultiInterfaceHardware"/>
     </xacro:if>
     <!-- 3. Load ROS2_CONTROL: -->
@@ -169,5 +169,5 @@
         <xacro:if value="${EE}">
           <xacro:include filename="$(find ros2srrc_endeffectors)/${EE_name}/urdf/${EE_name}_ros2control.xacro" />
-          <xacro:EE_ros2control prefix="" />
+          <xacro:EE_ros2control prefix="${prefix}" />
         </xacro:if>
       </xacro:unless>

File: ros2srrc_robots/irb1200/urdf/irb1200_ros2control.xacro (robot description, xacro)
@@ -52,9 +52,9 @@
     <!-- A. GAZEBO SIMULATION: -->
     <xacro:unless value="${bringup}">
-      <xacro:property name="name" value="GazeboSystem"/>
+      <xacro:property name="name" value="${prefix}GazeboSystem"/>
     </xacro:unless>
     <!-- B. ROBOT BRINGUP: -->
     <xacro:if value="${bringup}">
-      <xacro:property name="name" value="ABBMultiInterfaceHardware"/>
+      <xacro:property name="name" value="${prefix}ABBMultiInterfaceHardware"/>
     </xacro:if>
     <!-- 3. Load ROS2_CONTROL: -->
@@ -169,5 +169,5 @@
         <xacro:if value="${EE}">
           <xacro:include filename="$(find ros2srrc_endeffectors)/${EE_name}/urdf/${EE_name}_ros2control.xacro" />
-          <xacro:EE_ros2control prefix="" />
+          <xacro:EE_ros2control prefix="${prefix}" />
         </xacro:if>
       </xacro:unless>

File: ros2srrc_robots/irb1600/urdf/irb1600_ros2control.xacro (robot description, xacro)
@@ -52,9 +52,9 @@
     <!-- A. GAZEBO SIMULATION: -->
     <xacro:unless value="${bringup}">
-      <xacro:property name="name" value="GazeboSystem"/>
+      <xacro:property name="name" value="${prefix}GazeboSystem"/>
     </xacro:unless>
     <!-- B. ROBOT BRINGUP: -->
     <xacro:if value="${bringup}">
-      <xacro:property name="name" value="ABBMultiInterfaceHardware"/>
+      <xacro:property name="name" value="${prefix}ABBMultiInterfaceHardware"/>
     </xacro:if>
     <!-- 3. Load ROS2_CONTROL: -->
@@ -169,5 +169,5 @@
         <xacro:if value="${EE}">
           <xacro:include filename="$(find ros2srrc_endeffectors)/${EE_name}/urdf/${EE_name}_ros2control.xacro" />
-          <xacro:EE_ros2control prefix="" />
+          <xacro:EE_ros2control prefix="${prefix}" />
         </xacro:if>
       </xacro:unless>

File: ros2srrc_robots/irb6640/urdf/irb6640_ros2control.xacro (robot description, xacro)
@@ -52,9 +52,9 @@
     <!-- A. GAZEBO SIMULATION: -->
     <xacro:unless value="${bringup}">
-      <xacro:property name="name" value="GazeboSystem"/>
+      <xacro:property name="name" value="${prefix}GazeboSystem"/>
     </xacro:unless>
     <!-- B. ROBOT BRINGUP: -->
     <xacro:if value="${bringup}">
-      <xacro:property name="name" value="ABBMultiInterfaceHardware"/>
+      <xacro:property name="name" value="${prefix}ABBMultiInterfaceHardware"/>
     </xacro:if>
     <!-- 3. Load ROS2_CONTROL: -->
@@ -184,5 +184,5 @@
         <xacro:if value="${EE}">
           <xacro:include filename="$(find ros2srrc_endeffectors)/${EE_name}/urdf/${EE_name}_ros2control.xacro" />
-          <xacro:EE_ros2control prefix="" />
+          <xacro:EE_ros2control prefix="${prefix}" />
         </xacro:if>
       </xacro:unless>

File: ros2srrc_robots/rx160/urdf/rx160_ros2control.xacro (robot description, xacro)
@@ -50,9 +50,9 @@
     <!-- A. GAZEBO SIMULATION: -->
     <xacro:unless value="${bringup}">
-      <xacro:property name="name" value="GazeboSystem"/>
+      <xacro:property name="name" value="${prefix}GazeboSystem"/>
     </xacro:unless>
     <!-- B. ROBOT BRINGUP:
     <xacro:if value="${bringup}">
-      <xacro:property name="name" value=""/>
+      <xacro:property name="name" value="${prefix}"/>
     </xacro:if> -->
     <!-- 3. Load ROS2_CONTROL: -->
@@ -163,5 +163,5 @@
         <xacro:if value="${EE}">
           <xacro:include filename="$(find ros2srrc_endeffectors)/${EE_name}/urdf/${EE_name}_ros2control.xacro" />
-          <xacro:EE_ros2control prefix="" />
+          <xacro:EE_ros2control prefix="${prefix}" />
         </xacro:if>
       </xacro:unless>

File: ros2srrc_robots/ur10/urdf/ur10_ros2control.xacro (robot description, xacro)
@@ -102,9 +102,9 @@
     <!-- A. GAZEBO SIMULATION: -->
     <xacro:unless value="${bringup}">
-      <xacro:property name="name" value="GazeboSystem"/>
+      <xacro:property name="name" value="${prefix}GazeboSystem"/>
     </xacro:unless>
     <!-- B. ROBOT BRINGUP: -->
     <xacro:if value="${bringup}">
-      <xacro:property name="name" value="ur10"/>
+      <xacro:property name="name" value="${prefix}ur10"/>
     </xacro:if>
     <!-- Load ROS2_CONTROL: -->
@@ -279,5 +279,5 @@
         <xacro:if value="${EE}">
           <xacro:include filename="$(find ros2srrc_endeffectors)/${EE_name}/urdf/${EE_name}_ros2control.xacro" />
-          <xacro:EE_ros2control prefix="" />
+          <xacro:EE_ros2control prefix="${prefix}" />
         </xacro:if>
       </xacro:unless>

File: ros2srrc_robots/ur10e/urdf/ur10e_ros2control.xacro (robot description, xacro)
@@ -102,9 +102,9 @@
     <!-- A. GAZEBO SIMULATION: -->
     <xacro:unless value="${bringup}">
-      <xacro:property name="name" value="GazeboSystem"/>
+      <xacro:property name="name" value="${prefix}GazeboSystem"/>
     </xacro:unless>
     <!-- B. ROBOT BRINGUP: -->
     <xacro:if value="${bringup}">
-      <xacro:property name="name" value="ur10e"/>
+      <xacro:property name="name" value="${prefix}ur10e"/>
     </xacro:if>
     <!-- Load ROS2_CONTROL: -->
@@ -279,5 +279,5 @@
         <xacro:if value="${EE}">
           <xacro:include filename="$(find ros2srrc_endeffectors)/${EE_name}/urdf/${EE_name}_ros2control.xacro" />
-          <xacro:EE_ros2control prefix="" />
+          <xacro:EE_ros2control prefix="${prefix}" />
         </xacro:if>
       </xacro:unless>

File: ros2srrc_robots/ur16e/urdf/ur16e_ros2control.xacro (robot description, xacro)
@@ -102,9 +102,9 @@
     <!-- A. GAZEBO SIMULATION: -->
     <xacro:unless value="${bringup}">
-      <xacro:property name="name" value="GazeboSystem"/>
+      <xacro:property name="name" value="${prefix}GazeboSystem"/>
     </xacro:unless>
     <!-- B. ROBOT BRINGUP: -->
     <xacro:if value="${bringup}">
-      <xacro:property name="name" value="ur16e"/>
+      <xacro:property name="name" value="${prefix}ur16e"/>
     </xacro:if>
     <!-- Load ROS2_CONTROL: -->
@@ -279,5 +279,5 @@
         <xacro:if value="${EE}">
           <xacro:include filename="$(find ros2srrc_endeffectors)/${EE_name}/urdf/${EE_name}_ros2control.xacro" />
-          <xacro:EE_ros2control prefix="" />
+          <xacro:EE_ros2control prefix="${prefix}" />
         </xacro:if>
       </xacro:unless>

File: ros2srrc_robots/ur20/urdf/ur20_ros2control.xacro (robot description, xacro)
@@ -102,9 +102,9 @@
     <!-- A. GAZEBO SIMULATION: -->
     <xacro:unless value="${bringup}">
-      <xacro:property name="name" value="GazeboSystem"/>
+      <xacro:property name="name" value="${prefix}GazeboSystem"/>
     </xacro:unless>
     <!-- B. ROBOT BRINGUP: -->
     <xacro:if value="${bringup}">
-      <xacro:property name="name" value="ur20"/>
+      <xacro:property name="name" value="${prefix}ur20"/>
     </xacro:if>
     <!-- Load ROS2_CONTROL: -->
@@ -279,5 +279,5 @@
         <xacro:if value="${EE}">
           <xacro:include filename="$(find ros2srrc_endeffectors)/${EE_name}/urdf/${EE_name}_ros2control.xacro" />
-          <xacro:EE_ros2control prefix="" />
+          <xacro:EE_ros2control prefix="${prefix}" />
         </xacro:if>
       </xacro:unless>

File: ros2srrc_robots/ur3/urdf/ur3_ros2control.xacro (robot description, xacro)
@@ -102,9 +102,9 @@
     <!-- A. GAZEBO SIMULATION: -->
     <xacro:unless value="${bringup}">
-      <xacro:property name="name" value="GazeboSystem"/>
+      <xacro:property name="name" value="${prefix}GazeboSystem"/>
     </xacro:unless>
     <!-- B. ROBOT BRINGUP: -->
     <xacro:if value="${bringup}">
-      <xacro:property name="name" value="ur3"/>
+      <xacro:property name="name" value="${prefix}ur3"/>
     </xacro:if>
     <!-- Load ROS2_CONTROL: -->
@@ -279,5 +279,5 @@
         <xacro:if value="${EE}">
           <xacro:include filename="$(find ros2srrc_endeffectors)/${EE_name}/urdf/${EE_name}_ros2control.xacro" />
-          <xacro:EE_ros2control prefix="" />
+          <xacro:EE_ros2control prefix="${prefix}" />
         </xacro:if>
       </xacro:unless>

File: ros2srrc_robots/ur3e/urdf/ur3e_ros2control.xacro (robot description, xacro)
@@ -102,9 +102,9 @@
     <!-- A. GAZEBO SIMULATION: -->
     <xacro:unless value="${bringup}">
-      <xacro:property name="name" value="GazeboSystem"/>
+      <xacro:property name="name" value="${prefix}GazeboSystem"/>
     </xacro:unless>
     <!-- B. ROBOT BRINGUP: -->
     <xacro:if value="${bringup}">
-      <xacro:property name="name" value="ur3e"/>
+      <xacro:property name="name" value="${prefix}ur3e"/>
     </xacro:if>
     <!-- Load ROS2_CONTROL: -->
@@ -279,5 +279,5 @@
         <xacro:if value="${EE}">
           <xacro:include filename="$(find ros2srrc_endeffectors)/${EE_name}/urdf/${EE_name}_ros2control.xacro" />
-          <xacro:EE_ros2control prefix="" />
+          <xacro:EE_ros2control prefix="${prefix}" />
         </xacro:if>
       </xacro:unless>

File: ros2srrc_robots/ur5/urdf/ur5_ros2control.xacro (robot description, xacro)
@@ -102,9 +102,9 @@
     <!-- A. GAZEBO SIMULATION: -->
     <xacro:unless value="${bringup}">
-      <xacro:property name="name" value="GazeboSystem"/>
+      <xacro:property name="name" value="${prefix}GazeboSystem"/>
     </xacro:unless>
     <!-- B. ROBOT BRINGUP: -->
     <xacro:if value="${bringup}">
-      <xacro:property name="name" value="ur5"/>
+      <xacro:property name="name" value="${prefix}ur5"/>
     </xacro:if>
     <!-- Load ROS2_CONTROL: -->
@@ -279,5 +279,5 @@
         <xacro:if value="${EE}">
           <xacro:include filename="$(find ros2srrc_endeffectors)/${EE_name}/urdf/${EE_name}_ros2control.xacro" />
-          <xacro:EE_ros2control prefix="" />
+          <xacro:EE_ros2control prefix="${prefix}" />
         </xacro:if>
       </xacro:unless>

File: ros2srrc_robots/ur5e/urdf/ur5e_ros2control.xacro (robot description, xacro)
@@ -102,9 +102,9 @@
     <!-- A. GAZEBO SIMULATION: -->
     <xacro:unless value="${bringup}">
-      <xacro:property name="name" value="GazeboSystem"/>
+      <xacro:property name="name" value="${prefix}GazeboSystem"/>
     </xacro:unless>
     <!-- B. ROBOT BRINGUP: -->
     <xacro:if value="${bringup}">
-      <xacro:property name="name" value="ur5e"/>
+      <xacro:property name="name" value="${prefix}ur5e"/>
     </xacro:if>
     <!-- Load ROS2_CONTROL: -->
@@ -279,5 +279,5 @@
         <xacro:if value="${EE}">
           <xacro:include filename="$(find ros2srrc_endeffectors)/${EE_name}/urdf/${EE_name}_ros2control.xacro" />
-          <xacro:EE_ros2control prefix="" />
+          <xacro:EE_ros2control prefix="${prefix}" />
         </xacro:if>
       </xacro:unless>
