Commit message: Add {prefix} variable to allow multi-robot environments.

File: packages/ros2srrc_ur10/urdf/ur10.urdf.xacro (robot description, xacro)
@@ -39,4 +39,6 @@
   <xacro:arg name="EE_name" default="none"/>
   <xacro:property name="EE_name" value="$(arg EE_name)"/>
+  <xacro:arg name="prefix" default=""/>
+  <xacro:property name="prefix" value="$(arg prefix)"/>
   <!-- UR10 Control ARGUMENTS -->
   <xacro:arg name="script_filename" default="none"/>
@@ -56,4 +58,5 @@
     input_recipe_filename="${input_recipe_filename}"
     output_recipe_filename="${output_recipe_filename}"
+    prefix="${prefix}"
   />
   <!-- Load ROS 2 Gazebo Plugin -->
@@ -70,5 +73,5 @@
   <link name="world"/>
   <!-- Robot Stand: LINK -->
-  <link name='robot_stand'>
+  <link name='${prefix}robot_stand'>
     <inertial>
       <origin xyz="0 0 0" rpy="0 0 0"/>
@@ -90,13 +93,13 @@
   </link>
   <!-- Robot Stand: FIXED JOINT -->
-  <joint name="world_joint" type="fixed">
+  <joint name="${prefix}world_joint" type="fixed">
     <parent link= "world" />
-    <child link = "robot_stand" />
+    <child link = "${prefix}robot_stand" />
     <origin xyz="0.0 0.0 0.25" rpy="0.0 0.0 0.0" />
   </joint>
   <!-- Robot Stand: Robot+Stand JOINT -->
-  <joint name="stand_joint" type="fixed">
-    <parent link= "robot_stand" />
-    <child link = "base_link" />
+  <joint name="${prefix}stand_joint" type="fixed">
+    <parent link= "${prefix}robot_stand" />
+    <child link = "${prefix}base_link" />
     <origin xyz="0.0 0.0 0.255" rpy="0.0 0.0 0.0" />
   </joint>

File: packages/ros2srrc_ur10/urdf/ur10_robotiq_2f85.urdf.xacro (robot description, xacro)
@@ -39,4 +39,6 @@
   <xacro:arg name="EE_name" default="none"/>
   <xacro:property name="EE_name" value="$(arg EE_name)"/>
+  <xacro:arg name="prefix" default=""/>
+  <xacro:property name="prefix" value="$(arg prefix)"/>
   <!-- UR10 Control ARGUMENTS -->
   <xacro:arg name="script_filename" default="none"/>
@@ -56,4 +58,5 @@
     input_recipe_filename="${input_recipe_filename}"
     output_recipe_filename="${output_recipe_filename}"
+    prefix="${prefix}"
   />
   <!-- Include XACRO-MACRO file of the Robotiq 2f-85: -->
@@ -61,5 +64,6 @@
   <xacro:robotiq_2f85
     bringup="${bringup}"
-    parent_link="tool0"
+    parent_link="${prefix}tool0"
+    prefix="${prefix}"
   />
   <!-- Load ROS 2 Gazebo Plugin -->
@@ -78,5 +82,5 @@
   <link name="world"/>
   <!-- Robot Stand: LINK -->
-  <link name='robot_stand'>
+  <link name='${prefix}robot_stand'>
     <inertial>
       <origin xyz="0 0 0" rpy="0 0 0"/>
@@ -98,13 +102,13 @@
   </link>
   <!-- Robot Stand: FIXED JOINT -->
-  <joint name="world_joint" type="fixed">
+  <joint name="${prefix}world_joint" type="fixed">
     <parent link= "world" />
-    <child link = "robot_stand" />
+    <child link = "${prefix}robot_stand" />
     <origin xyz="0.0 0.0 0.25" rpy="0.0 0.0 0.0" />
   </joint>
   <!-- Robot Stand: Robot+Stand JOINT -->
-  <joint name="stand_joint" type="fixed">
-    <parent link= "robot_stand" />
-    <child link = "base_link" />
+  <joint name="${prefix}stand_joint" type="fixed">
+    <parent link= "${prefix}robot_stand" />
+    <child link = "${prefix}base_link" />
     <origin xyz="0.0 0.0 0.255" rpy="0.0 0.0 0.0" />
   </joint>

File: packages/ros2srrc_ur10/urdf/ur10_robotiq_hande.urdf.xacro (robot description, xacro)
@@ -39,4 +39,6 @@
   <xacro:arg name="EE_name" default="none"/>
   <xacro:property name="EE_name" value="$(arg EE_name)"/>
+  <xacro:arg name="prefix" default=""/>
+  <xacro:property name="prefix" value="$(arg prefix)"/>
   <!-- UR10 Control ARGUMENTS -->
   <xacro:arg name="script_filename" default="none"/>
@@ -56,4 +58,5 @@
     input_recipe_filename="${input_recipe_filename}"
     output_recipe_filename="${output_recipe_filename}"
+    prefix="${prefix}"
   />
   <!-- Include XACRO-MACRO file of the Robotiq 2f-85: -->
@@ -61,5 +64,6 @@
   <xacro:robotiq_hande
     bringup="${bringup}"
-    parent_link="tool0"
+    parent_link="${prefix}tool0"
+    prefix="${prefix}"
   />
   <!-- Load ROS 2 Gazebo Plugin -->
@@ -78,5 +82,5 @@
   <link name="world"/>
   <!-- Robot Stand: LINK -->
-  <link name='robot_stand'>
+  <link name='${prefix}robot_stand'>
     <inertial>
       <origin xyz="0 0 0" rpy="0 0 0"/>
@@ -98,13 +102,13 @@
   </link>
   <!-- Robot Stand: FIXED JOINT -->
-  <joint name="world_joint" type="fixed">
+  <joint name="${prefix}world_joint" type="fixed">
     <parent link= "world" />
-    <child link = "robot_stand" />
+    <child link = "${prefix}robot_stand" />
     <origin xyz="0.0 0.0 0.25" rpy="0.0 0.0 0.0" />
   </joint>
   <!-- Robot Stand: Robot+Stand JOINT -->
-  <joint name="stand_joint" type="fixed">
-    <parent link= "robot_stand" />
-    <child link = "base_link" />
+  <joint name="${prefix}stand_joint" type="fixed">
+    <parent link= "${prefix}robot_stand" />
+    <child link = "${prefix}base_link" />
     <origin xyz="0.0 0.0 0.255" rpy="0.0 0.0 0.0" />
   </joint>

File: packages/ros2srrc_ur10e/urdf/ur10e.urdf.xacro (robot description, xacro)
@@ -38,4 +38,6 @@
   <xacro:arg name="EE_name" default="none"/>
   <xacro:property name="EE_name" value="$(arg EE_name)"/>
+  <xacro:arg name="prefix" default=""/>
+  <xacro:property name="prefix" value="$(arg prefix)"/>
   <!-- UR10e Control ARGUMENTS -->
   <xacro:arg name="script_filename" default="none"/>
@@ -55,4 +57,5 @@
     input_recipe_filename="${input_recipe_filename}"
     output_recipe_filename="${output_recipe_filename}"
+    prefix="${prefix}"
   />
   <!-- Load ROS 2 Gazebo Plugin -->
@@ -69,5 +72,5 @@
   <link name="world"/>
   <!-- Robot Stand: LINK -->
-  <link name='robot_stand'>
+  <link name='${prefix}robot_stand'>
     <inertial>
       <origin xyz="0 0 0" rpy="0 0 0"/>
@@ -89,13 +92,13 @@
   </link>
   <!-- Robot Stand: FIXED JOINT -->
-  <joint name="world_joint" type="fixed">
+  <joint name="${prefix}world_joint" type="fixed">
     <parent link= "world" />
-    <child link = "robot_stand" />
+    <child link = "${prefix}robot_stand" />
     <origin xyz="0.0 0.0 0.25" rpy="0.0 0.0 0.0" />
   </joint>
   <!-- Robot Stand: Robot+Stand JOINT -->
-  <joint name="stand_joint" type="fixed">
-    <parent link= "robot_stand" />
-    <child link = "base_link" />
+  <joint name="${prefix}stand_joint" type="fixed">
+    <parent link= "${prefix}robot_stand" />
+    <child link = "${prefix}base_link" />
     <origin xyz="0.0 0.0 0.255" rpy="0.0 0.0 0.0" />
   </joint>

File: packages/ros2srrc_ur10e/urdf/ur10e_robotiq_2f85.urdf.xacro (robot description, xacro)
@@ -38,4 +38,6 @@
   <xacro:arg name="EE_name" default="none"/>
   <xacro:property name="EE_name" value="$(arg EE_name)"/>
+  <xacro:arg name="prefix" default=""/>
+  <xacro:property name="prefix" value="$(arg prefix)"/>
   <!-- UR10e Control ARGUMENTS -->
   <xacro:arg name="script_filename" default="none"/>
@@ -55,4 +57,5 @@
     input_recipe_filename="${input_recipe_filename}"
     output_recipe_filename="${output_recipe_filename}"
+    prefix="${prefix}"
   />
   <!-- Include XACRO-MACRO file of the Robotiq 2f-85: -->
@@ -60,5 +63,6 @@
   <xacro:robotiq_2f85
     bringup="${bringup}"
-    parent_link="tool0"
+    parent_link="${prefix}tool0"
+    prefix="${prefix}"
   />
   <!-- Load ROS 2 Gazebo Plugin -->
@@ -77,5 +81,5 @@
   <link name="world"/>
   <!-- Robot Stand: LINK -->
-  <link name='robot_stand'>
+  <link name='${prefix}robot_stand'>
     <inertial>
       <origin xyz="0 0 0" rpy="0 0 0"/>
@@ -97,13 +101,13 @@
   </link>
   <!-- Robot Stand: FIXED JOINT -->
-  <joint name="world_joint" type="fixed">
+  <joint name="${prefix}world_joint" type="fixed">
     <parent link= "world" />
-    <child link = "robot_stand" />
+    <child link = "${prefix}robot_stand" />
     <origin xyz="0.0 0.0 0.25" rpy="0.0 0.0 0.0" />
   </joint>
   <!-- Robot Stand: Robot+Stand JOINT -->
-  <joint name="stand_joint" type="fixed">
-    <parent link= "robot_stand" />
-    <child link = "base_link" />
+  <joint name="${prefix}stand_joint" type="fixed">
+    <parent link= "${prefix}robot_stand" />
+    <child link = "${prefix}base_link" />
     <origin xyz="0.0 0.0 0.255" rpy="0.0 0.0 0.0" />
   </joint>

File: packages/ros2srrc_ur10e/urdf/ur10e_robotiq_hande.urdf.xacro (robot description, xacro)
@@ -38,4 +38,6 @@
   <xacro:arg name="EE_name" default="none"/>
   <xacro:property name="EE_name" value="$(arg EE_name)"/>
+  <xacro:arg name="prefix" default=""/>
+  <xacro:property name="prefix" value="$(arg prefix)"/>
   <!-- UR10e Control ARGUMENTS -->
   <xacro:arg name="script_filename" default="none"/>
@@ -55,4 +57,5 @@
     input_recipe_filename="${input_recipe_filename}"
     output_recipe_filename="${output_recipe_filename}"
+    prefix="${prefix}"
   />
   <!-- Include XACRO-MACRO file of the Robotiq 2f-85: -->
@@ -60,5 +63,6 @@
   <xacro:robotiq_hande
     bringup="${bringup}"
-    parent_link="tool0"
+    parent_link="${prefix}tool0"
+    prefix="${prefix}"
   />
   <!-- Load ROS 2 Gazebo Plugin -->
@@ -77,5 +81,5 @@
   <link name="world"/>
   <!-- Robot Stand: LINK -->
-  <link name='robot_stand'>
+  <link name='${prefix}robot_stand'>
     <inertial>
       <origin xyz="0 0 0" rpy="0 0 0"/>
@@ -97,13 +101,13 @@
   </link>
   <!-- Robot Stand: FIXED JOINT -->
-  <joint name="world_joint" type="fixed">
+  <joint name="${prefix}world_joint" type="fixed">
     <parent link= "world" />
-    <child link = "robot_stand" />
+    <child link = "${prefix}robot_stand" />
     <origin xyz="0.0 0.0 0.25" rpy="0.0 0.0 0.0" />
   </joint>
   <!-- Robot Stand: Robot+Stand JOINT -->
-  <joint name="stand_joint" type="fixed">
-    <parent link= "robot_stand" />
-    <child link = "base_link" />
+  <joint name="${prefix}stand_joint" type="fixed">
+    <parent link= "${prefix}robot_stand" />
+    <child link = "${prefix}base_link" />
     <origin xyz="0.0 0.0 0.255" rpy="0.0 0.0 0.0" />
   </joint>
