Commit message: Adapt ros2srrc for multi-arm (prefix) (urdf, srdf and rviz files).

File: packages/ros2srrc_ar4/urdf/ar4.urdf.xacro (robot description, xacro)
@@ -38,4 +38,6 @@
   <xacro:arg name="EE_name" default="none"/>
   <xacro:property name="EE_name" value="$(arg EE_name)"/>
+  <xacro:arg name="prefix" default=""/>
+  <xacro:property name="prefix" value="$(arg prefix)"/>
   <!-- Include XACRO-MACRO file of the AR4: -->
   <xacro:include filename="$(find ros2srrc_robots)/ar4/urdf/ar4_macro.urdf.xacro"/>
@@ -45,4 +47,5 @@
     EE="${EE}"
     EE_name="${EE_name}"
+    prefix="${prefix}"
   />
   <!-- Load ROS 2 Gazebo Plugin -->
@@ -58,5 +61,5 @@
   <link name="world"/>
   <!-- Robot Stand: LINK -->
-  <link name='robot_stand'>
+  <link name='${prefix}robot_stand'>
     <inertial>
       <origin xyz="0 0 0" rpy="0 0 0"/>
@@ -78,13 +81,13 @@
   </link>
   <!-- Robot Stand: FIXED JOINT -->
-  <joint name="world_joint" type="fixed">
+  <joint name="${prefix}world_joint" type="fixed">
     <parent link="world" />
-    <child link = "robot_stand" />
+    <child link = "${prefix}robot_stand" />
     <origin xyz="0.0 0.0 0.25" rpy="0.0 0.0 0.0" />
   </joint>
   <!-- Robot Stand: Robot+Stand JOINT -->
-  <joint name="stand_joint" type="fixed">
-    <parent link="robot_stand" />
-    <child link = "base_link" />
+  <joint name="${prefix}stand_joint" type="fixed">
+    <parent link="${prefix}robot_stand" />
+    <child link = "${prefix}base_link" />
     <origin xyz="0.0 0.0 0.255" rpy="0.0 0.0 0.0" />
   </joint>

File: packages/ros2srrc_ar4/urdf/ar4_ar4gripper.urdf.xacro (robot description, xacro)
@@ -38,4 +38,6 @@
   <xacro:arg name="EE_name" default="none"/>
   <xacro:property name="EE_name" value="$(arg EE_name)"/>
+  <xacro:arg name="prefix" default=""/>
+  <xacro:property name="prefix" value="$(arg prefix)"/>
   <!-- Include XACRO-MACRO file of the AR4: -->
   <xacro:include filename="$(find ros2srrc_robots)/ar4/urdf/ar4_macro.urdf.xacro"/>
@@ -45,4 +47,5 @@
     EE="${EE}"
     EE_name="${EE_name}"
+    prefix="${prefix}"
   />
   <!-- Include XACRO-MACRO file of the GRIPPER: -->
@@ -50,5 +53,6 @@
   <xacro:ar4gripper
     bringup="${bringup}"
-    parent_link="tool0"
+    parent_link="${prefix}tool0"
+    prefix="${prefix}"
   />
   <!-- Load ROS 2 Gazebo Plugin -->
@@ -66,5 +70,5 @@
   <link name="world"/>
   <!-- Robot Stand: LINK -->
-  <link name='robot_stand'>
+  <link name='${prefix}robot_stand'>
     <inertial>
       <origin xyz="0 0 0" rpy="0 0 0"/>
@@ -86,13 +90,13 @@
   </link>
   <!-- Robot Stand: FIXED JOINT -->
-  <joint name="world_joint" type="fixed">
+  <joint name="${prefix}world_joint" type="fixed">
     <parent link="world" />
-    <child link = "robot_stand" />
+    <child link = "${prefix}robot_stand" />
     <origin xyz="0.0 0.0 0.25" rpy="0.0 0.0 0.0" />
   </joint>
   <!-- Robot Stand: Robot+Stand JOINT -->
-  <joint name="stand_joint" type="fixed">
-    <parent link="robot_stand" />
-    <child link = "base_link" />
+  <joint name="${prefix}stand_joint" type="fixed">
+    <parent link="${prefix}robot_stand" />
+    <child link = "${prefix}base_link" />
     <origin xyz="0.0 0.0 0.255" rpy="0.0 0.0 0.0" />
   </joint>

File: packages/ros2srrc_iiwa/urdf/iiwa.urdf.xacro (robot description, xacro)
@@ -38,4 +38,6 @@
   <xacro:arg name="EE_name" default="none"/>
   <xacro:property name="EE_name" value="$(arg EE_name)"/>
+  <xacro:arg name="prefix" default=""/>
+  <xacro:property name="prefix" value="$(arg prefix)"/>
   <!-- Include XACRO-MACRO file of the iiwa: -->
   <xacro:include filename="$(find ros2srrc_robots)/iiwa/urdf/iiwa_macro.urdf.xacro"/>
@@ -45,5 +47,5 @@
     EE="${EE}"
     EE_name="${EE_name}"
-  />
+    prefix="${prefix}" />
   <!-- Load ROS 2 Gazebo Plugin -->
   <xacro:unless value="${bringup}">
@@ -58,5 +60,5 @@
   <link name="world"/>
   <!-- Robot Stand: LINK -->
-  <link name='robot_stand'>
+  <link name='${prefix}robot_stand'>
     <inertial>
       <origin xyz="0 0 0" rpy="0 0 0"/>
@@ -78,13 +80,13 @@
   </link>
   <!-- Robot Stand: FIXED JOINT -->
-  <joint name="world_joint" type="fixed">
+  <joint name="${prefix}world_joint" type="fixed">
     <parent link="world" />
-    <child link = "robot_stand" />
+    <child link = "${prefix}robot_stand" />
     <origin xyz="0.0 0.0 0.25" rpy="0.0 0.0 0.0" />
   </joint>
   <!-- Robot Stand: Robot+Stand JOINT -->
-  <joint name="stand_joint" type="fixed">
-    <parent link="robot_stand" />
-    <child link = "base_link" />
+  <joint name="${prefix}stand_joint" type="fixed">
+    <parent link="${prefix}robot_stand" />
+    <child link = "${prefix}base_link" />
     <origin xyz="0.0 0.0 0.255" rpy="0.0 0.0 0.0" />
   </joint>

File: packages/ros2srrc_iiwa/urdf/iiwa_robotiq_2f85.urdf.xacro (robot description, xacro)
@@ -38,4 +38,6 @@
   <xacro:arg name="EE_name" default="none"/>
   <xacro:property name="EE_name" value="$(arg EE_name)"/>
+  <xacro:arg name="prefix" default=""/>
+  <xacro:property name="prefix" value="$(arg prefix)"/>
   <!-- Include XACRO-MACRO file of the iiwa: -->
   <xacro:include filename="$(find ros2srrc_robots)/iiwa/urdf/iiwa_macro.urdf.xacro"/>
@@ -45,11 +47,11 @@
     EE="${EE}"
     EE_name="${EE_name}"
-  />
+    prefix="${prefix}" />
   <!-- Include XACRO-MACRO file of the End-Effector: -->
   <xacro:include filename="$(find ros2srrc_endeffectors)/robotiq_2f85/urdf/robotiq_2f85_macro.urdf.xacro"/>
   <xacro:robotiq_2f85
     bringup="${bringup}"
-    parent_link="tool0"
-  />
+    parent_link="${prefix}tool0"
+    prefix="${prefix}" />
   <!-- Load ROS 2 Gazebo Plugin -->
   <xacro:unless value="${bringup}">
@@ -66,5 +68,5 @@
   <link name="world"/>
   <!-- Robot Stand: LINK -->
-  <link name='robot_stand'>
+  <link name='${prefix}robot_stand'>
     <inertial>
       <origin xyz="0 0 0" rpy="0 0 0"/>
@@ -86,13 +88,13 @@
   </link>
   <!-- Robot Stand: FIXED JOINT -->
-  <joint name="world_joint" type="fixed">
+  <joint name="${prefix}world_joint" type="fixed">
     <parent link="world" />
-    <child link = "robot_stand" />
+    <child link = "${prefix}robot_stand" />
     <origin xyz="0.0 0.0 0.25" rpy="0.0 0.0 0.0" />
   </joint>
   <!-- Robot Stand: Robot+Stand JOINT -->
-  <joint name="stand_joint" type="fixed">
-    <parent link="robot_stand" />
-    <child link = "base_link" />
+  <joint name="${prefix}stand_joint" type="fixed">
+    <parent link="${prefix}robot_stand" />
+    <child link = "${prefix}base_link" />
     <origin xyz="0.0 0.0 0.255" rpy="0.0 0.0 0.0" />
   </joint>

File: packages/ros2srrc_irb120/urdf/irb120.urdf.xacro (robot description, xacro)
@@ -38,4 +38,6 @@
   <xacro:arg name="EE_name" default="none"/>
   <xacro:property name="EE_name" value="$(arg EE_name)"/>
+  <xacro:arg name="prefix" default=""/>
+  <xacro:property name="prefix" value="$(arg prefix)"/>
   <!-- Include XACRO-MACRO file of the IRB120: -->
   <xacro:include filename="$(find ros2srrc_robots)/irb120/urdf/irb120_macro.urdf.xacro"/>
@@ -45,5 +47,5 @@
     EE="${EE}"
     EE_name="${EE_name}"
-  />
+    prefix="${prefix}" />
   <!-- Load ROS 2 Gazebo Plugin -->
   <xacro:unless value="${bringup}">
@@ -58,5 +60,5 @@
   <link name="world"/>
   <!-- Robot Stand: LINK -->
-  <link name='robot_stand'>
+  <link name='${prefix}robot_stand'>
     <inertial>
       <origin xyz="0 0 0" rpy="0 0 0"/>
@@ -78,13 +80,13 @@
   </link>
   <!-- Robot Stand: FIXED JOINT -->
-  <joint name="world_joint" type="fixed">
+  <joint name="${prefix}world_joint" type="fixed">
     <parent link="world" />
-    <child link = "robot_stand" />
+    <child link = "${prefix}robot_stand" />
     <origin xyz="0.0 0.0 0.25" rpy="0.0 0.0 0.0" />
   </joint>
   <!-- Robot Stand: Robot+Stand JOINT -->
-  <joint name="stand_joint" type="fixed">
-    <parent link="robot_stand" />
-    <child link = "base_link" />
+  <joint name="${prefix}stand_joint" type="fixed">
+    <parent link="${prefix}robot_stand" />
+    <child link = "${prefix}base_link" />
     <origin xyz="0.0 0.0 0.255" rpy="0.0 0.0 0.0" />
   </joint>

File: packages/ros2srrc_irb120/urdf/irb120_egp64.urdf.xacro (robot description, xacro)
@@ -38,4 +38,6 @@
   <xacro:arg name="EE_name" default="none"/>
   <xacro:property name="EE_name" value="$(arg EE_name)"/>
+  <xacro:arg name="prefix" default=""/>
+  <xacro:property name="prefix" value="$(arg prefix)"/>
   <!-- Include XACRO-MACRO file of the IRB120: -->
   <xacro:include filename="$(find ros2srrc_robots)/irb120/urdf/irb120_macro.urdf.xacro"/>
@@ -45,11 +47,11 @@
     EE="${EE}"
     EE_name="${EE_name}"
-  />
+    prefix="${prefix}" />
   <!-- Include XACRO-MACRO file of the EGP64: -->
   <xacro:include filename="$(find ros2srrc_endeffectors)/egp64/urdf/egp64_macro.urdf.xacro"/>
   <xacro:egp64
     bringup="${bringup}"
-    parent_link="tool0"
-  />
+    parent_link="${prefix}tool0"
+    prefix="${prefix}" />
   <!-- Load ROS 2 Gazebo Plugin -->
   <xacro:unless value="${bringup}">
@@ -66,5 +68,5 @@
   <link name="world"/>
   <!-- Robot Stand: LINK -->
-  <link name='robot_stand'>
+  <link name='${prefix}robot_stand'>
     <inertial>
       <origin xyz="0 0 0" rpy="0 0 0"/>
@@ -86,13 +88,13 @@
   </link>
   <!-- Robot Stand: FIXED JOINT -->
-  <joint name="world_joint" type="fixed">
+  <joint name="${prefix}world_joint" type="fixed">
     <parent link="world" />
-    <child link = "robot_stand" />
+    <child link = "${prefix}robot_stand" />
     <origin xyz="0.0 0.0 0.25" rpy="0.0 0.0 0.0" />
   </joint>
   <!-- Robot Stand: Robot+Stand JOINT -->
-  <joint name="stand_joint" type="fixed">
-    <parent link="robot_stand" />
-    <child link = "base_link" />
+  <joint name="${prefix}stand_joint" type="fixed">
+    <parent link="${prefix}robot_stand" />
+    <child link = "${prefix}base_link" />
     <origin xyz="0.0 0.0 0.255" rpy="0.0 0.0 0.0" />
   </joint>

File: packages/ros2srrc_irb120/urdf/irb120_egp64v2.urdf.xacro (robot description, xacro)
@@ -38,4 +38,6 @@
   <xacro:arg name="EE_name" default="none"/>
   <xacro:property name="EE_name" value="$(arg EE_name)"/>
+  <xacro:arg name="prefix" default=""/>
+  <xacro:property name="prefix" value="$(arg prefix)"/>
   <!-- Include XACRO-MACRO file of the IRB120: -->
   <xacro:include filename="$(find ros2srrc_robots)/irb120/urdf/irb120_macro.urdf.xacro"/>
@@ -45,11 +47,11 @@
     EE="${EE}"
     EE_name="${EE_name}"
-  />
+    prefix="${prefix}" />
   <!-- Include XACRO-MACRO file of the EGP64: -->
   <xacro:include filename="$(find ros2srrc_endeffectors)/egp64/urdf/egp64v2_macro.urdf.xacro"/>
   <xacro:egp64
     bringup="${bringup}"
-    parent_link="tool0"
-  />
+    parent_link="${prefix}tool0"
+    prefix="${prefix}" />
   <!-- Load ROS 2 Gazebo Plugin -->
   <xacro:unless value="${bringup}">
@@ -66,5 +68,5 @@
   <link name="world"/>
   <!-- Robot Stand: LINK -->
-  <link name='robot_stand'>
+  <link name='${prefix}robot_stand'>
     <inertial>
       <origin xyz="0 0 0" rpy="0 0 0"/>
@@ -86,13 +88,13 @@
   </link>
   <!-- Robot Stand: FIXED JOINT -->
-  <joint name="world_joint" type="fixed">
+  <joint name="${prefix}world_joint" type="fixed">
     <parent link="world" />
-    <child link = "robot_stand" />
+    <child link = "${prefix}robot_stand" />
     <origin xyz="0.0 0.0 0.25" rpy="0.0 0.0 0.0" />
   </joint>
   <!-- Robot Stand: Robot+Stand JOINT -->
-  <joint name="stand_joint" type="fixed">
-    <parent link="robot_stand" />
-    <child link = "base_link" />
+  <joint name="${prefix}stand_joint" type="fixed">
+    <parent link="${prefix}robot_stand" />
+    <child link = "${prefix}base_link" />
     <origin xyz="0.0 0.0 0.255" rpy="0.0 0.0 0.0" />
   </joint>

File: packages/ros2srrc_irb120/urdf/irb120_ls_vgr.urdf.xacro (robot description, xacro)
@@ -38,4 +38,6 @@
   <xacro:arg name="EE_name" default="none"/>
   <xacro:property name="EE_name" value="$(arg EE_name)"/>
+  <xacro:arg name="prefix" default=""/>
+  <xacro:property name="prefix" value="$(arg prefix)"/>
   <!-- Include XACRO-MACRO file of the IRB120: -->
   <xacro:include filename="$(find ros2srrc_robots)/irb120/urdf/irb120_macro.urdf.xacro"/>
@@ -45,11 +47,11 @@
     EE="${EE}"
     EE_name="${EE_name}"
-  />
+    prefix="${prefix}" />
   <!-- Include XACRO-MACRO file of the LS-VGR: -->
   <xacro:include filename="$(find ros2srrc_endeffectors)/ls_vgr/urdf/ls_vgr_macro.urdf.xacro"/>
   <xacro:ls_vgr
     bringup="${bringup}"
-    parent_link="tool0"
-  />
+    parent_link="${prefix}tool0"
+    prefix="${prefix}" />
   <!-- Load ROS 2 Gazebo Plugin -->
   <xacro:unless value="${bringup}">
@@ -66,5 +68,5 @@
   <link name="world"/>
   <!-- Robot Stand: LINK -->
-  <link name='robot_stand'>
+  <link name='${prefix}robot_stand'>
     <inertial>
       <origin xyz="0 0 0" rpy="0 0 0"/>
@@ -86,13 +88,13 @@
   </link>
   <!-- Robot Stand: FIXED JOINT -->
-  <joint name="world_joint" type="fixed">
+  <joint name="${prefix}world_joint" type="fixed">
     <parent link="world" />
-    <child link = "robot_stand" />
+    <child link = "${prefix}robot_stand" />
     <origin xyz="0.0 0.0 0.25" rpy="0.0 0.0 0.0" />
   </joint>
   <!-- Robot Stand: Robot+Stand JOINT -->
-  <joint name="stand_joint" type="fixed">
-    <parent link="robot_stand" />
-    <child link = "base_link" />
+  <joint name="${prefix}stand_joint" type="fixed">
+    <parent link="${prefix}robot_stand" />
+    <child link = "${prefix}base_link" />
     <origin xyz="0.0 0.0 0.255" rpy="0.0 0.0 0.0" />
   </joint>

File: packages/ros2srrc_irb1200/urdf/irb1200.urdf.xacro (robot description, xacro)
@@ -38,4 +38,6 @@
   <xacro:arg name="EE_name" default="none"/>
   <xacro:property name="EE_name" value="$(arg EE_name)"/>
+  <xacro:arg name="prefix" default=""/>
+  <xacro:property name="prefix" value="$(arg prefix)"/>
   <!-- Include XACRO-MACRO file of the IRB1200: -->
   <xacro:include filename="$(find ros2srrc_robots)/irb1200/urdf/irb1200_macro.urdf.xacro"/>
@@ -45,5 +47,5 @@
     EE="${EE}"
     EE_name="${EE_name}"
-  />
+    prefix="${prefix}" />
   <!-- Load ROS 2 Gazebo Plugin -->
   <xacro:unless value="${bringup}">
@@ -58,5 +60,5 @@
   <link name="world"/>
   <!-- Robot Stand: LINK -->
-  <link name='robot_stand'>
+  <link name='${prefix}robot_stand'>
     <inertial>
       <origin xyz="0 0 0" rpy="0 0 0"/>
@@ -78,13 +80,13 @@
   </link>
   <!-- Robot Stand: FIXED JOINT -->
-  <joint name="world_joint" type="fixed">
+  <joint name="${prefix}world_joint" type="fixed">
     <parent link="world" />
-    <child link = "robot_stand" />
+    <child link = "${prefix}robot_stand" />
     <origin xyz="0.0 0.0 0.25" rpy="0.0 0.0 0.0" />
   </joint>
   <!-- Robot Stand: Robot+Stand JOINT -->
-  <joint name="stand_joint" type="fixed">
-    <parent link="robot_stand" />
-    <child link = "base_link" />
+  <joint name="${prefix}stand_joint" type="fixed">
+    <parent link="${prefix}robot_stand" />
+    <child link = "${prefix}base_link" />
     <origin xyz="0.0 0.0 0.255" rpy="0.0 0.0 0.0" />
   </joint>

File: packages/ros2srrc_irb1200/urdf/irb1200_egp64.urdf.xacro (robot description, xacro)
@@ -38,4 +38,6 @@
   <xacro:arg name="EE_name" default="none"/>
   <xacro:property name="EE_name" value="$(arg EE_name)"/>
+  <xacro:arg name="prefix" default=""/>
+  <xacro:property name="prefix" value="$(arg prefix)"/>
   <!-- Include XACRO-MACRO file of the IRB1200: -->
   <xacro:include filename="$(find ros2srrc_robots)/irb1200/urdf/irb1200_macro.urdf.xacro"/>
@@ -45,11 +47,11 @@
     EE="${EE}"
     EE_name="${EE_name}"
-  />
+    prefix="${prefix}" />
   <!-- Include XACRO-MACRO file of the EGP64: -->
   <xacro:include filename="$(find ros2srrc_endeffectors)/egp64/urdf/egp64_macro.urdf.xacro"/>
   <xacro:egp64
     bringup="${bringup}"
-    parent_link="tool0"
-  />
+    parent_link="${prefix}tool0"
+    prefix="${prefix}" />
   <!-- Load ROS 2 Gazebo Plugin -->
   <xacro:unless value="${bringup}">
@@ -66,5 +68,5 @@
   <link name="world"/>
   <!-- Robot Stand: LINK -->
-  <link name='robot_stand'>
+  <link name='${prefix}robot_stand'>
     <inertial>
       <origin xyz="0 0 0" rpy="0 0 0"/>
@@ -86,13 +88,13 @@
   </link>
   <!-- Robot Stand: FIXED JOINT -->
-  <joint name="world_joint" type="fixed">
+  <joint name="${prefix}world_joint" type="fixed">
     <parent link="world" />
-    <child link = "robot_stand" />
+    <child link = "${prefix}robot_stand" />
     <origin xyz="0.0 0.0 0.25" rpy="0.0 0.0 0.0" />
   </joint>
   <!-- Robot Stand: Robot+Stand JOINT -->
-  <joint name="stand_joint" type="fixed">
-    <parent link="robot_stand" />
-    <child link = "base_link" />
+  <joint name="${prefix}stand_joint" type="fixed">
+    <parent link="${prefix}robot_stand" />
+    <child link = "${prefix}base_link" />
     <origin xyz="0.0 0.0 0.255" rpy="0.0 0.0 0.0" />
   </joint>

File: packages/ros2srrc_irb1600/urdf/irb1600.urdf.xacro (robot description, xacro)
@@ -38,4 +38,6 @@
   <xacro:arg name="EE_name" default="none"/>
   <xacro:property name="EE_name" value="$(arg EE_name)"/>
+  <xacro:arg name="prefix" default=""/>
+  <xacro:property name="prefix" value="$(arg prefix)"/>
   <!-- Include XACRO-MACRO file of the IRB1600: -->
   <xacro:include filename="$(find ros2srrc_robots)/irb1600/urdf/irb1600_macro.urdf.xacro"/>
@@ -45,5 +47,5 @@
     EE="${EE}"
     EE_name="${EE_name}"
-  />
+    prefix="${prefix}" />
   <!-- Load ROS 2 Gazebo Plugin -->
   <xacro:unless value="${bringup}">
@@ -58,5 +60,5 @@
   <link name="world"/>
   <!-- Robot Stand: LINK -->
-  <link name='robot_stand'>
+  <link name='${prefix}robot_stand'>
     <inertial>
       <origin xyz="0 0 0" rpy="0 0 0"/>
@@ -78,13 +80,13 @@
   </link>
   <!-- Robot Stand: FIXED JOINT -->
-  <joint name="world_joint" type="fixed">
+  <joint name="${prefix}world_joint" type="fixed">
     <parent link="world" />
-    <child link = "robot_stand" />
+    <child link = "${prefix}robot_stand" />
     <origin xyz="0.0 0.0 0.25" rpy="0.0 0.0 0.0" />
   </joint>
   <!-- Robot Stand: Robot+Stand JOINT -->
-  <joint name="stand_joint" type="fixed">
-    <parent link="robot_stand" />
-    <child link = "base_link" />
+  <joint name="${prefix}stand_joint" type="fixed">
+    <parent link="${prefix}robot_stand" />
+    <child link = "${prefix}base_link" />
     <origin xyz="0.0 0.0 0.255" rpy="0.0 0.0 0.0" />
   </joint>

File: packages/ros2srrc_irb6640/urdf/irb6640.urdf.xacro (robot description, xacro)
@@ -38,4 +38,6 @@
   <xacro:arg name="EE_name" default="none"/>
   <xacro:property name="EE_name" value="$(arg EE_name)"/>
+  <xacro:arg name="prefix" default=""/>
+  <xacro:property name="prefix" value="$(arg prefix)"/>
   <!-- Include XACRO-MACRO file of the IRB6640: -->
   <xacro:include filename="$(find ros2srrc_robots)/irb6640/urdf/irb6640_macro.urdf.xacro"/>
@@ -45,5 +47,5 @@
     EE="${EE}"
     EE_name="${EE_name}"
-  />
+    prefix="${prefix}" />
   <!-- Load ROS 2 Gazebo Plugin -->
   <xacro:unless value="${bringup}">
@@ -58,5 +60,5 @@
   <link name="world"/>
   <!-- Robot Stand: LINK -->
-  <link name='robot_stand'>
+  <link name='${prefix}robot_stand'>
     <inertial>
       <origin xyz="0 0 0" rpy="0 0 0"/>
@@ -78,13 +80,13 @@
   </link>
   <!-- Robot Stand: FIXED JOINT -->
-  <joint name="world_joint" type="fixed">
+  <joint name="${prefix}world_joint" type="fixed">
     <parent link="world" />
-    <child link = "robot_stand" />
+    <child link = "${prefix}robot_stand" />
     <origin xyz="0.0 0.0 0.25" rpy="0.0 0.0 0.0" />
   </joint>
   <!-- Robot Stand: Robot+Stand JOINT -->
-  <joint name="stand_joint" type="fixed">
-    <parent link="robot_stand" />
-    <child link = "base_link" />
+  <joint name="${prefix}stand_joint" type="fixed">
+    <parent link="${prefix}robot_stand" />
+    <child link = "${prefix}base_link" />
     <origin xyz="0.0 0.0 0.255" rpy="0.0 0.0 0.0" />
   </joint>

File: packages/ros2srrc_irb6640/urdf/irb6640_gpp5010nc.urdf.xacro (robot description, xacro)
@@ -38,4 +38,6 @@
   <xacro:arg name="EE_name" default="none"/>
   <xacro:property name="EE_name" value="$(arg EE_name)"/>
+  <xacro:arg name="prefix" default=""/>
+  <xacro:property name="prefix" value="$(arg prefix)"/>
   <!-- Include XACRO-MACRO file of the IRB6640: -->
   <xacro:include filename="$(find ros2srrc_robots)/irb6640/urdf/irb6640_macro.urdf.xacro"/>
@@ -45,7 +47,7 @@
     EE="${EE}"
     EE_name="${EE_name}"
-  />
+    prefix="${prefix}" />
   <!-- Include: IRB6640/GPP5010NC ADAPTER -->
-  <link name="adapter">
+  <link name="${prefix}adapter">
     <visual>
       <geometry>
@@ -64,8 +66,8 @@
     </inertial>
   </link>
-  <joint name="adapter_joint" type="fixed">
+  <joint name="${prefix}adapter_joint" type="fixed">
     <origin xyz="0.0 0 0.023" rpy="0 ${pi/2} ${pi}" />
-    <parent link="tool0"/>
-    <child link="adapter"/>
+    <parent link="${prefix}tool0"/>
+    <child link="${prefix}adapter"/>
   </joint>
   <!-- Include XACRO-MACRO file of the GPP5010NC: -->
@@ -73,6 +75,6 @@
   <xacro:gpp5010nc
     bringup="${bringup}"
-    parent_link="adapter"
-  />
+    parent_link="${prefix}adapter"
+    prefix="${prefix}" />
   <!-- Load ROS 2 Gazebo Plugin -->
   <xacro:unless value="${bringup}">
@@ -89,5 +91,5 @@
   <link name="world"/>
   <!-- Robot Stand: LINK -->
-  <link name='robot_stand'>
+  <link name='${prefix}robot_stand'>
     <inertial>
       <origin xyz="0 0 0" rpy="0 0 0"/>
@@ -109,13 +111,13 @@
   </link>
   <!-- Robot Stand: FIXED JOINT -->
-  <joint name="world_joint" type="fixed">
+  <joint name="${prefix}world_joint" type="fixed">
     <parent link="world" />
-    <child link = "robot_stand" />
+    <child link = "${prefix}robot_stand" />
     <origin xyz="0.0 0.0 0.25" rpy="0.0 0.0 0.0" />
   </joint>
   <!-- Robot Stand: Robot+Stand JOINT -->
-  <joint name="stand_joint" type="fixed">
-    <parent link="robot_stand" />
-    <child link = "base_link" />
+  <joint name="${prefix}stand_joint" type="fixed">
+    <parent link="${prefix}robot_stand" />
+    <child link = "${prefix}base_link" />
     <origin xyz="0.0 0.0 0.255" rpy="0.0 0.0 0.0" />
   </joint>
