Commit message: Repo sanity check: Fix inconsistencies, fix typos/errors and improve .md files.

File: packages/ros2srrc_ur10/urdf/ur10_robotiq_hande.urdf.xacro (robot description, xacro)
@@ -59,5 +59,5 @@
     output_recipe_filename="${output_recipe_filename}"
     prefix="${prefix}" />
-  <!-- Include XACRO-MACRO file of the Robotiq 2f-85: -->
+  <!-- Include XACRO-MACRO file of the Robotiq HandE: -->
   <xacro:include filename="$(find ros2srrc_endeffectors)/robotiq_hande/urdf/robotiq_hande_macro.urdf.xacro"/>
   <xacro:robotiq_hande

File: packages/ros2srrc_ur10e/urdf/ur10e_robotiq_hande.urdf.xacro (robot description, xacro)
@@ -58,5 +58,5 @@
     output_recipe_filename="${output_recipe_filename}"
     prefix="${prefix}" />
-  <!-- Include XACRO-MACRO file of the Robotiq 2f-85: -->
+  <!-- Include XACRO-MACRO file of the Robotiq HandE: -->
   <xacro:include filename="$(find ros2srrc_endeffectors)/robotiq_hande/urdf/robotiq_hande_macro.urdf.xacro"/>
   <xacro:robotiq_hande

File: packages/ros2srrc_ur16e/urdf/ur16e_robotiq_hande.urdf.xacro (robot description, xacro)
@@ -58,5 +58,5 @@
     output_recipe_filename="${output_recipe_filename}"
     prefix="${prefix}" />
-  <!-- Include XACRO-MACRO file of the Robotiq 2f-85: -->
+  <!-- Include XACRO-MACRO file of the Robotiq HandE: -->
   <xacro:include filename="$(find ros2srrc_endeffectors)/robotiq_hande/urdf/robotiq_hande_macro.urdf.xacro"/>
   <xacro:robotiq_hande

File: packages/ros2srrc_ur20/urdf/ur20_robotiq_hande.urdf.xacro (robot description, xacro)
@@ -58,5 +58,5 @@
     output_recipe_filename="${output_recipe_filename}"
     prefix="${prefix}" />
-  <!-- Include XACRO-MACRO file of the Robotiq 2f-85: -->
+  <!-- Include XACRO-MACRO file of the Robotiq HandE: -->
   <xacro:include filename="$(find ros2srrc_endeffectors)/robotiq_hande/urdf/robotiq_hande_macro.urdf.xacro"/>
   <xacro:robotiq_hande

File: packages/ros2srrc_ur3/urdf/ur3_robotiq_hande.urdf.xacro (robot description, xacro)
@@ -58,5 +58,5 @@
     output_recipe_filename="${output_recipe_filename}"
     prefix="${prefix}" />
-  <!-- Include XACRO-MACRO file of the Robotiq 2f-85: -->
+  <!-- Include XACRO-MACRO file of the Robotiq HandE: -->
   <xacro:include filename="$(find ros2srrc_endeffectors)/robotiq_hande/urdf/robotiq_hande_macro.urdf.xacro"/>
   <xacro:robotiq_hande

File: packages/ros2srrc_ur3e/urdf/ur3e_robotiq_hande.urdf.xacro (robot description, xacro)
@@ -58,5 +58,5 @@
     output_recipe_filename="${output_recipe_filename}"
     prefix="${prefix}" />
-  <!-- Include XACRO-MACRO file of the Robotiq 2f-85: -->
+  <!-- Include XACRO-MACRO file of the Robotiq HandE: -->
   <xacro:include filename="$(find ros2srrc_endeffectors)/robotiq_hande/urdf/robotiq_hande_macro.urdf.xacro"/>
   <xacro:robotiq_hande

File: packages/ros2srrc_ur5/urdf/ur5_robotiq_hande.urdf.xacro (robot description, xacro)
@@ -58,5 +58,5 @@
     output_recipe_filename="${output_recipe_filename}"
     prefix="${prefix}" />
-  <!-- Include XACRO-MACRO file of the Robotiq 2f-85: -->
+  <!-- Include XACRO-MACRO file of the Robotiq HandE: -->
   <xacro:include filename="$(find ros2srrc_endeffectors)/robotiq_hande/urdf/robotiq_hande_macro.urdf.xacro"/>
   <xacro:robotiq_hande

File: packages/ros2srrc_ur5e/urdf/ur5e_robotiq_hande.urdf.xacro (robot description, xacro)
@@ -58,5 +58,5 @@
     output_recipe_filename="${output_recipe_filename}"
     prefix="${prefix}" />
-  <!-- Include XACRO-MACRO file of the Robotiq 2f-85: -->
+  <!-- Include XACRO-MACRO file of the Robotiq HandE: -->
   <xacro:include filename="$(find ros2srrc_endeffectors)/robotiq_hande/urdf/robotiq_hande_macro.urdf.xacro"/>
   <xacro:robotiq_hande

File: ros2srrc_endeffectors/ar4gripper/urdf/ar4gripper_macro.urdf.xacro (robot description, xacro)
@@ -36,5 +36,5 @@
       <xacro:ar4gripper_transmission prefix="${prefix}"/>
     </xacro:unless>
-    <!-- ***** AR4 ROBOT's GRIPPER .urdf SERIAL CHAIN ***** -->
+    <!-- ***** AR4 robot's GRIPPER .urdf SERIAL CHAIN ***** -->
     <!-- GRIPPER BASE -->
     <link name="${prefix}gripper_base_link">

File: ros2srrc_robots/ar4/urdf/ar4_macro.urdf.xacro (robot description, xacro)
@@ -37,5 +37,5 @@
 #                                                                                       #
 #  CHANGES MADE:                                                                        #
-#  The ROS 2 Robot URDF files have been adapted to the ros2srrc repo structure.         #                                                      #
+#  The ROS 2 Robot URDF files have been adapted to the ros2srrc repo structure.         #
 #                                                                                       #
 # ===================================== COPYRIGHT ===================================== #
@@ -52,5 +52,5 @@
       <xacro:ar4_transmission prefix="${prefix}"/>
     </xacro:unless>
-    <!-- AR4 GAZEBO - ROS2_CONTROL: -->
+    <!-- AR4 GZ Sim - ros2_control: -->
     <xacro:include filename="$(find ros2srrc_robots)/ar4/urdf/ar4_ros2control.xacro" />
     <xacro:ar4_ros2control

File: ros2srrc_robots/ar4/urdf/ar4_ros2control.xacro (robot description, xacro)
@@ -37,5 +37,5 @@
 #                                                                                       #
 #  CHANGES MADE:                                                                        #
-#  The ROS 2 Robot URDF files have been adapted to the ros2srrc repo structure.         #                                                      #
+#  The ROS 2 Robot URDF files have been adapted to the ros2srrc repo structure.         #
 #                                                                                       #
 # ===================================== COPYRIGHT ===================================== #
@@ -46,6 +46,6 @@
 <robot xmlns:xacro="http://www.ros.org/wiki/xacro">
   <xacro:macro name="ar4_ros2control" params="bringup robot_ip EE EE_name prefix" >
-    <!-- 1. ROS2_CONTROL tag name: -->
-    <!-- A. GAZEBO SIMULATION: -->
+    <!-- 1. ros2_control tag name: -->
+    <!-- A. GZ Sim simulation: -->
     <xacro:unless value="${bringup}">
       <xacro:property name="name" value="${prefix}GazeboSimSystem"/>
@@ -54,7 +54,7 @@
     <xacro:if value="${bringup}">
     </xacro:if> -->
-    <!-- 3. Load ROS2_CONTROL: -->
+    <!-- 3. Load ros2_control: -->
     <ros2_control name="${name}" type="system">
-      <!-- A. GAZEBO SIMULATION: -->
+      <!-- A. GZ Sim simulation: -->
       <xacro:unless value="${bringup}">
         <hardware>

File: ros2srrc_robots/iiwa/urdf/iiwa_macro.urdf.xacro (robot description, xacro)
@@ -26,6 +26,6 @@
 # ===================================== COPYRIGHT ===================================== #
 #                                                                                       #
-#  Some of the information used to build the LBR-IIWA robot .urdf files in this ROS2    #
-#  repository has been taken from the following resource:                               #
+#  Some of the information used to build the LBR-IIWA robot .urdf files in this         #
+#  ROS 2 repository has been taken from the following resource:                         #
 #       - ros-industrial https://github.com/ros-industrial/kuka_experimental            #
 #                                                                                       #
@@ -56,5 +56,5 @@
       prefix="${prefix}" />
     </xacro:unless>
-    <!-- KUKA LBR-IIWA GAZEBO - ROS2_CONTROL: -->
+    <!-- KUKA LBR-IIWA GZ Sim - ros2_control: -->
     <xacro:include filename="$(find ros2srrc_robots)/iiwa/urdf/iiwa_ros2control.xacro" />
     <xacro:iiwa_ros2control
@@ -276,5 +276,5 @@
       <axis xyz="0 -1 0"/>
       <limit effort="176" lower="-2.0942" upper="2.0942" velocity="1.3089"/>
-      <dynamics damping="10.0" friction="1.0"/> <!-- High values of damping + friction were added, to avoid bac joint behaviour in GzFortress. -->
+      <dynamics damping="10.0" friction="1.0"/> <!-- High values of damping + friction were added, to avoid bad joint behavior in GzFortress. -->
     </joint>
     <joint name="${prefix}joint_5" type="revolute">

File: ros2srrc_robots/iiwa/urdf/iiwa_ros2control.xacro (robot description, xacro)
@@ -26,6 +26,6 @@
 # ===================================== COPYRIGHT ===================================== #
 #                                                                                       #
-#  Some of the information used to build the LBR-IIWA robot .urdf files in this ROS2    #
-#  repository has been taken from the following resource:                               #
+#  Some of the information used to build the LBR-IIWA robot .urdf files in this         #
+#  ROS 2 repository has been taken from the following resource:                         #
 #       - ros-industrial https://github.com/ros-industrial/kuka_experimental            #
 #                                                                                       #
@@ -49,6 +49,6 @@
 <robot xmlns:xacro="http://www.ros.org/wiki/xacro">
   <xacro:macro name="iiwa_ros2control" params="bringup robot_ip EE EE_name prefix" >
-    <!-- 1. ROS2_CONTROL tag name: -->
-    <!-- A. GAZEBO SIMULATION: -->
+    <!-- 1. ros2_control tag name: -->
+    <!-- A. GZ Sim simulation: -->
     <xacro:unless value="${bringup}">
       <xacro:property name="name" value="${prefix}GazeboSimSystem"/>
@@ -58,7 +58,7 @@
       <xacro:property name="name" value="${prefix}TBD"/>
     </xacro:if>
-    <!-- 3. Load ROS2_CONTROL: -->
+    <!-- 3. Load ros2_control: -->
     <ros2_control name="${name}" type="system">
-      <!-- A. GAZEBO SIMULATION: -->
+      <!-- A. GZ Sim simulation: -->
       <xacro:unless value="${bringup}">
         <hardware>

File: ros2srrc_robots/iiwa/urdf/iiwa_transmission.xacro (robot description, xacro)
@@ -26,6 +26,6 @@
 # ===================================== COPYRIGHT ===================================== #
 #                                                                                       #
-#  Some of the information used to build the LBR-IIWA robot .urdf files in this ROS2    #
-#  repository has been taken from the following resource:                               #
+#  Some of the information used to build the LBR-IIWA robot .urdf files in this         #
+#  ROS 2 repository has been taken from the following resource:                         #
 #       - ros-industrial https://github.com/ros-industrial/kuka_experimental            #
 #                                                                                       #

File: ros2srrc_robots/irb120/urdf/irb120_macro.urdf.xacro (robot description, xacro)
@@ -26,6 +26,6 @@
 # ===================================== COPYRIGHT ===================================== #
 #                                                                                       #
-#  Some of the information used to build the ROS2 ABB-IRB120 .urdf files in this ROS2   #
-#  repository has been taken from the following resource:                               #
+#  Some of the information used to build the ROS 2 ABB-IRB120 .urdf files in this       #
+#  ROS 2 repository has been taken from the following resource:                         #
 #       - abb_experimental (https://github.com/ros-industrial/abb_experimental)         #
 #                                                                                       #
@@ -58,5 +58,5 @@
       prefix="${prefix}" />
     </xacro:unless>
-    <!-- ABB-IRB120 GAZEBO - ROS2_CONTROL: -->
+    <!-- ABB-IRB120 GZ Sim - ros2_control: -->
     <xacro:include filename="$(find ros2srrc_robots)/irb120/urdf/irb120_ros2control.xacro" />
     <xacro:irb120_ros2control

File: ros2srrc_robots/irb120/urdf/irb120_ros2control.xacro (robot description, xacro)
@@ -26,6 +26,6 @@
 # ===================================== COPYRIGHT ===================================== #
 #                                                                                       #
-#  Some of the information used to build the ROS2 ABB-IRB120 .urdf files in this ROS2   #
-#  repository has been taken from the following resource:                               #
+#  Some of the information used to build the ROS 2 ABB-IRB120 .urdf files in this       #
+#  ROS 2 repository has been taken from the following resource:                         #
 #       - abb_experimental (https://github.com/ros-industrial/abb_experimental)         #
 #                                                                                       #
@@ -49,6 +49,6 @@
 <robot xmlns:xacro="http://www.ros.org/wiki/xacro">
   <xacro:macro name="irb120_ros2control" params="bringup robot_ip EE EE_name prefix" >
-    <!-- 1. ROS2_CONTROL tag name: -->
-    <!-- A. GAZEBO SIMULATION: -->
+    <!-- 1. ros2_control tag name: -->
+    <!-- A. GZ Sim simulation: -->
     <xacro:unless value="${bringup}">
       <xacro:property name="name" value="${prefix}GazeboSimSystem"/>
@@ -58,7 +58,7 @@
       <xacro:property name="name" value="${prefix}ABBMultiInterfaceHardware"/>
     </xacro:if>
-    <!-- 3. Load ROS2_CONTROL: -->
+    <!-- 3. Load ros2_control: -->
     <ros2_control name="${name}" type="system">
-      <!-- A. GAZEBO SIMULATION: -->
+      <!-- A. GZ Sim simulation: -->
       <xacro:unless value="${bringup}">
         <hardware>

File: ros2srrc_robots/irb120/urdf/irb120_transmission.xacro (robot description, xacro)
@@ -26,6 +26,6 @@
 # ===================================== COPYRIGHT ===================================== #
 #                                                                                       #
-#  Some of the information used to build the ROS2 ABB-IRB120 .urdf files in this ROS2   #
-#  repository has been taken from the following resource:                               #
+#  Some of the information used to build the ROS 2 ABB-IRB120 .urdf files in this       #
+#  ROS 2 repository has been taken from the following resource:                         #
 #       - abb_experimental (https://github.com/ros-industrial/abb_experimental)         #
 #                                                                                       #

File: ros2srrc_robots/irb1200/urdf/irb1200_macro.urdf.xacro (robot description, xacro)
@@ -26,6 +26,6 @@
 # ===================================== COPYRIGHT ===================================== #
 #                                                                                       #
-#  Some of the information used to build the ROS2 ABB-IRB1200 .urdf files in this ROS2   #
-#  repository has been taken from the following resource:                               #
+#  Some of the information used to build the ROS 2 ABB-IRB1200 .urdf files in this      #
+#  ROS 2 repository has been taken from the following resource:                         #
 #       - abb_experimental (https://github.com/ros-industrial/abb_experimental)         #
 #                                                                                       #
@@ -58,5 +58,5 @@
       prefix="${prefix}" />
     </xacro:unless>
-    <!-- ABB-IRB1200 GAZEBO - ROS2_CONTROL: -->
+    <!-- ABB-IRB1200 GZ Sim - ros2_control: -->
     <xacro:include filename="$(find ros2srrc_robots)/irb1200/urdf/irb1200_ros2control.xacro" />
     <xacro:irb1200_ros2control

File: ros2srrc_robots/irb1200/urdf/irb1200_ros2control.xacro (robot description, xacro)
@@ -26,6 +26,6 @@
 # ===================================== COPYRIGHT ===================================== #
 #                                                                                       #
-#  Some of the information used to build the ROS2 ABB-IRB1200 .urdf files in this ROS2   #
-#  repository has been taken from the following resource:                               #
+#  Some of the information used to build the ROS 2 ABB-IRB1200 .urdf files in this      #
+#  ROS 2 repository has been taken from the following resource:                         #
 #       - abb_experimental (https://github.com/ros-industrial/abb_experimental)         #
 #                                                                                       #
@@ -49,6 +49,6 @@
 <robot xmlns:xacro="http://www.ros.org/wiki/xacro">
   <xacro:macro name="irb1200_ros2control" params="bringup robot_ip EE EE_name prefix" >
-    <!-- 1. ROS2_CONTROL tag name: -->
-    <!-- A. GAZEBO SIMULATION: -->
+    <!-- 1. ros2_control tag name: -->
+    <!-- A. GZ Sim simulation: -->
     <xacro:unless value="${bringup}">
       <xacro:property name="name" value="${prefix}GazeboSimSystem"/>
@@ -58,7 +58,7 @@
       <xacro:property name="name" value="${prefix}ABBMultiInterfaceHardware"/>
     </xacro:if>
-    <!-- 3. Load ROS2_CONTROL: -->
+    <!-- 3. Load ros2_control: -->
     <ros2_control name="${name}" type="system">
-      <!-- A. GAZEBO SIMULATION: -->
+      <!-- A. GZ Sim simulation: -->
       <xacro:unless value="${bringup}">
         <hardware>

File: ros2srrc_robots/irb1200/urdf/irb1200_transmission.xacro (robot description, xacro)
@@ -26,6 +26,6 @@
 # ===================================== COPYRIGHT ===================================== #
 #                                                                                       #
-#  Some of the information used to build the ROS2 ABB-IRB1200 .urdf files in this ROS2   #
-#  repository has been taken from the following resource:                               #
+#  Some of the information used to build the ROS 2 ABB-IRB1200 .urdf files in this      #
+#  ROS 2 repository has been taken from the following resource:                         #
 #       - abb_experimental (https://github.com/ros-industrial/abb_experimental)         #
 #                                                                                       #
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