Commit message: ros2srrc for ROS 2 Jazzy: Finalise repo (fix inconsistencies, update documentation).

File: packages/ros2srrc_ur20/urdf/ur20.urdf.xacro (robot description, xacro)
@@ -47,5 +47,5 @@
   <xacro:arg name="output_recipe_filename" default="none"/>
   <xacro:property name="output_recipe_filename" value="$(arg output_recipe_filename)"/>
-  <!-- Include XACRO-MACRO file of the ur20: -->
+  <!-- Include XACRO-MACRO file of the UR20: -->
   <xacro:include filename="$(find ros2srrc_robots)/ur20/urdf/ur20_macro.urdf.xacro"/>
   <xacro:ur20
@@ -62,5 +62,5 @@
     <gazebo>
       <plugin filename="gz_ros2_control-system" name="gz_ros2_control::GazeboSimROS2ControlPlugin">
-        <!-- ur20 Controller -->
+        <!-- UR20 Controller -->
         <parameters>$(find ros2srrc_robots)/ur20/config/controller.yaml</parameters>
       </plugin>

File: ros2srrc_robots/iiwa/urdf/iiwa_macro.urdf.xacro (robot description, xacro)
@@ -276,5 +276,5 @@
       <axis xyz="0 -1 0"/>
       <limit effort="176" lower="-2.0942" upper="2.0942" velocity="1.3089"/>
-      <dynamics damping="10.0" friction="1.0"/> <!-- High values of damping + friction were added, to avoid bac joint behaviour in GzFortress. -->
+      <dynamics damping="10.0" friction="1.0"/> <!-- High values of damping + friction were added to avoid bad joint behaviour in Gz Harmonic. -->
     </joint>
     <joint name="${prefix}joint_5" type="revolute">

File: ros2srrc_robots/ur20/urdf/ur20_macro.urdf.xacro (robot description, xacro)
@@ -79,5 +79,5 @@
       output_recipe_filename="${output_recipe_filename}"
       prefix="${prefix}" />
-    <!-- ***** ur20 ROBOT .urdf SERIAL CHAIN ***** -->
+    <!-- ***** UR20 ROBOT .urdf SERIAL CHAIN ***** -->
     <!-- Links: -->
     <link name="${prefix}base_link"/>

File: ros2srrc_robots/ur20/urdf/ur20_ros2control.xacro (robot description, xacro)
@@ -26,5 +26,5 @@
 # ===================================== COPYRIGHT ===================================== #
 #                                                                                       #
-#  Some of the information used to build the ROS2 ur20-Robot .urdf files in this ROS2    #
+#  Some of the information used to build the ROS2 UR20-Robot .urdf files in this ROS2   #
 #  repository has been taken from the following resources:                              #
 #       - Universal Robots ROS2 Description:                                            #

File: ros2srrc_robots/ur20/urdf/ur20_transmission.xacro (robot description, xacro)
@@ -27,5 +27,5 @@
 # ===================================== COPYRIGHT ===================================== #
 #                                                                                       #
-#  Some of the information used to build the ROS2 ur20-Robot .urdf files in this ROS2    #
+#  Some of the information used to build the ROS2 UR20-Robot .urdf files in this ROS2   #
 #  repository has been taken from the following resources:                              #
 #       - Universal Robots ROS2 Description:                                            #

File: ros2srrc_robots/ur3e/urdf/ur3e_common.xacro (robot description, xacro)
@@ -26,5 +26,5 @@
 # ===================================== COPYRIGHT ===================================== #
 #                                                                                       #
-#  Some of the information used to build the ROS2 UR3-Robot .urdf files in this ROS2    #
+#  Some of the information used to build the ROS2 UR3e-Robot .urdf files in this ROS2   #
 #  repository has been taken from the following resources:                              #
 #       - Universal Robots ROS2 Description:                                            #

File: ros2srrc_robots/ur3e/urdf/ur3e_macro.urdf.xacro (robot description, xacro)
@@ -26,5 +26,5 @@
 # ===================================== COPYRIGHT ===================================== #
 #                                                                                       #
-#  Some of the information used to build the ROS2 UR3-Robot .urdf files in this ROS2    #
+#  Some of the information used to build the ROS2 UR3e-Robot .urdf files in this ROS2   #
 #  repository has been taken from the following resources:                              #
 #       - Universal Robots ROS2 Description:                                            #

File: ros2srrc_robots/ur3e/urdf/ur3e_ros2control.xacro (robot description, xacro)
@@ -26,5 +26,5 @@
 # ===================================== COPYRIGHT ===================================== #
 #                                                                                       #
-#  Some of the information used to build the ROS2 UR3-Robot .urdf files in this ROS2    #
+#  Some of the information used to build the ROS2 UR3e-Robot .urdf files in this ROS2   #
 #  repository has been taken from the following resources:                              #
 #       - Universal Robots ROS2 Description:                                            #

File: ros2srrc_robots/ur3e/urdf/ur3e_transmission.xacro (robot description, xacro)
@@ -26,5 +26,5 @@
 # ===================================== COPYRIGHT ===================================== #
 #                                                                                       #
-#  Some of the information used to build the ROS2 UR3-Robot .urdf files in this ROS2    #
+#  Some of the information used to build the ROS2 UR3e-Robot .urdf files in this ROS2   #
 #  repository has been taken from the following resources:                              #
 #       - Universal Robots ROS2 Description:                                            #

File: ros2srrc_robots/ur5e/urdf/ur5e_macro.urdf.xacro (robot description, xacro)
@@ -26,5 +26,5 @@
 # ===================================== COPYRIGHT ===================================== #
 #                                                                                       #
-#  Some of the information used to build the ROS2 UR5-Robot .urdf files in this ROS2    #
+#  Some of the information used to build the ROS2 UR5e-Robot .urdf files in this ROS2   #
 #  repository has been taken from the following resources:                              #
 #       - Universal Robots ROS2 Description:                                            #

File: ros2srrc_robots/ur5e/urdf/ur5e_ros2control.xacro (robot description, xacro)
@@ -26,5 +26,5 @@
 # ===================================== COPYRIGHT ===================================== #
 #                                                                                       #
-#  Some of the information used to build the ROS2 UR5-Robot .urdf files in this ROS2    #
+#  Some of the information used to build the ROS2 UR5e-Robot .urdf files in this ROS2   #
 #  repository has been taken from the following resources:                              #
 #       - Universal Robots ROS2 Description:                                            #
